Commit message: Removed underscore after prefix.

File: jackal_description/urdf/accessories/sick_lms1xx_mount.urdf.xacro (robot description, xacro)
@@ -43,5 +43,5 @@
       <origin xyz="0 0 0.149" rpy="0 0 0" />
       <parent link="${prefix}_laser_mount" />
-      <child link="${prefix}_laser" />
+      <child link="${prefix}laser" />
     </joint>
   </xacro:macro>
