Commit message: Simulate the depthimage_to_laserscan node by adding the laser plugin for the kinect too; ideally we want to remove this, but there's a bug with the openni kinect plugin for gazebo that prevents that from working correctly for now

File: jackal_description/urdf/accessories/azure_kinect.urdf.xacro (robot description, xacro)
@@ -21,5 +21,8 @@
 -->
 <robot xmlns:xacro="http://www.ros.org/wiki/xacro">
-  <xacro:macro name="azure_kinect" params="prefix">
+  <xacro:macro name="azure_kinect" params="prefix min_range:=0.5 max_range:=5.46
+                    update_rate:=30
+                    h_fov:=1.3089958333333334 v_fov:=1.1344630555555555
+                    width:=576 height:=640">
     <link name="${prefix}_kinect_body">
       <visual>
@@ -79,9 +82,9 @@
       <turnGravityOff>true</turnGravityOff>
       <sensor type="depth" name="${prefix}_kinect_depth">
-        <update_rate>30</update_rate>
+        <update_rate>${update_rate}</update_rate>
         <camera>
           <!-- 75x65 degree FOV for the depth sensor -->
-          <horizontal_fov>1.3089958333333334</horizontal_fov>
-          <vertical_fov>1.1344630555555555</vertical_fov>
+          <horizontal_fov>${h_fov}</horizontal_fov>
+          <vertical_fov>${v_fov}</vertical_fov>
           <!-- 90x59 degree FOV for the hardware color camera -->
           <!-- currently disabled, as this would mangle the depth data
@@ -95,6 +98,6 @@
               see: https://docs.microsoft.com/en-us/azure/kinect-dk/hardware-specification
             -->
-            <width>640</width>
-            <height>576</height>
+            <width>${width}</width>
+            <height>${height}</height>
             <!-- TODO: check what format the Azure Kinect hardware delivers and set this to match! -->
             <format>R8G8B8</format>
@@ -109,5 +112,5 @@
           <baseline>0.2</baseline>
           <alwaysOn>true</alwaysOn>
-          <updateRate>1.0</updateRate>
+          <updateRate>0.0</updateRate>
           <cameraName>kinect</cameraName>
           <imageTopicName>/color/image_raw</imageTopicName>
@@ -118,6 +121,6 @@
           <frameName>${prefix}_kinect_gazebo_lens</frameName>
           <!-- the Azure Kinect has an effective depth-sensing range of 0.5m to 5.46m -->
-          <pointCloudCutoff>0.5</pointCloudCutoff>
-          <pointCloudCutoffMax>5.46</pointCloudCutoffMax>
+          <pointCloudCutoff>${min_range}</pointCloudCutoff>
+          <pointCloudCutoffMax>${max_range}</pointCloudCutoffMax>
           <distortionK1>0.00000001</distortionK1>
           <distortionK2>0.00000001</distortionK2>
@@ -132,4 +135,40 @@
         </plugin>
       </sensor>
+      <!--
+        to simulate the depthimage_to_laserscan node in the bringup, we also add a laser
+        plugin that publishes to the same topic
+        ideally we would just launch the depthimage_to_laserscan node, but there seems to be a bug
+        in the libgazebo_ros_openni_kinect plugin that's preventing the (required) /depth/camera_data
+        topic from publishing correctly.  so for now we'll fake it with the laser plugin
+      -->
+      <sensor type="ray" name="${prefix}_kinect_scan">
+        <pose>0 0 0 0 0 0</pose>
+        <visualize>false</visualize>
+        <update_rate>${update_rate}</update_rate>
+        <ray>
+          <scan>
+            <horizontal>
+              <samples>${width}</samples>
+              <resolution>1</resolution>
+              <min_angle>${h_fov/-2}</min_angle>
+              <max_angle>${h_fov/2}</max_angle>
+            </horizontal>
+          </scan>
+          <range>
+            <min>${min_range}</min>
+            <max>${max_range}</max>
+            <resolution>0.001</resolution>
+          </range>
+          <noise>
+            <type>gaussian</type>
+            <mean>0.0</mean>
+            <stddev>0.001</stddev>
+          </noise>
+        </ray>
+        <plugin name="gazebo_ros_laser" filename="libgazebo_ros_laser.so">
+          <topicName>/$(optenv JACKAL_AZURE_KINECT_MOUNT front)/scan</topicName>
+          <frameName>${prefix}_kinect_visor</frameName>
+        </plugin>
+      </sensor>
     </gazebo>
   </xacro:macro>

Commit message: Update the Azure kinect description after testing on the physical robot

File: jackal_description/urdf/accessories/azure_kinect.urdf.xacro (robot description, xacro)
@@ -22,4 +22,10 @@
 <robot xmlns:xacro="http://www.ros.org/wiki/xacro">
   <xacro:macro name="azure_kinect_mount" params="prefix topic parent_link">
+    <!--
+      NOTE: the frame parameter not currently used as-intended!
+      The Azure Kinect ROS driver requires links named camera_base, camera_visor, and camera_body.  We cannot
+      override these right now and have the driver work in its current state.
+      Therefore the links are named camera_*, while joints & gazebo work-arounds use the specified frame
+    -->
     <xacro:macro name="azure_kinect" params="
                       frame:=kinect       topic:=kinect
@@ -29,5 +35,5 @@
                       width:=576 height:=640">
       <!-- this link is the origin for the camera data and corresponds to the front visor of the camera -->
-      <link name="${frame}">
+      <link name="camera_visor">
         <visual>
           <origin xyz="-0.0128 0. 0." />
@@ -38,5 +44,5 @@
         </visual>
       </link>
-      <link name="${frame}_body">
+      <link name="camera_body">
         <visual>
           <origin xyz="0. 0. 0." />
@@ -47,5 +53,5 @@
         </visual>
       </link>
-      <link name="${frame}_base">
+      <link name="camera_base">
         <visual>
           <origin xyz="-0.013 0. 0." />
@@ -57,11 +63,11 @@
       </link>
       <joint name="${frame}_base_to_body" type="fixed">
-        <parent link="${frame}_base" />
-        <child link="${frame}_body" />
+        <parent link="camera_base" />
+        <child link="camera_body" />
         <origin xyz="-0.0757 0. 0.008" rpy="0. 0. 0." />
       </joint>
       <joint name="${frame}_base_to_visor" type="fixed">
-        <parent link="${frame}_base" />
-        <child link="${frame}" />
+        <parent link="camera_base" />
+        <child link="camera_visor" />
         <origin xyz="0. 0. 0." rpy="0. 0. 0." />
       </joint>
@@ -71,7 +77,7 @@
         This link only exists to give the gazebo plugin the correctly-oriented frame
       -->
-      <link name="${prefix}_kinect_gazebo" />
-      <joint name="${prefix}_kinect_gazebo_joint" type="fixed">
-        <parent link="${frame}"/>
+      <link name="${frame}_gazebo" />
+      <joint name="${frame}_gazebo_joint" type="fixed">
+        <parent link="camera_visor"/>
         <child link="${frame}_gazebo"/>
         <origin xyz="0 0 0" rpy="-1.5707963267948966 0 -1.5707963267948966"/>
@@ -83,5 +89,5 @@
         But for now the OpenNI kinect plugin is the closest analogue
       -->
-      <gazebo reference="${frame}">
+      <gazebo reference="camera_visor">
         <turnGravityOff>true</turnGravityOff>
         <sensor type="depth" name="${prefix}_kinect_depth">
@@ -122,5 +128,5 @@
             <depthImageTopicName>depth/image_raw</depthImageTopicName>
             <depthImageInfoTopicName>depth/camera_info</depthImageInfoTopicName>
-            <pointCloudTopicName>depth/points</pointCloudTopicName>
+            <pointCloudTopicName>depth/points2</pointCloudTopicName>
             <frameName>${frame}_gazebo</frameName>
             <!-- the Azure Kinect has an effective depth-sensing range of 0.5m to 5.46m -->

Commit message: Fix the link between the mounting plate and the camera base

File: jackal_description/urdf/accessories/azure_kinect.urdf.xacro (robot description, xacro)
@@ -166,5 +166,5 @@
       <origin xyz="0.09 0 0.0335" rpy="0 -0.17453292519444444 0"/>
       <parent link="${prefix}_kinect_mount_plate"/>
-      <child link="${prefix}_kinect_base"/>
+      <child link="camera_base"/>
     </joint>
     <xacro:azure_kinect frame="${prefix}_kinect" topic="${topic}"/>
