Commit message: Replace the slightly wonky-looking Smart7 DAE with a new STL from Jeff

File: jackal_description/urdf/accessories/novatel_smart7.urdf.xacro (robot description, xacro)
@@ -4,7 +4,7 @@
     <link name="${prefix}_navsat">
       <visual>
-        <origin xyz="0 0 0" rpy="0 0 0" />
+        <origin xyz="-0.095 0 0" rpy="${pi/2} 0 -${pi/2}" />
         <geometry>
-          <mesh filename="package://jackal_description/meshes/novatel-smart7.dae"/>
+          <mesh filename="package://jackal_description/meshes/novatel-smart7.stl"/>
         </geometry>
         <material name="novatel_white">

Commit message: Add the collision body for the Smart7, just in case we need to worry about IK implications with an arm.

File: jackal_description/urdf/accessories/novatel_smart7.urdf.xacro (robot description, xacro)
@@ -12,4 +12,10 @@
         </material>
       </visual>
+      <collision>
+        <origin xyz="-0.095 0 0" rpy="${pi/2} 0 -${pi/2}" />
+        <geometry>
+          <mesh filename="package://jackal_description/meshes/novatel-smart7.stl"/>
+        </geometry>
+      </collision>
     </link>
   </xacro:macro>

Commit message: Update the mesh for the Smart7 so it's more accurate (#87)
* Replace the slightly wonky-looking Smart7 DAE with a new STL from Jeff

* Add the collision body for the Smart7, just in case we need to worry about IK implications with an arm.

File: jackal_description/urdf/accessories/novatel_smart7.urdf.xacro (robot description, xacro)
@@ -4,7 +4,7 @@
     <link name="${prefix}_navsat">
       <visual>
-        <origin xyz="0 0 0" rpy="0 0 0" />
+        <origin xyz="-0.095 0 0" rpy="${pi/2} 0 -${pi/2}" />
         <geometry>
-          <mesh filename="package://jackal_description/meshes/novatel-smart7.dae"/>
+          <mesh filename="package://jackal_description/meshes/novatel-smart7.stl"/>
         </geometry>
         <material name="novatel_white">
@@ -12,4 +12,10 @@
         </material>
       </visual>
+      <collision>
+        <origin xyz="-0.095 0 0" rpy="${pi/2} 0 -${pi/2}" />
+        <geometry>
+          <mesh filename="package://jackal_description/meshes/novatel-smart7.stl"/>
+        </geometry>
+      </collision>
     </link>
   </xacro:macro>
