Commit message: Added a tab and space

File: jackal_description/urdf/accessories/vlp16_mount.urdf.xacro (robot description, xacro)
@@ -2,93 +2,93 @@
   <xacro:include filename="$(find velodyne_description)/urdf/VLP-16.urdf.xacro" />
   <xacro:macro name="vlp16_mount" params="prefix parent_link topic tower height:=0.1 *origin">
-   <xacro:if value="${tower}">
-     <link name="${prefix}_vlp16_mount" />
-     <link name="${prefix}_vlp16_plate">
-       <visual>
-         <geometry>
-           <box size="0.1 0.1 0.002" />
-         </geometry>
-         <material name="black" />
-         <origin xyz="0 0 -0.001" rpy="0 0 0" />
-       </visual>
-     </link>
-     <link name="${prefix}_vlp16_leg1">
-       <visual>
-         <geometry>
-           <cylinder length="${height}" radius="0.003" />
-         </geometry>
-         <material name="white">
-           <color rgba="1 1 1 1" />
-         </material>
-         <origin xyz="0 0 ${height/2}" rpy="0 0 0" />
-       </visual>
-     </link>
-     <link name="${prefix}_vlp16_leg2">
-       <visual>
-         <geometry>
-           <cylinder length="${height}" radius="0.003" />
-         </geometry>
-         <material name="white">
-           <color rgba="1 1 1 1" />
-         </material>
-         <origin xyz="0 0 ${height/2}" rpy="0 0 0" />
-       </visual>
-     </link>
-     <link name="${prefix}_vlp16_leg3">
-       <visual>
-         <geometry>
-           <cylinder length="${height}" radius="0.003" />
-         </geometry>
-         <material name="white">
-           <color rgba="1 1 1 1" />
-         </material>
-         <origin xyz="0 0 ${height/2}" rpy="0 0 0" />
-       </visual>
-     </link>
-     <link name="${prefix}_vlp16_leg4">
-       <visual>
-         <geometry>
-           <cylinder length="${height}" radius="0.003" />
-         </geometry>
-         <material name="white">
-           <color rgba="1 1 1 1" />
-         </material>
-         <origin xyz="0 0 ${height/2}" rpy="0 0 0" />
-       </visual>
-     </link>
-     <joint name="${prefix}_vlp16_mount_joint" type="fixed">
-       <parent link="${parent_link}" />
-       <child link="${prefix}_vlp16_mount" />
-       <xacro:insert_block name="origin" />
-     </joint>
-     <joint name="${prefix}_vlp16_leg1_joint" type="fixed">
-       <parent link="${prefix}_vlp16_mount" />
-       <child link="${prefix}_vlp16_leg1" />
-       <origin xyz="0.05 0.05 0" rpy="0 0 0" />
-     </joint>
-     <joint name="${prefix}_vlp16_leg2_joint" type="fixed">
-       <parent link="${prefix}_vlp16_mount" />
-       <child link="${prefix}_vlp16_leg2" />
-       <origin xyz="0.05 -0.05 0" rpy="0 0 0" />
-     </joint>
-     <joint name="${prefix}_vlp16_leg3_joint" type="fixed">
-       <parent link="${prefix}_vlp16_mount" />
-       <child link="${prefix}_vlp16_leg3" />
-       <origin xyz="-0.05 0.05 0" rpy="0 0 0" />
-     </joint>
-     <joint name="${prefix}_vlp16_leg4_joint" type="fixed">
-       <parent link="${prefix}_vlp16_mount" />
-       <child link="${prefix}_vlp16_leg4" />
-       <origin xyz="-0.05 -0.05 0" rpy="0 0 0" />
-     </joint>
-     <joint name="${prefix}_vlp16_plate_joint" type="fixed">
-       <parent link="${prefix}_vlp16_mount" />
-       <child link="${prefix}_vlp16_plate" />
-       <origin xyz="0 0 ${height}" rpy="0 0 0" />
-     </joint>
-     <xacro:VLP-16 parent="${prefix}_vlp16_plate" topic="${topic}">
-       <origin xyz="0 0 0" rpy="0 0 0" />
-     </xacro:VLP-16>
-   </xacro:if>
+      <xacro:if value="${tower}">
+        <link name="${prefix}_vlp16_mount" />
+        <link name="${prefix}_vlp16_plate">
+          <visual>
+            <geometry>
+              <box size="0.1 0.1 0.002" />
+            </geometry>
+            <material name="black" />
+            <origin xyz="0 0 -0.001" rpy="0 0 0" />
+          </visual>
+        </link>
+        <link name="${prefix}_vlp16_leg1">
+          <visual>
+            <geometry>
+              <cylinder length="${height}" radius="0.003" />
+            </geometry>
+            <material name="white">
+              <color rgba="1 1 1 1" />
+            </material>
+            <origin xyz="0 0 ${height/2}" rpy="0 0 0" />
+          </visual>
+        </link>
+        <link name="${prefix}_vlp16_leg2">
+          <visual>
+            <geometry>
+              <cylinder length="${height}" radius="0.003" />
+            </geometry>
+            <material name="white">
+              <color rgba="1 1 1 1" />
+            </material>
+            <origin xyz="0 0 ${height/2}" rpy="0 0 0" />
+          </visual>
+        </link>
+        <link name="${prefix}_vlp16_leg3">
+          <visual>
+            <geometry>
+              <cylinder length="${height}" radius="0.003" />
+            </geometry>
+            <material name="white">
+              <color rgba="1 1 1 1" />
+            </material>
+            <origin xyz="0 0 ${height/2}" rpy="0 0 0" />
+          </visual>
+        </link>
+        <link name="${prefix}_vlp16_leg4">
+          <visual>
+            <geometry>
+              <cylinder length="${height}" radius="0.003" />
+            </geometry>
+            <material name="white">
+              <color rgba="1 1 1 1" />
+            </material>
+            <origin xyz="0 0 ${height/2}" rpy="0 0 0" />
+          </visual>
+        </link>
+        <joint name="${prefix}_vlp16_mount_joint" type="fixed">
+          <parent link="${parent_link}" />
+          <child link="${prefix}_vlp16_mount" />
+          <xacro:insert_block name="origin" />
+        </joint>
+        <joint name="${prefix}_vlp16_leg1_joint" type="fixed">
+          <parent link="${prefix}_vlp16_mount" />
+          <child link="${prefix}_vlp16_leg1" />
+          <origin xyz="0.05 0.05 0" rpy="0 0 0" />
+        </joint>
+        <joint name="${prefix}_vlp16_leg2_joint" type="fixed">
+          <parent link="${prefix}_vlp16_mount" />
+          <child link="${prefix}_vlp16_leg2" />
+          <origin xyz="0.05 -0.05 0" rpy="0 0 0" />
+        </joint>
+        <joint name="${prefix}_vlp16_leg3_joint" type="fixed">
+          <parent link="${prefix}_vlp16_mount" />
+          <child link="${prefix}_vlp16_leg3" />
+          <origin xyz="-0.05 0.05 0" rpy="0 0 0" />
+        </joint>
+        <joint name="${prefix}_vlp16_leg4_joint" type="fixed">
+          <parent link="${prefix}_vlp16_mount" />
+          <child link="${prefix}_vlp16_leg4" />
+          <origin xyz="-0.05 -0.05 0" rpy="0 0 0" />
+        </joint>
+        <joint name="${prefix}_vlp16_plate_joint" type="fixed">
+          <parent link="${prefix}_vlp16_mount" />
+          <child link="${prefix}_vlp16_plate" />
+          <origin xyz="0 0 ${height}" rpy="0 0 0" />
+        </joint>
+        <xacro:VLP-16 parent="${prefix}_vlp16_plate" topic="${topic}">
+          <origin xyz="0 0 0" rpy="0 0 0" />
+        </xacro:VLP-16>
+      </xacro:if>
     <xacro:unless value="${tower}">
       <xacro:VLP-16 parent="${parent_link}" topic="${topic}">

Commit message: Removed tab

File: jackal_description/urdf/accessories/vlp16_mount.urdf.xacro (robot description, xacro)
@@ -2,93 +2,93 @@
   <xacro:include filename="$(find velodyne_description)/urdf/VLP-16.urdf.xacro" />
   <xacro:macro name="vlp16_mount" params="prefix parent_link topic tower height:=0.1 *origin">
-      <xacro:if value="${tower}">
-        <link name="${prefix}_vlp16_mount" />
-        <link name="${prefix}_vlp16_plate">
-          <visual>
-            <geometry>
-              <box size="0.1 0.1 0.002" />
-            </geometry>
-            <material name="black" />
-            <origin xyz="0 0 -0.001" rpy="0 0 0" />
-          </visual>
-        </link>
-        <link name="${prefix}_vlp16_leg1">
-          <visual>
-            <geometry>
-              <cylinder length="${height}" radius="0.003" />
-            </geometry>
-            <material name="white">
-              <color rgba="1 1 1 1" />
-            </material>
-            <origin xyz="0 0 ${height/2}" rpy="0 0 0" />
-          </visual>
-        </link>
-        <link name="${prefix}_vlp16_leg2">
-          <visual>
-            <geometry>
-              <cylinder length="${height}" radius="0.003" />
-            </geometry>
-            <material name="white">
-              <color rgba="1 1 1 1" />
-            </material>
-            <origin xyz="0 0 ${height/2}" rpy="0 0 0" />
-          </visual>
-        </link>
-        <link name="${prefix}_vlp16_leg3">
-          <visual>
-            <geometry>
-              <cylinder length="${height}" radius="0.003" />
-            </geometry>
-            <material name="white">
-              <color rgba="1 1 1 1" />
-            </material>
-            <origin xyz="0 0 ${height/2}" rpy="0 0 0" />
-          </visual>
-        </link>
-        <link name="${prefix}_vlp16_leg4">
-          <visual>
-            <geometry>
-              <cylinder length="${height}" radius="0.003" />
-            </geometry>
-            <material name="white">
-              <color rgba="1 1 1 1" />
-            </material>
-            <origin xyz="0 0 ${height/2}" rpy="0 0 0" />
-          </visual>
-        </link>
-        <joint name="${prefix}_vlp16_mount_joint" type="fixed">
-          <parent link="${parent_link}" />
-          <child link="${prefix}_vlp16_mount" />
-          <xacro:insert_block name="origin" />
-        </joint>
-        <joint name="${prefix}_vlp16_leg1_joint" type="fixed">
-          <parent link="${prefix}_vlp16_mount" />
-          <child link="${prefix}_vlp16_leg1" />
-          <origin xyz="0.05 0.05 0" rpy="0 0 0" />
-        </joint>
-        <joint name="${prefix}_vlp16_leg2_joint" type="fixed">
-          <parent link="${prefix}_vlp16_mount" />
-          <child link="${prefix}_vlp16_leg2" />
-          <origin xyz="0.05 -0.05 0" rpy="0 0 0" />
-        </joint>
-        <joint name="${prefix}_vlp16_leg3_joint" type="fixed">
-          <parent link="${prefix}_vlp16_mount" />
-          <child link="${prefix}_vlp16_leg3" />
-          <origin xyz="-0.05 0.05 0" rpy="0 0 0" />
-        </joint>
-        <joint name="${prefix}_vlp16_leg4_joint" type="fixed">
-          <parent link="${prefix}_vlp16_mount" />
-          <child link="${prefix}_vlp16_leg4" />
-          <origin xyz="-0.05 -0.05 0" rpy="0 0 0" />
-        </joint>
-        <joint name="${prefix}_vlp16_plate_joint" type="fixed">
-          <parent link="${prefix}_vlp16_mount" />
-          <child link="${prefix}_vlp16_plate" />
-          <origin xyz="0 0 ${height}" rpy="0 0 0" />
-        </joint>
-        <xacro:VLP-16 parent="${prefix}_vlp16_plate" topic="${topic}">
-          <origin xyz="0 0 0" rpy="0 0 0" />
-        </xacro:VLP-16>
-      </xacro:if>
+    <xacro:if value="${tower}">
+      <link name="${prefix}_vlp16_mount" />
+      <link name="${prefix}_vlp16_plate">
+        <visual>
+          <geometry>
+            <box size="0.1 0.1 0.002" />
+          </geometry>
+          <material name="black" />
+          <origin xyz="0 0 -0.001" rpy="0 0 0" />
+        </visual>
+      </link>
+      <link name="${prefix}_vlp16_leg1">
+        <visual>
+          <geometry>
+            <cylinder length="${height}" radius="0.003" />
+          </geometry>
+          <material name="white">
+            <color rgba="1 1 1 1" />
+          </material>
+          <origin xyz="0 0 ${height/2}" rpy="0 0 0" />
+        </visual>
+      </link>
+      <link name="${prefix}_vlp16_leg2">
+        <visual>
+          <geometry>
+            <cylinder length="${height}" radius="0.003" />
+          </geometry>
+          <material name="white">
+            <color rgba="1 1 1 1" />
+          </material>
+          <origin xyz="0 0 ${height/2}" rpy="0 0 0" />
+        </visual>
+      </link>
+      <link name="${prefix}_vlp16_leg3">
+        <visual>
+          <geometry>
+            <cylinder length="${height}" radius="0.003" />
+          </geometry>
+          <material name="white">
+            <color rgba="1 1 1 1" />
+          </material>
+          <origin xyz="0 0 ${height/2}" rpy="0 0 0" />
+        </visual>
+      </link>
+      <link name="${prefix}_vlp16_leg4">
+        <visual>
+          <geometry>
+            <cylinder length="${height}" radius="0.003" />
+          </geometry>
+          <material name="white">
+            <color rgba="1 1 1 1" />
+          </material>
+          <origin xyz="0 0 ${height/2}" rpy="0 0 0" />
+        </visual>
+      </link>
+      <joint name="${prefix}_vlp16_mount_joint" type="fixed">
+        <parent link="${parent_link}" />
+        <child link="${prefix}_vlp16_mount" />
+        <xacro:insert_block name="origin" />
+      </joint>
+      <joint name="${prefix}_vlp16_leg1_joint" type="fixed">
+        <parent link="${prefix}_vlp16_mount" />
+        <child link="${prefix}_vlp16_leg1" />
+        <origin xyz="0.05 0.05 0" rpy="0 0 0" />
+      </joint>
+      <joint name="${prefix}_vlp16_leg2_joint" type="fixed">
+        <parent link="${prefix}_vlp16_mount" />
+        <child link="${prefix}_vlp16_leg2" />
+        <origin xyz="0.05 -0.05 0" rpy="0 0 0" />
+      </joint>
+      <joint name="${prefix}_vlp16_leg3_joint" type="fixed">
+        <parent link="${prefix}_vlp16_mount" />
+        <child link="${prefix}_vlp16_leg3" />
+        <origin xyz="-0.05 0.05 0" rpy="0 0 0" />
+      </joint>
+      <joint name="${prefix}_vlp16_leg4_joint" type="fixed">
+        <parent link="${prefix}_vlp16_mount" />
+        <child link="${prefix}_vlp16_leg4" />
+        <origin xyz="-0.05 -0.05 0" rpy="0 0 0" />
+      </joint>
+      <joint name="${prefix}_vlp16_plate_joint" type="fixed">
+        <parent link="${prefix}_vlp16_mount" />
+        <child link="${prefix}_vlp16_plate" />
+        <origin xyz="0 0 ${height}" rpy="0 0 0" />
+      </joint>
+      <xacro:VLP-16 parent="${prefix}_vlp16_plate" topic="${topic}">
+        <origin xyz="0 0 0" rpy="0 0 0" />
+      </xacro:VLP-16>
+    </xacro:if>
     <xacro:unless value="${tower}">
       <xacro:VLP-16 parent="${parent_link}" topic="${topic}">

Commit message: Added tab to vlp16_plate

File: jackal_description/urdf/accessories/vlp16_mount.urdf.xacro (robot description, xacro)
@@ -4,13 +4,13 @@
     <xacro:if value="${tower}">
       <link name="${prefix}_vlp16_mount" />
-      <link name="${prefix}_vlp16_plate">
-        <visual>
-          <geometry>
-            <box size="0.1 0.1 0.002" />
-          </geometry>
-          <material name="black" />
-          <origin xyz="0 0 -0.001" rpy="0 0 0" />
-        </visual>
-      </link>
+        <link name="${prefix}_vlp16_plate">
+          <visual>
+            <geometry>
+              <box size="0.1 0.1 0.002" />
+            </geometry>
+            <material name="black" />
+            <origin xyz="0 0 -0.001" rpy="0 0 0" />
+          </visual>
+        </link>
       <link name="${prefix}_vlp16_leg1">
         <visual>

Commit message: Removed tab from vlp16_plate

File: jackal_description/urdf/accessories/vlp16_mount.urdf.xacro (robot description, xacro)
@@ -4,13 +4,13 @@
     <xacro:if value="${tower}">
       <link name="${prefix}_vlp16_mount" />
-        <link name="${prefix}_vlp16_plate">
-          <visual>
-            <geometry>
-              <box size="0.1 0.1 0.002" />
-            </geometry>
-            <material name="black" />
-            <origin xyz="0 0 -0.001" rpy="0 0 0" />
-          </visual>
-        </link>
+      <link name="${prefix}_vlp16_plate">
+        <visual>
+          <geometry>
+            <box size="0.1 0.1 0.002" />
+          </geometry>
+          <material name="black" />
+          <origin xyz="0 0 -0.001" rpy="0 0 0" />
+        </visual>
+      </link>
       <link name="${prefix}_vlp16_leg1">
         <visual>

Commit message: Removed indentation

File: jackal_description/urdf/accessories/vlp16_mount.urdf.xacro (robot description, xacro)
@@ -4,13 +4,13 @@
     <xacro:if value="${tower}">
       <link name="${prefix}_vlp16_mount" />
-      <link name="${prefix}_vlp16_plate">
-        <visual>
-          <geometry>
-            <box size="0.1 0.1 0.002" />
-          </geometry>
-          <material name="black" />
-          <origin xyz="0 0 -0.001" rpy="0 0 0" />
-        </visual>
-      </link>
+<link name="${prefix}_vlp16_plate">
+<visual>
+<geometry>
+<box size="0.1 0.1 0.002" />
+</geometry>
+<material name="black" />
+<origin xyz="0 0 -0.001" rpy="0 0 0" />
+</visual>
+</link>
       <link name="${prefix}_vlp16_leg1">
         <visual>

Commit message: Restored indentation

File: jackal_description/urdf/accessories/vlp16_mount.urdf.xacro (robot description, xacro)
@@ -4,13 +4,13 @@
     <xacro:if value="${tower}">
       <link name="${prefix}_vlp16_mount" />
-<link name="${prefix}_vlp16_plate">
-<visual>
-<geometry>
-<box size="0.1 0.1 0.002" />
-</geometry>
-<material name="black" />
-<origin xyz="0 0 -0.001" rpy="0 0 0" />
-</visual>
-</link>
+      <link name="${prefix}_vlp16_plate">
+        <visual>
+          <geometry>
+            <box size="0.1 0.1 0.002" />
+          </geometry>
+          <material name="black" />
+          <origin xyz="0 0 -0.001" rpy="0 0 0" />
+        </visual>
+      </link>
       <link name="${prefix}_vlp16_leg1">
         <visual>

Commit message: Update vlp16_mount.urdf.xacro

File: jackal_description/urdf/accessories/vlp16_mount.urdf.xacro (robot description, xacro)
@@ -4,13 +4,13 @@
     <xacro:if value="${tower}">
       <link name="${prefix}_vlp16_mount" />
-      <link name="${prefix}_vlp16_plate">
-        <visual>
-          <geometry>
-            <box size="0.1 0.1 0.002" />
-          </geometry>
-          <material name="black" />
-          <origin xyz="0 0 -0.001" rpy="0 0 0" />
-        </visual>
-      </link>
+    <link name="${prefix}_vlp16_plate">
+      <visual>
+        <geometry>
+          <box size="0.1 0.1 0.002" />
+        </geometry>
+        <material name="black" />
+        <origin xyz="0 0 -0.001" rpy="0 0 0" />
+      </visual>
+    </link>
       <link name="${prefix}_vlp16_leg1">
         <visual>

Commit message: Update vlp16_mount.urdf.xacro

File: jackal_description/urdf/accessories/vlp16_mount.urdf.xacro (robot description, xacro)
@@ -4,13 +4,13 @@
     <xacro:if value="${tower}">
       <link name="${prefix}_vlp16_mount" />
-    <link name="${prefix}_vlp16_plate">
-      <visual>
-        <geometry>
-          <box size="0.1 0.1 0.002" />
-        </geometry>
-        <material name="black" />
-        <origin xyz="0 0 -0.001" rpy="0 0 0" />
-      </visual>
-    </link>
+        <link name="${prefix}_vlp16_plate">
+          <visual>
+            <geometry>
+              <box size="0.1 0.1 0.002" />
+            </geometry>
+            <material name="black" />
+            <origin xyz="0 0 -0.001" rpy="0 0 0" />
+          </visual>
+        </link>
       <link name="${prefix}_vlp16_leg1">
         <visual>

Commit message: Update vlp16_mount.urdf.xacro

File: jackal_description/urdf/accessories/vlp16_mount.urdf.xacro (robot description, xacro)
@@ -4,13 +4,4 @@
     <xacro:if value="${tower}">
       <link name="${prefix}_vlp16_mount" />
-      <link name="${prefix}_vlp16_plate">
-        <visual>
-          <geometry>
-            <box size="0.1 0.1 0.002" />
-          </geometry>
-          <material name="black" />
-          <origin xyz="0 0 -0.001" rpy="0 0 0" />
-        </visual>
-      </link>
       <link name="${prefix}_vlp16_leg1">
         <visual>

Commit message: Update vlp16_mount.urdf.xacro

File: jackal_description/urdf/accessories/vlp16_mount.urdf.xacro (robot description, xacro)
@@ -4,4 +4,13 @@
     <xacro:if value="${tower}">
       <link name="${prefix}_vlp16_mount" />
+      <link name="${prefix}_vlp16_plate">
+        <visual>
+          <geometry>
+            <box size="0.1 0.1 0.002" />
+          </geometry>
+          <material name="black" />
+          <origin xyz="0 0 -0.001" rpy="0 0 0" />
+        </visual>
+      </link>
       <link name="${prefix}_vlp16_leg1">
         <visual>

Commit message: VLP-16 Functional

File: jackal_description/urdf/accessories/vlp16_mount.urdf.xacro (robot description, xacro)
@@ -1,5 +1,5 @@
 <robot xmlns:xacro="http://wiki.ros.org/xacro">
   <xacro:include filename="$(find velodyne_description)/urdf/VLP-16.urdf.xacro" />
-  <xacro:macro name="vlp16_mount" params="prefix parent_link topic height:=0.1 *origin">
+  <xacro:macro name="vlp16_mount" params="prefix parent_link topic tower height:=0.1 *origin">
     <link name="${prefix}_vlp16_mount" />
     <link name="${prefix}_vlp16_plate">
@@ -86,5 +86,5 @@
       <origin xyz="0 0 ${height}" rpy="0 0 0" />
     </joint>
-    <xacro:VLP-16 parent="${prefix}_vlp16_plate" topic="${topic}">
+    <xacro:VLP-16 parent="${prefix}_vlp16_plate" name="velodyne" topic="/velodyne_points" organize_cloud="false" hz="10" samples="440" gpu="false">
       <origin xyz="0 0 0" rpy="0 0 0" />
     </xacro:VLP-16>
