Commit message: Added switches to enable the new accessory fender, and switches to attach ust10 lasers to those fenders.  Also added ark enclosure with its own variable

File: jackal_description/urdf/jackal.urdf.xacro (robot description, xacro)
@@ -105,16 +105,65 @@
       </inertial>
   </link>
-  <link name="fenders_link">
-    <visual>
-      <origin xyz="0 0 ${footprint_vertical_offset}" rpy="${PI/2} 0 ${PI/2}"/>
-      <geometry>
-        <mesh filename="package://jackal_description/meshes/jackal-fenders.stl"/>
-      </geometry>
-      <material name="yellow" />
-    </visual>
-  </link>
-  <joint name="fenders_joint" type="fixed">
-    <parent link="chassis_link" />
-    <child link="fenders_link" />
+  <xacro:unless value="$(optenv JACKAL_FRONT_ACCESSORY_FENDER 0)">
+    <link name="front_fender_link">
+      <visual>
+        <geometry>
+          <mesh filename="package://jackal_description/meshes/jackal-fender.stl"/>
+        </geometry>
+        <material name="yellow" />
+      </visual>
+    </link>
+  </xacro:unless>
+  <xacro:if value="$(optenv JACKAL_FRONT_ACCESSORY_FENDER 0)">
+    <link name="front_fender_link">
+      <visual>
+        <geometry>
+          <mesh filename="package://jackal_description/meshes/accessory_fender.stl"/>
+        </geometry>
+        <material name="yellow" />
+      </visual>
+    </link>
+    <link name="front_fender_accessory_link"/>
+    <joint name="front_fender_accessory_joint" type="fixed">
+      <origin xyz="0.25629 0 0.07455" rpy="${PI} 0 0" />
+      <parent link="front_fender_link" />
+      <child link="front_fender_accessory_link" />
+    </joint>
+  </xacro:if>
+  <joint name="front_fender_joint" type="fixed">
+    <origin xyz="0 0 0" rpy="0 0 0"/>
+    <parent link="chassis_link" />
+    <child link="front_fender_link" />
+  </joint>
+  <xacro:unless value="$(optenv JACKAL_REAR_ACCESSORY_FENDER 0)">
+    <link name="rear_fender_link">
+      <visual>
+        <geometry>
+          <mesh filename="package://jackal_description/meshes/jackal-fender.stl"/>
+        </geometry>
+        <material name="yellow" />
+      </visual>
+    </link>
+  </xacro:unless>
+  <xacro:if value="$(optenv JACKAL_REAR_ACCESSORY_FENDER 0)">
+    <link name="rear_fender_link">
+      <visual>
+        <geometry>
+          <mesh filename="package://jackal_description/meshes/accessory_fender.stl"/>
+        </geometry>
+        <material name="yellow" />
+      </visual>
+    </link>
+    <link name="rear_fender_accessory_link"/>
+    <joint name="rear_fender_accessory_joint" type="fixed">
+      <origin xyz="0.25629 0 0.07455" rpy="${PI} 0 0" />
+      <parent link="rear_fender_link" />
+      <child link="rear_fender_accessory_link" />
+    </joint>
+  </xacro:if>
+  <joint name="rear_fender_joint" type="fixed">
+    <origin xyz="0 0 0" rpy="0 0 ${PI}"/>
+    <parent link="chassis_link" />
+    <child link="rear_fender_link" />
   </joint>
   <!-- TODO: Make this internal_imu_link or something, and use a mixed-in xacro

Commit message: Add an alternate EKF file that uses the secondary IMU.  Add the GX5 link to the URDF if necessary. Standard mounting location TBD, so don't merge this yet.

File: jackal_description/urdf/jackal.urdf.xacro (robot description, xacro)
@@ -203,4 +203,16 @@
     <origin xyz="-0.180 0.126 0.1815" />
   </joint>
+  <!--
+    Optionally add a GX5 IMU
+  -->
+  <xacro:if value="$(optenv JACKAL_GX5_IMU 0)">
+    <link name="gx5_link" />
+    <joint name="gx5_joint">
+      <parent link="base_link" />
+      <child link="gx5_link" />
+      <!-- TODO fill in the sane defaults. See RSCI-10 -->
+      <origin xyz="$(optenv JACKAL_GX5_IMU_OFFSET 0 0 0)" rpy="$(optenv JACKAL_GX5_IMU_RPY 0 0 0)" />
+    </joint>
+  </xacro:if>
   <link name="mid_mount"></link>
   <joint name="mid_mount_joint" type="fixed">

Commit message: Add a sane default we can use for mounting the GX5.  RSCI-10 is low-priority, so we may not finalize the default position. But this way Integration can at least start using the envars and ensure they set the xyz/rpy offsets correctly.

File: jackal_description/urdf/jackal.urdf.xacro (robot description, xacro)
@@ -208,9 +208,9 @@
   <xacro:if value="$(optenv JACKAL_GX5_IMU 0)">
     <link name="gx5_link" />
-    <joint name="gx5_joint">
+    <joint name="gx5_joint" type="fixed">
       <parent link="base_link" />
       <child link="gx5_link" />
-      <!-- TODO fill in the sane defaults. See RSCI-10 -->
-      <origin xyz="$(optenv JACKAL_GX5_IMU_OFFSET 0 0 0)" rpy="$(optenv JACKAL_GX5_IMU_RPY 0 0 0)" />
+      <!-- TODO This offset & rotation may not be final, but it's good enough for now.  May update, pending RSCI-10 -->
+      <origin xyz="$(optenv JACKAL_GX5_IMU_OFFSET -0.139 0.096 0.100)" rpy="$(optenv JACKAL_GX5_IMU_RPY ${PI} 0 -${PI/2})" />
     </joint>
   </xacro:if>

Commit message: Added environment variable to set parent link of the GX5

File: jackal_description/urdf/jackal.urdf.xacro (robot description, xacro)
@@ -209,5 +209,5 @@
     <link name="gx5_link" />
     <joint name="gx5_joint" type="fixed">
-      <parent link="base_link" />
+      <parent link="$(optenv JACKAL_GX5_IMU_PARENT base_link)" />
       <child link="gx5_link" />
       <!-- TODO This offset & rotation may not be final, but it's good enough for now.  May update, pending RSCI-10 -->
