Commit message: Integration WIP

File: jackal_description/urdf/accessories.urdf.xacro (robot description, xacro)
@@ -13,5 +13,6 @@
     <xacro:sick_lms100 prefix="front" />
     <joint name="front_laser_joint" type="fixed">
-      <origin xyz="0.04 0 0.04" rpy="${PI} 0 0" />
+      <!-- RYANDEBUG      <origin xyz="0.04 0 0.04" rpy="${PI} 0 0" /> -->
+      <origin xyz="0.04 0 0.04" rpy="0 0 0" />
       <parent link="front_mount" />
       <child link="front_laser" />

Commit message: mike's overal mods

File: jackal_description/urdf/accessories.urdf.xacro (robot description, xacro)
@@ -20,7 +20,16 @@
     </joint>
   </xacro:if>
-  <xacro:if value="$(optenv JACKAL_LASER 0)">
-	 <xacro:include filename="accessories/basic-smart6.urdf.xacro" />
-         <xacro:include filename="accessories/jackal-standard-bridge-plate.urdf.xacro" />
+  <xacro:include filename="accessories/novatel_smart6.urdf.xacro" />
+  <xacro:include filename="accessories/bridge_plate.urdf.xacro" />
+  <xacro:if value="$(optenv JACKAL_NAVSAT 0)">
+    <bridge_plate mount="$(optenv JACKAL_NAVSAT_MOUNT rear)"
+                  height="$(optenv JACKAL_NAVSAT_HEIGHT 0.12)" />
+    <novatel_smart6 prefix="$(optenv JACKAL_NAVSAT_MOUNT rear)"/>
+    <joint name="$(optenv JACKAL_NAVSAT_MOUNT rear)_navsat_joint" type="fixed">
+      <origin xyz="0 0 0"
+              rpy="0 0 0" />
+      <parent link="$(optenv JACKAL_NAVSAT_MOUNT rear)_bridge" />
+      <child link="$(optenv JACKAL_NAVSAT_MOUNT rear)_navsat" />
+    </joint>
   </xacro:if>
   <!--

Commit message: added correct mount plate and fixed orientation

File: jackal_description/urdf/accessories.urdf.xacro (robot description, xacro)
@@ -28,5 +28,5 @@
     <joint name="$(optenv JACKAL_NAVSAT_MOUNT rear)_navsat_joint" type="fixed">
       <origin xyz="0 0 0"
-              rpy="0 0 0" />
+              rpy="0 1.57070 1.5707" />
       <parent link="$(optenv JACKAL_NAVSAT_MOUNT rear)_bridge" />
       <child link="$(optenv JACKAL_NAVSAT_MOUNT rear)_navsat" />

File: jackal_description/urdf/accessories/bridge_plate.urdf.xacro (robot description, xacro)
@@ -6,5 +6,5 @@
 		<child link="${mount}_bridge"/>
 		<!-- <origin xyz="0.1016 0.0 0.1143" rpy="0.0 0.0 0.0"/> -->
-		<origin xyz="0.0 0.0 ${height}" rpy="0.0 0.0 0.0"/>
+		<origin xyz="0.0 0.0 ${height}" rpy="1.5707 0.0 1.5707"/>
 	</joint>
 	<link name="${mount}_bridge">

Commit message: Rename meshes, add standoff macro.

File: jackal_description/urdf/accessories.urdf.xacro (robot description, xacro)
@@ -9,4 +9,34 @@
     jackal_base/launch/base.launch
   -->
+  <xacro:macro name="standoff" params="name length parent *origin">
+    <link name="${name}">
+      <visual>
+        <origin xyz="0 0 ${length/2}" rpy="0 0 0" />
+        <geometry>
+          <cylinder radius="0.004" length="${length}" />
+        </geometry>
+        <material name="light_grey" />
+      </visual>
+    </link>
+    <joint name="${name}_joint" type="fixed">
+      <xacro:insert_block name="origin" />
+      <parent link="${parent}" />
+      <child link="${name}" />
+    </joint>
+  </xacro:macro>
+  <xacro:macro name="standoff_box" params="mount height">
+    <standoff name="${mount}_standoff0" length="${height}" parent="${mount}_mount">
+      <origin xyz="0.060 0.060 0" rpy="0 0 0"/>
+    </standoff>
+    <standoff name="${mount}_standoff1" length="${height}" parent="${mount}_mount">
+      <origin xyz="0.060 -0.060 0" rpy="0 0 0"/>
+    </standoff>
+    <standoff name="${mount}_standoff2" length="${height}" parent="${mount}_mount">
+      <origin xyz="-0.060 0.060 0" rpy="0 0 0"/>
+    </standoff>
+    <standoff name="${mount}_standoff3" length="${height}" parent="${mount}_mount">
+      <origin xyz="-0.060 -0.060 0" rpy="0 0 0"/>
+    </standoff>
+  </xacro:macro>
   <xacro:include filename="accessories/sick_lms1xx.urdf.xacro" />
   <xacro:if value="$(optenv JACKAL_LASER 0)">
@@ -27,6 +57,5 @@
     <novatel_smart6 prefix="$(optenv JACKAL_NAVSAT_MOUNT rear)"/>
     <joint name="$(optenv JACKAL_NAVSAT_MOUNT rear)_navsat_joint" type="fixed">
-      <origin xyz="0 0 0"
-              rpy="0 1.57070 1.5707" />
+      <origin xyz="0 0 0" rpy="0 0 0" />
       <parent link="$(optenv JACKAL_NAVSAT_MOUNT rear)_bridge" />
       <child link="$(optenv JACKAL_NAVSAT_MOUNT rear)_navsat" />

File: jackal_description/urdf/accessories/bridge_plate.urdf.xacro (robot description, xacro)
@@ -2,18 +2,19 @@
 <robot xmlns:xacro="http://ros.org/wiki/xacro">
   <xacro:macro name="bridge_plate" params="mount height">
-	<joint name="${mount}_mount_to_${mount}_bridge" type="fixed">
-		<parent link="${mount}_mount"/>
-		<child link="${mount}_bridge"/>
-		<!-- <origin xyz="0.1016 0.0 0.1143" rpy="0.0 0.0 0.0"/> -->
-		<origin xyz="0.0 0.0 ${height}" rpy="1.5707 0.0 1.5707"/>
-	</joint>
-	<link name="${mount}_bridge">
-		<visual>
-			<geometry>
-				<mesh filename="package://jackal_description/meshes/jackal-standard-bridge-plate.STL"/>
-			</geometry>
-			<material name="dark_grey" />
-		</visual>
-	</link>
+    <joint name="${mount}_mount_to_${mount}_bridge" type="fixed">
+      <parent link="${mount}_mount"/>
+      <child link="${mount}_bridge"/>
+      <origin xyz="0.0 0.0 ${height}" rpy="0 0 0"/>
+    </joint>
+    <link name="${mount}_bridge">
+      <visual>
+        <origin xyz="0 0 0" rpy="1.5707 0.0 1.5707" />
+        <geometry>
+          <mesh filename="package://jackal_description/meshes/bridge-plate.stl"/>
+        </geometry>
+        <material name="dark_grey" />
+      </visual>
+    </link>
+    <standoff_box mount="${mount}" height="${height}" />
   </xacro:macro>
 </robot>

File: jackal_description/urdf/accessories/novatel_smart6.urdf.xacro (robot description, xacro)
@@ -2,14 +2,15 @@
 <robot xmlns:xacro="http://ros.org/wiki/xacro">
   <xacro:macro name="novatel_smart6" params="prefix">
-	<link name="${prefix}_navsat">
-		<visual>
-			<geometry>
-				<mesh filename="package://jackal_description/meshes/basic-smart6.STL"/>
-			</geometry>
-			<material name="white">
-				<color rgba="255 255 255 .9"/>
-			</material>
-		</visual>
-	</link>
+  <link name="${prefix}_navsat">
+    <visual>
+      <origin xyz="0 0 0" rpy="0 0 0" />
+      <geometry>
+        <mesh filename="package://jackal_description/meshes/novatel-smart6.stl"/>
+      </geometry>
+      <material name="white">
+        <color rgba="255 255 255 .9"/>
+      </material>
+    </visual>
+  </link>
   </xacro:macro>
 </robot>

Commit message: Added Sick LMS1XX URDF.

File: jackal_description/urdf/accessories.urdf.xacro (robot description, xacro)
@@ -14,5 +14,5 @@
   <xacro:include filename="accessories/bridge_plate.urdf.xacro" />
   <!-- If enabled, generate the LASER payload (by default, a SICK LMS111). -->
-  <xacro:include filename="accessories/sick_lms1xx.urdf.xacro" />
+  <xacro:include filename="accessories/sick_lms1xx_mount.urdf.xacro" />
   <xacro:if value="$(optenv JACKAL_LASER 0)">
     <sick_lms1xx_mount prefix="$(optenv JACKAL_LASER_MOUNT front)"

File: jackal_description/urdf/accessories/sick_lms1xx_mount.urdf.xacro (robot description, xacro)
@@ -26,18 +26,7 @@
 -->
 <robot xmlns:xacro="http://ros.org/wiki/xacro">
-  <xacro:property name="laser_x" value="0.105" />
-  <xacro:property name="laser_y" value="0.102" />
-  <xacro:property name="laser_z" value="0.152" />
-  <xacro:property name="laser_mass" value="1.1" />
-  <xacro:macro name="box_inertial" params="x y z mass">
-    <inertial>
-      <mass value="${mass}" />
-      <origin xyz="0 0 0" />
-      <inertia ixx="${0.0833333 * mass * (y*y + z*z)}" ixy="0.0" ixz="0.0"
-        iyy="${0.0833333 * mass * (x*x + z*z)}" iyz="0.0"
-        izz="${0.0833333 * mass * (x*x + y*y)}" />
-    </inertial>
-  </xacro:macro>
+  <xacro:include filename="$(find lms1xx)/urdf/sick_lms1xx.urdf.xacro" />
   <xacro:macro name="sick_lms1xx_mount" params="prefix topic">
+    <sick_lms1xx prefix="${prefix}" topic="${topic}" />
     <link name="${prefix}_laser_mount">
       <visual>
@@ -50,21 +39,4 @@
       </visual>
     </link>
-    <link name="${prefix}_laser">
-      <xacro:box_inertial x="${laser_x}" y="${laser_y}" z="${laser_z}" mass="${laser_mass}" />
-      <visual>
-        <origin xyz="0 0 0" rpy="0 0 0" />
-        <geometry>
-          <!-- Origin of this mesh is the focal point of the LIDAR. -->
-          <mesh filename="package://jackal_description/meshes/sick-lms1xx.stl" />
-        </geometry>
-        <material name="light_grey" />
-      </visual>
-      <collision>
-        <origin xyz="0 0 -0.05" rpy="0 0 0" />
-        <geometry>
-          <box size="${laser_x} ${laser_y} ${laser_z}" />
-        </geometry>
-      </collision>
-    </link>
     <joint name="${prefix}_laser_joint" type="fixed">
       <!-- This offset is from the base of the bracket to the LIDAR's focal point. -->
@@ -73,37 +45,4 @@
       <child link="${prefix}_laser" />
     </joint>
-    <gazebo reference="${prefix}_laser">
-      <material>Gazebo/Grey</material>
-      <turnGravityOff>true</turnGravityOff>
-      <sensor type="ray" name="${prefix}_laser">
-        <pose>0 0 0 0 0 0</pose>
-        <visualize>false</visualize>
-        <update_rate>40</update_rate>
-        <ray>
-          <scan>
-            <horizontal>
-              <samples>720</samples>
-              <resolution>1</resolution>
-              <min_angle>-1.570796</min_angle>
-              <max_angle>1.570796</max_angle>
-            </horizontal>
-          </scan>
-          <range>
-            <min>0.10</min>
-            <max>30.0</max>
-            <resolution>0.01</resolution>
-          </range>
-          <noise>
-            <type>gaussian</type>
-            <mean>0.0</mean>
-            <stddev>0.001</stddev>
-          </noise>
-        </ray>
-        <plugin name="gazebo_ros_laser" filename="libgazebo_ros_laser.so">
-          <topicName>${topic}</topicName>
-          <frameName>${prefix}_laser</frameName>
-        </plugin>
-      </sensor>
-    </gazebo>
   </xacro:macro>
 </robot>

Commit message: Updated for changes in lms1xx urdf macro.

File: jackal_description/urdf/accessories.urdf.xacro (robot description, xacro)
@@ -17,5 +17,5 @@
   <xacro:if value="$(optenv JACKAL_LASER 0)">
     <sick_lms1xx_mount prefix="$(optenv JACKAL_LASER_MOUNT front)"
-                       topic="$(optenv JACKAL_LASER_TOPIC scan)" />
+                       topic="$(optenv JACKAL_LASER_TOPIC scan)"/>
     <joint name="$front_laser_mount_joint" type="fixed">
       <origin xyz="$(optenv JACKAL_LASER_OFFSET 0 0 0)"

File: jackal_description/urdf/accessories/sick_lms1xx_mount.urdf.xacro (robot description, xacro)
@@ -28,5 +28,5 @@
   <xacro:include filename="$(find lms1xx)/urdf/sick_lms1xx.urdf.xacro" />
   <xacro:macro name="sick_lms1xx_mount" params="prefix topic">
-    <sick_lms1xx prefix="${prefix}" topic="${topic}" />
+    <sick_lms1xx frame="${prefix}_laser" topic="${topic}" />
     <link name="${prefix}_laser_mount">
       <visual>
@@ -43,5 +43,5 @@
       <origin xyz="0 0 0.149" rpy="0 0 0" />
       <parent link="${prefix}_laser_mount" />
-      <child link="${prefix}laser" />
+      <child link="${prefix}_laser" />
     </joint>
   </xacro:macro>

Commit message: Add support for adding an Azure Kinect to the model with new environment variables, add the (very boxy) model for the Azure Kinect itself (largely copied from MS' driver for the same, but turned into a macro)

File: jackal_description/urdf/accessories.urdf.xacro (robot description, xacro)
@@ -147,3 +147,30 @@
     </gazebo>
   </xacro:if>
+  <xacro:if value="$(optenv JACKAL_AZURE_KINECT 0)">
+    <!--
+      Microsoft kindly provided a 3d printable mounting plate for the Azure Kinect
+      To make printing easier the model's origin is offset a bit and it's in mm,
+      so we need to scale and offset the model a little.
+    -->
+    <link name="$(optenv JACKAL_AZURE_KINECT_MOUNT front)_kinect_mount_plate">
+      <visual>
+        <origin xyz="0 0 -0.055" rpy="0 0 -1.57079632675" />
+        <geometry>
+          <mesh filename="package://jackal_description/meshes/kinect_mount.stl" scale="0.001 0.001 0.001"/>
+        </geometry>
+        <material name="black"/>
+      </visual>
+    </link>
+    <joint name="$(optenv JACKAL_AZURE_KINECT_MOUNT front)_kinect_mount_joint" type="fixed">
+      <parent link="$(optenv JACKAL_AZURE_KINECT_MOUNT front)_mount"/>
+      <child link="$(optenv JACKAL_AZURE_KINECT_MOUNT front)_kinect_mount_plate"/>
+    </joint>
+    <xacro:include filename="$(find jackal_description)/urdf/accessories/azure_kinect.urdf.xacro" />
+    <xacro:azure_kinect prefix="$(optenv JACKAL_AZURE_KINECT_MOUNT front)" />
+    <joint name="$(optenv JACKAL_AZURE_KINECT_MOUNT front)_kinect_mount_point" type="fixed">
+      <origin xyz="0.09 0 0.0335" rpy="0 -0.17453292519444444 0"/>
+      <parent link="$(optenv JACKAL_AZURE_KINECT_MOUNT front)_kinect_mount_plate"/>
+      <child link="$(optenv JACKAL_AZURE_KINECT_MOUNT front)camera_base"/>
+    </joint>
+  </xacro:if>
 </robot>

File: jackal_description/urdf/jackal.urdf.xacro (robot description, xacro)
@@ -14,7 +14,9 @@
   <xacro:property name="mount_spacing" value="0.120" />
   <material name="dark_grey"><color rgba="0.2 0.2 0.2 1.0" /></material>
-  <material name="light_grey"><color rgba="0.4 0.4 0.4 1.0" /></material>
+  <material name="medium_grey"><color rgba="0.6 0.6 0.6 1.0" /></material>
+  <material name="light_grey"><color rgba="0.8 0.8 0.8 1.0" /></material>
   <material name="yellow"><color rgba="0.8 0.8 0.0 1.0" /></material>
   <material name="black"><color rgba="0.15 0.15 0.15 1.0" /></material>
+  <material name="white"><color rgba="1.0 1.0 1.0 1.0" /></material>
   <xacro:macro name="wheel" params="prefix *joint_pose">
     <link name="${prefix}_wheel_link">

Commit message: Rename the base/body/visor links & joints in the Kinect's URDF to reduce ambiguity. Add support for getting the camera data in Gazebo using the OpenNI kinect plugin. It's not 100% accurate, but it's a reasonable analogue for now.

File: jackal_description/urdf/accessories.urdf.xacro (robot description, xacro)
@@ -171,5 +171,5 @@
       <origin xyz="0.09 0 0.0335" rpy="0 -0.17453292519444444 0"/>
       <parent link="$(optenv JACKAL_AZURE_KINECT_MOUNT front)_kinect_mount_plate"/>
-      <child link="$(optenv JACKAL_AZURE_KINECT_MOUNT front)camera_base"/>
+      <child link="$(optenv JACKAL_AZURE_KINECT_MOUNT front)_kinect_base"/>
     </joint>
   </xacro:if>

File: jackal_description/urdf/accessories/azure_kinect.urdf.xacro (robot description, xacro)
@@ -22,5 +22,5 @@
 <robot xmlns:xacro="http://www.ros.org/wiki/xacro">
   <xacro:macro name="azure_kinect" params="prefix">
-    <link name="${prefix}camera_body">
+    <link name="${prefix}_kinect_body">
       <visual>
         <origin xyz="0. 0. 0." />
@@ -31,5 +31,5 @@
       </visual>
     </link>
-    <link name="${prefix}camera_base">
+    <link name="${prefix}_kinect_base">
       <visual>
         <origin xyz="-0.013 0. 0." />
@@ -40,5 +40,5 @@
       </visual>
     </link>
-    <link name="${prefix}camera_visor">
+    <link name="${prefix}_kinect_visor">
       <visual>
         <origin xyz="-0.0128 0. 0." />
@@ -49,14 +49,80 @@
       </visual>
     </link>
-    <joint name="${prefix}camera_base_to_body" type="fixed">
-      <parent link="${prefix}camera_base" />
-      <child link="${prefix}camera_body" />
+    <joint name="${prefix}_kinect_base_to_body" type="fixed">
+      <parent link="${prefix}_kinect_base" />
+      <child link="${prefix}_kinect_body" />
       <origin xyz="-0.0757 0. 0.008" rpy="0. 0. 0." />
     </joint>
-    <joint name="${prefix}camera_base_to_visor" type="fixed">
-      <parent link="${prefix}camera_base" />
-      <child link="${prefix}camera_visor" />
+    <joint name="${prefix}_kinect_base_to_visor" type="fixed">
+      <parent link="${prefix}_kinect_base" />
+      <child link="${prefix}_kinect_visor" />
       <origin xyz="0. 0. 0." rpy="0. 0. 0." />
     </joint>
+    <!--
+      The gazebo plugin aligns the depth data with the Z axis, with X=left and Y=up
+      ROS expects the depth data along the X axis, with Y=left and Z=up
+      This link only exists to give the gazebo plugin the correctly-oriented frame
+    -->
+    <link name="${prefix}_kinect_gazebo_lens" />
+    <joint name="${prefix}_kinect_gazebo_joint" type="fixed">
+      <parent link="${prefix}_kinect_visor"/>
+      <child link="${prefix}_kinect_gazebo_lens"/>
+      <origin xyz="0 0 0" rpy="-1.5707963267948966 0 -1.5707963267948966"/>
+    </joint>
+    <!--
+      This isn't a 100% accurate representation of the Azure Kinect's data, but it's reasonably close.
+      The color data on the real camera has a 90x59 degree FOV, and the depth data is the full vision
+      cone approximated as a hexagon within the frame.
+      But for now the OpenNI kinect plugin is the closest analogue
+    -->
+    <gazebo reference="${prefix}_kinect_visor">
+      <turnGravityOff>true</turnGravityOff>
+      <sensor type="depth" name="${prefix}_kinect_depth">
+        <update_rate>30</update_rate>
+        <camera>
+          <!-- 75x65 degree FOV -->
+          <horizontal_fov>1.3089958333333334</horizontal_fov>
+          <vertical_fov>1.1344630555555555</vertical_fov>
+          <image>
+            <!--
+              The Azure Kinect has a bit of a weird frame size for the depth data
+              see: https://docs.microsoft.com/en-us/azure/kinect-dk/hardware-specification
+            -->
+            <width>640</width>
+            <height>576</height>
+            <!-- TODO: check what format the Azure Kinect hardware delivers and set this to match! -->
+            <format>R8G8B8</format>
+          </image>
+          <clip>
+            <near>0.5</near>
+            <far>5.46</far>
+          </clip>
+        </camera>
+        <plugin name="kinect_controller" filename="libgazebo_ros_openni_kinect.so">
+          <baseline>0.2</baseline>
+          <alwaysOn>true</alwaysOn>
+          <updateRate>1.0</updateRate>
+          <cameraName>kinect</cameraName>
+          <imageTopicName>/kinect/color/image_raw</imageTopicName>
+          <cameraInfoTopicName>/kinect/color/camera_info</cameraInfoTopicName>
+          <depthImageTopicName>/kinect/depth/image_raw</depthImageTopicName>
+          <depthImageInfoTopicName>/kinect/depth/camera_info</depthImageInfoTopicName>
+          <pointCloudTopicName>/kinect/depth/points</pointCloudTopicName>
+          <frameName>${prefix}_kinect_gazebo_lens</frameName>
+          <pointCloudCutoff>0.5</pointCloudCutoff>
+          <pointCloudCutoffMax>3.0</pointCloudCutoffMax>
+          <distortionK1>0.00000001</distortionK1>
+          <distortionK2>0.00000001</distortionK2>
+          <distortionK3>0.00000001</distortionK3>
+          <distortionT1>0.00000001</distortionT1>
+          <distortionT2>0.00000001</distortionT2>
+          <CxPrime>0</CxPrime>
+          <Cx>0</Cx>
+          <Cy>0</Cy>
+          <focalLength>0</focalLength>
+          <hackBaseline>0</hackBaseline>
+        </plugin>
+      </sensor>
+    </gazebo>
   </xacro:macro>
 </robot>

Commit message: Rescale & rotate the kinect mount so it's in meters w/ the correct edge forward; this eliminates the need to manually scale & rotate the mount in the URDF.  Add support for 2 new environment vars: JACKAL_AZURE_KINECT_OFFSET and _RPY

File: jackal_description/urdf/accessories.urdf.xacro (robot description, xacro)
@@ -148,14 +148,9 @@
   </xacro:if>
   <xacro:if value="$(optenv JACKAL_AZURE_KINECT 0)">
-    <!--
-      Microsoft kindly provided a 3d printable mounting plate for the Azure Kinect
-      To make printing easier the model's origin is offset a bit and it's in mm,
-      so we need to scale and offset the model a little.
-    -->
     <link name="$(optenv JACKAL_AZURE_KINECT_MOUNT front)_kinect_mount_plate">
       <visual>
-        <origin xyz="0 0 -0.055" rpy="0 0 -1.57079632675" />
+        <origin xyz="0 0 0" rpy="0 0 0" />
         <geometry>
-          <mesh filename="package://jackal_description/meshes/kinect_mount.stl" scale="0.001 0.001 0.001"/>
+          <mesh filename="package://jackal_description/meshes/kinect_mount.stl"/>
         </geometry>
         <material name="black"/>
@@ -163,4 +158,5 @@
     </link>
     <joint name="$(optenv JACKAL_AZURE_KINECT_MOUNT front)_kinect_mount_joint" type="fixed">
+      <origin xyz="$(optenv JACKAL_AZURE_KINECT_OFFSET 0 0 0)" rpy="$(optenv JACKAL_AZURE_KINECT_RPY 0 0 0)"/>
       <parent link="$(optenv JACKAL_AZURE_KINECT_MOUNT front)_mount"/>
       <child link="$(optenv JACKAL_AZURE_KINECT_MOUNT front)_kinect_mount_plate"/>

Commit message: Add support for the slamtec A1/2, as that's the lidar we're currently using in our Windows testing

File: jackal_description/urdf/accessories.urdf.xacro (robot description, xacro)
@@ -14,4 +14,10 @@
   <xacro:include filename="$(find jackal_description)/urdf/accessories/bridge_plate.urdf.xacro" />
   <!-- If enabled, generate the LASER payload (by default, a SICK LMS111). -->
+  <!--
+    We support 3 different lidar accessories out of the box:
+      - sick lms1xx (default) if JACKAL_LASER=1
+      - hokuyo ust10 if JACKAL_LASER=1 && JACKAL_LASER_HOKUYO=1
+      - slamtec a1/2 if JACKAL_LASER=1 && JACKAL_LASER_RP=1
+  -->
   <xacro:if value="$(optenv JACKAL_LASER 0)">
     <xacro:if value="$(optenv JACKAL_LASER_HOKUYO 0)">
@@ -22,8 +28,16 @@
     </xacro:if>
     <xacro:unless value="$(optenv JACKAL_LASER_HOKUYO 0)">
-      <xacro:include filename="$(find jackal_description)/urdf/accessories/sick_lms1xx_mount.urdf.xacro" />
-      <xacro:sick_lms1xx_mount prefix="$(optenv JACKAL_LASER_MOUNT front)"
-                         parent_link="$(optenv JACKAL_LASER_MOUNT front)_mount"
-                         topic="$(optenv JACKAL_LASER_TOPIC front/scan)"/>
+      <xacro:if value="$(optenv JACKAL_LASER_RP 0)">
+        <xacro:include filename="$(find jackal_description)/urdf/accessories/rp_lidar.urdf.xacro" />
+        <xacro:rp_lidar_mount prefix="$(optenv JACKAL_LASER_MOUNT front)"
+                            parent_link="$(optenv JACKAL_LASER_MOUNT front)_mount"
+                            topic="$(optenv JACKAL_LASER_TOPIC front/scan)" />
+      </xacro:if>
+      <xacro:unless value="$(optenv JACKAL_LASER_RP 0)">
+        <xacro:include filename="$(find jackal_description)/urdf/accessories/sick_lms1xx_mount.urdf.xacro" />
+        <xacro:sick_lms1xx_mount prefix="$(optenv JACKAL_LASER_MOUNT front)"
+                           parent_link="$(optenv JACKAL_LASER_MOUNT front)_mount"
+                           topic="$(optenv JACKAL_LASER_TOPIC front/scan)"/>
+      </xacro:unless>
     </xacro:unless>
   </xacro:if>

File: jackal_description/urdf/jackal.urdf.xacro (robot description, xacro)
@@ -19,4 +19,5 @@
   <material name="black"><color rgba="0.15 0.15 0.15 1.0" /></material>
   <material name="white"><color rgba="1.0 1.0 1.0 1.0" /></material>
+  <material name="red"><color rgba="1.0 0.0 0.0 1.0" /></material>
   <xacro:macro name="wheel" params="prefix *joint_pose">
     <link name="${prefix}_wheel_link">
