Commit message: Replace our hacky RP A2 made out of cylinders with a CC-licensed STL.  Include the license for the STL.

File: jackal_description/urdf/accessories.urdf.xacro (robot description, xacro)
@@ -29,5 +29,5 @@
     <xacro:unless value="$(optenv JACKAL_LASER_HOKUYO 0)">
       <xacro:if value="$(optenv JACKAL_LASER_RP 0)">
-        <xacro:include filename="$(find jackal_description)/urdf/accessories/rp_lidar.urdf.xacro" />
+        <xacro:include filename="$(find jackal_description)/urdf/accessories/rplidar_a2.urdf.xacro" />
         <xacro:rp_lidar_mount prefix="$(optenv JACKAL_LASER_MOUNT front)"
                             parent_link="$(optenv JACKAL_LASER_MOUNT front)_mount"

File: jackal_description/urdf/accessories/rplidar_a2.urdf.xacro (robot description, xacro)
@@ -45,23 +45,5 @@
         <origin xyz="0 0 0" rpy="0 0 0" />
         <geometry>
-          <cylinder radius="0.04" length="0.04"/>
-        </geometry>
-        <material name="dark_grey" />
-      </visual>
-    </link>
-    <link name="${prefix}_laser_ring">
-      <visual>
-        <origin xyz="0 0 0" rpy="0 0 0" />
-        <geometry>
-          <cylinder radius="0.039" length="0.004"/>
-        </geometry>
-        <material name="red" />
-      </visual>
-    </link>
-    <link name="${prefix}_laser_cap">
-      <visual>
-        <origin xyz="0 0 0" rpy="0 0 0" />
-        <geometry>
-          <cylinder radius="0.038" length="0.036"/>
+          <mesh filename="package://jackal_description/meshes/rplidar_a2.stl" />
         </geometry>
         <material name="dark_grey" />
@@ -74,18 +56,8 @@
       <child link="${prefix}_laser_mount" />
     </joint>
-    <joint name="${prefix}_laser_ring_joint" type="fixed">
-      <origin xyz="0 0 0.02" rpy="0 0 0" />
-      <parent link="${prefix}_laser_mount" />
-      <child link="${prefix}_laser_ring" />
-    </joint>
-    <joint name="${prefix}_laser_cap_joint" type="fixed">
-      <origin xyz="0 0 0.002" rpy="0 0 0" />
-      <parent link="${prefix}_laser_ring" />
-      <child link="${prefix}_laser_cap" />
-    </joint>
     <joint name="${prefix}_laser_joint" type="fixed">
       <!-- This offset is from the base of the bracket to the LIDAR's focal point. -->
-      <origin xyz="0 0 0" rpy="0 0 0" />
-      <parent link="${prefix}_laser_cap" />
+      <origin xyz="0 0 0.029" rpy="0 0 0" />
+      <parent link="${prefix}_laser_mount" />
       <child link="${prefix}_laser" />
     </joint>

Commit message: Add front and rear fender mounts for attaching e.g. RealSense cameras to. Add the initial gazebo plugin for a RealSense camera (topic names not fixed yet). Add a fixed copy of the D415 STL that's oriented correctly. Remove the laserscan plugin from the azure kinect, as we've removed that from the bringup

File: jackal_description/urdf/accessories.urdf.xacro (robot description, xacro)
@@ -185,3 +185,16 @@
     </joint>
   </xacro:if>
+  <xacro:if value="$(optenv JACKAL_REALSENSE 0)">
+    <link name="$(optenv JACKAL_REALSENSE_MOUNT front_fender)_realsense_mount"></link>
+    <joint name="$(optenv JACKAL_REALSNESE_MOUNT front_fender)_realsense_mount_joint" type="fixed">
+      <origin xyz="$(optenv JACKAL_REALSENSE_OFFSET 0 0 0)" rpy="$(optenv JACKAL_REALSENSE_RPY 0 0 0)" />
+      <parent link="$(optenv JACKAL_REALSENSE_MOUNT front_fender)_mount" />
+      <child link="$(optenv JACKAL_REALSENSE_MOUNT front_fender)_realsense_mount" />
+    </joint>
+    <xacro:include filename="$(find jackal_description)/urdf/accessories/intel_realsense.urdf.xacro" />
+    <xacro:intel_realsense_mount
+      prefix="$(optenv JACKAL_REALSENSE_MOUNT front_fender)"
+      topic="$(optenv JACKAL_REALSENSE_TOPIC realsense)"
+      parent_link="$(optenv JACKAL_REALSENSE_MOUNT front_fender)_realsense_mount" />
+  </xacro:if>
 </robot>

File: jackal_description/urdf/accessories/azure_kinect.urdf.xacro (robot description, xacro)
@@ -135,41 +135,4 @@
         </plugin>
       </sensor>
-      <!--
-        to simulate the depthimage_to_laserscan node in the bringup, we also add a laser
-        plugin that publishes to the same topic
-        ideally we would just launch the depthimage_to_laserscan node, but there seems to be a bug
-        in the libgazebo_ros_openni_kinect plugin that's preventing the (required) /depth/camera_data
-        topic from publishing correctly.  so for now we'll fake it with the laser plugin
-      -->
-      <sensor type="ray" name="${prefix}_kinect_scan">
-        <pose>0 0 0 0 0 0</pose>
-        <visualize>false</visualize>
-        <update_rate>${update_rate}</update_rate>
-        <ray>
-          <scan>
-            <horizontal>
-              <samples>${width}</samples>
-              <resolution>1</resolution>
-              <min_angle>${h_fov/-2}</min_angle>
-              <max_angle>${h_fov/2}</max_angle>
-            </horizontal>
-          </scan>
-          <range>
-            <min>${min_range}</min>
-            <max>${max_range}</max>
-            <resolution>0.001</resolution>
-          </range>
-          <noise>
-            <type>gaussian</type>
-            <mean>0.0</mean>
-            <stddev>0.001</stddev>
-          </noise>
-        </ray>
-        <plugin name="gazebo_ros_laser" filename="libgazebo_ros_laser.so">
-          <topicName>/$(optenv JACKAL_AZURE_KINECT_MOUNT front)/scan</topicName>
-          <frameName>${prefix}_kinect_visor</frameName>
-        </plugin>
-      </sensor>
-    </gazebo>
   </xacro:macro>
 </robot>

File: jackal_description/urdf/jackal.urdf.xacro (robot description, xacro)
@@ -224,4 +224,21 @@
     <origin xyz="${mount_spacing} 0 0" />
   </joint>
+  <!--
+    Not official mounting points, but you can anchor light sensors to the front & rear fenders
+    with velcro or drill your own mounting holes
+  -->
+  <link name="front_fender_mount"></link>
+  <joint name="front_fender_mount_joint" type="fixed">
+    <parent link="front_mount" />
+    <child link="front_fender_mount" />
+    <!--<origin xyz="0.115 0 -0.015" rpy="0 -0.7853975 0" />-->
+    <origin xyz="0.115 0 -0.015" rpy="0 -0.7853975 0" />
+   </joint>
+   <link name="rear_fender_mount"></link>
+   <joint name="rear_fender_mount_joint" type="fixed">
+     <parent link="rear_mount" />
+     <child link="rear_fender_mount" />
+     <origin xyz="-0.115 0 -0.015" rpy="0 -0.7853975 -${PI}" />
+    </joint>
   <!-- Bring in simulation data for Gazebo. -->
   <xacro:include filename="$(find jackal_description)/urdf/jackal.gazebo" />

Commit message: Refactor the azure kinect accessory to use the same macro formatting as the realsense.

File: jackal_description/urdf/accessories.urdf.xacro (robot description, xacro)
@@ -162,26 +162,15 @@
   </xacro:if>
   <xacro:if value="$(optenv JACKAL_AZURE_KINECT 0)">
-    <link name="$(optenv JACKAL_AZURE_KINECT_MOUNT front)_kinect_mount_plate">
-      <visual>
-        <origin xyz="0 0 0" rpy="0 0 0" />
-        <geometry>
-          <mesh filename="package://jackal_description/meshes/kinect_mount.stl"/>
-        </geometry>
-        <material name="black"/>
-      </visual>
-    </link>
-    <joint name="$(optenv JACKAL_AZURE_KINECT_MOUNT front)_kinect_mount_joint" type="fixed">
-      <origin xyz="$(optenv JACKAL_AZURE_KINECT_OFFSET 0 0 0)" rpy="$(optenv JACKAL_AZURE_KINECT_RPY 0 0 0)"/>
-      <parent link="$(optenv JACKAL_AZURE_KINECT_MOUNT front)_mount"/>
-      <child link="$(optenv JACKAL_AZURE_KINECT_MOUNT front)_kinect_mount_plate"/>
+    <link name="$(optenv JACKAL_AZURE_KINECT_MOUNT front)_kinect_mount" />
+    <joint name="$(optenv JACKAL_AZURE_KINECT_MOUNT front)_kinect_moint_joint" type="fixed">
+      <parent link="$(optenv JACKAL_AZURE_KINECT_MOUNT front)_mount" />
+      <child link="$(optenv JACKAL_AZURE_KINECT_MOUNT front)_kinect_mount" />
+      <origin xyz="$(optenv JACKAL_AZURE_KINECT_OFFSET 0 0 0)" rpy="$(optenv JACKAL_AZURE_KINECT_RPY 0 0 0)" />
     </joint>
     <xacro:include filename="$(find jackal_description)/urdf/accessories/azure_kinect.urdf.xacro" />
-    <xacro:azure_kinect prefix="$(optenv JACKAL_AZURE_KINECT_MOUNT front)" />
-    <!-- this is the actual mounting hole in the mounting plate -->
-    <joint name="$(optenv JACKAL_AZURE_KINECT_MOUNT front)_kinect_mount_point" type="fixed">
-      <origin xyz="0.09 0 0.0335" rpy="0 -0.17453292519444444 0"/>
-      <parent link="$(optenv JACKAL_AZURE_KINECT_MOUNT front)_kinect_mount_plate"/>
-      <child link="$(optenv JACKAL_AZURE_KINECT_MOUNT front)_kinect_base"/>
-    </joint>
+    <xacro:azure_kinect_mount
+      prefix="$(optenv JACKAL_AZURE_KINECT_MOUNT front)"
+      topic="$(optenv JACKAL_AZURE_KINECT_TOPIC kinect)"
+      parent_link="$(optenv JACKAL_AZURE_KINECT_MOUNT front)_kinect_mount"  />
   </xacro:if>
   <xacro:if value="$(optenv JACKAL_REALSENSE 0)">

File: jackal_description/urdf/accessories/azure_kinect.urdf.xacro (robot description, xacro)
@@ -21,119 +21,146 @@
 -->
 <robot xmlns:xacro="http://www.ros.org/wiki/xacro">
-  <xacro:macro name="azure_kinect" params="prefix min_range:=0.5 max_range:=5.46
-                    update_rate:=30
-                    h_fov:=1.3089958333333334 v_fov:=1.1344630555555555
-                    width:=576 height:=640">
-    <link name="${prefix}_kinect_body">
+  <xacro:macro name="azure_kinect_mount" params="prefix topic parent_link">
+    <xacro:macro name="azure_kinect" params="
+                      frame:=kinect       topic:=kinect
+                      min_range:=0.5      max_range:=5.46
+                      update_rate:=30
+                      h_fov:=1.3089958333333334 v_fov:=1.1344630555555555
+                      width:=576 height:=640">
+      <!-- this link is the origin for the camera data and corresponds to the front visor of the camera -->
+      <link name="${frame}">
+        <visual>
+          <origin xyz="-0.0128 0. 0." />
+          <geometry>
+            <box size="0.026 0.101 0.037" />
+          </geometry>
+          <material name="black" />
+        </visual>
+      </link>
+      <link name="${frame}_body">
+        <visual>
+          <origin xyz="0. 0. 0." />
+          <geometry>
+            <box size="0.0994 0.0996 0.023" />
+          </geometry>
+          <material name="white" />
+        </visual>
+      </link>
+      <link name="${frame}_base">
+        <visual>
+          <origin xyz="-0.013 0. 0." />
+          <geometry>
+            <box size="0.026 0.103 0.039" />
+          </geometry>
+          <material name="medium_grey" />
+        </visual>
+      </link>
+      <joint name="${frame}_base_to_body" type="fixed">
+        <parent link="${frame}_base" />
+        <child link="${frame}_body" />
+        <origin xyz="-0.0757 0. 0.008" rpy="0. 0. 0." />
+      </joint>
+      <joint name="${frame}_base_to_visor" type="fixed">
+        <parent link="${frame}_base" />
+        <child link="${frame}" />
+        <origin xyz="0. 0. 0." rpy="0. 0. 0." />
+      </joint>
+      <!--
+        The gazebo plugin aligns the depth data with the Z axis, with X=left and Y=up
+        ROS expects the depth data along the X axis, with Y=left and Z=up
+        This link only exists to give the gazebo plugin the correctly-oriented frame
+      -->
+      <link name="${prefix}_kinect_gazebo" />
+      <joint name="${prefix}_kinect_gazebo_joint" type="fixed">
+        <parent link="${frame}"/>
+        <child link="${frame}_gazebo"/>
+        <origin xyz="0 0 0" rpy="-1.5707963267948966 0 -1.5707963267948966"/>
+      </joint>
+      <!--
+        This isn't a 100% accurate representation of the Azure Kinect's data, but it's reasonably close.
+        The color data on the real camera has a 90x59 degree FOV, and the depth data is the full vision
+        cone approximated as a hexagon within the frame.
+        But for now the OpenNI kinect plugin is the closest analogue
+      -->
+      <gazebo reference="${frame}">
+        <turnGravityOff>true</turnGravityOff>
+        <sensor type="depth" name="${prefix}_kinect_depth">
+          <update_rate>${update_rate}</update_rate>
+          <camera>
+            <!-- 75x65 degree FOV for the depth sensor -->
+            <horizontal_fov>${h_fov}</horizontal_fov>
+            <vertical_fov>${v_fov}</vertical_fov>
+            <!-- 90x59 degree FOV for the hardware color camera -->
+            <!-- currently disabled, as this would mangle the depth data
+            <horizontal_fov>1.5707963267948966</horizontal_fov>
+            <vertical_fov>1.0297442586766543</vertical_fov>
+            -->
+            <image>
+              <!--
+                The Azure Kinect has a bit of a weird frame size for the depth data
+                The color data is full-HD+, but that doesn't appear to be supported yet.
+                see: https://docs.microsoft.com/en-us/azure/kinect-dk/hardware-specification
+              -->
+              <width>${width}</width>
+              <height>${height}</height>
+              <!-- TODO: check what format the Azure Kinect hardware delivers and set this to match! -->
+              <format>RGB8</format>
+            </image>
+            <clip>
+              <!-- give the color sensor a maximum range of 50m so that the simulation renders nicely -->
+              <near>0.01</near>
+              <far>50.0</far>
+            </clip>
+          </camera>
+          <plugin name="kinect_controller" filename="libgazebo_ros_openni_kinect.so">
+            <baseline>0.2</baseline>
+            <alwaysOn>true</alwaysOn>
+            <updateRate>0.0</updateRate>
+            <cameraName>${topic}</cameraName>
+            <imageTopicName>color/image_raw</imageTopicName>
+            <cameraInfoTopicName>color/camera_info</cameraInfoTopicName>
+            <depthImageTopicName>depth/image_raw</depthImageTopicName>
+            <depthImageInfoTopicName>depth/camera_info</depthImageInfoTopicName>
+            <pointCloudTopicName>depth/points</pointCloudTopicName>
+            <frameName>${frame}_gazebo</frameName>
+            <!-- the Azure Kinect has an effective depth-sensing range of 0.5m to 5.46m -->
+            <pointCloudCutoff>${min_range}</pointCloudCutoff>
+            <pointCloudCutoffMax>${max_range}</pointCloudCutoffMax>
+            <distortionK1>0.00000001</distortionK1>
+            <distortionK2>0.00000001</distortionK2>
+            <distortionK3>0.00000001</distortionK3>
+            <distortionT1>0.00000001</distortionT1>
+            <distortionT2>0.00000001</distortionT2>
+            <CxPrime>0</CxPrime>
+            <Cx>0</Cx>
+            <Cy>0</Cy>
+            <focalLength>0</focalLength>
+            <hackBaseline>0</hackBaseline>
+          </plugin>
+        </sensor>
+      </gazebo>
+    </xacro:macro>
+    <!-- We assume the 3d-printed mounting plate is in use -->
+    <link name="${prefix}_kinect_mount_plate">
       <visual>
-        <origin xyz="0. 0. 0." />
+        <origin xyz="0 0 0" rpy="0 0 0" />
         <geometry>
-          <box size="0.0994 0.0996 0.023" />
+          <mesh filename="package://jackal_description/meshes/kinect_mount.stl"/>
         </geometry>
-        <material name="white" />
+        <material name="black"/>
       </visual>
     </link>
-    <link name="${prefix}_kinect_base">
-      <visual>
-        <origin xyz="-0.013 0. 0." />
-        <geometry>
-          <box size="0.026 0.103 0.039" />
-        </geometry>
-        <material name="medium_grey" />
-      </visual>
-    </link>
-    <link name="${prefix}_kinect_visor">
-      <visual>
-        <origin xyz="-0.0128 0. 0." />
-        <geometry>
-          <box size="0.026 0.101 0.037" />
-        </geometry>
-        <material name="black" />
-      </visual>
-    </link>
-    <joint name="${prefix}_kinect_base_to_body" type="fixed">
-      <parent link="${prefix}_kinect_base" />
-      <child link="${prefix}_kinect_body" />
-      <origin xyz="-0.0757 0. 0.008" rpy="0. 0. 0." />
+    <joint name="${prefix}_kinect_mount_joint" type="fixed">
+      <origin xyz="0 0 0" rpy="0 0 0"/>
+      <parent link="${parent_link}"/>
+      <child link="${prefix}_kinect_mount_plate"/>
     </joint>
-    <joint name="${prefix}_kinect_base_to_visor" type="fixed">
-      <parent link="${prefix}_kinect_base" />
-      <child link="${prefix}_kinect_visor" />
-      <origin xyz="0. 0. 0." rpy="0. 0. 0." />
+    <!-- this is the actual mounting hole in the mounting plate -->
+    <joint name="${prefix}_kinect_mount_hole" type="fixed">
+      <origin xyz="0.09 0 0.0335" rpy="0 -0.17453292519444444 0"/>
+      <parent link="${prefix}_kinect_mount_plate"/>
+      <child link="${prefix}_kinect_base"/>
     </joint>
-    <!--
-      The gazebo plugin aligns the depth data with the Z axis, with X=left and Y=up
-      ROS expects the depth data along the X axis, with Y=left and Z=up
-      This link only exists to give the gazebo plugin the correctly-oriented frame
-    -->
-    <link name="${prefix}_kinect_gazebo_lens" />
-    <joint name="${prefix}_kinect_gazebo_joint" type="fixed">
-      <parent link="${prefix}_kinect_visor"/>
-      <child link="${prefix}_kinect_gazebo_lens"/>
-      <origin xyz="0 0 0" rpy="-1.5707963267948966 0 -1.5707963267948966"/>
-    </joint>
-    <!--
-      This isn't a 100% accurate representation of the Azure Kinect's data, but it's reasonably close.
-      The color data on the real camera has a 90x59 degree FOV, and the depth data is the full vision
-      cone approximated as a hexagon within the frame.
-      But for now the OpenNI kinect plugin is the closest analogue
-    -->
-    <gazebo reference="${prefix}_kinect_visor">
-      <turnGravityOff>true</turnGravityOff>
-      <sensor type="depth" name="${prefix}_kinect_depth">
-        <update_rate>${update_rate}</update_rate>
-        <camera>
-          <!-- 75x65 degree FOV for the depth sensor -->
-          <horizontal_fov>${h_fov}</horizontal_fov>
-          <vertical_fov>${v_fov}</vertical_fov>
-          <!-- 90x59 degree FOV for the hardware color camera -->
-          <!-- currently disabled, as this would mangle the depth data
-          <horizontal_fov>1.5707963267948966</horizontal_fov>
-          <vertical_fov>1.0297442586766543</vertical_fov>
-          -->
-          <image>
-            <!--
-              The Azure Kinect has a bit of a weird frame size for the depth data
-              The color data is full-HD+, but that doesn't appear to be supported yet.
-              see: https://docs.microsoft.com/en-us/azure/kinect-dk/hardware-specification
-            -->
-            <width>${width}</width>
-            <height>${height}</height>
-            <!-- TODO: check what format the Azure Kinect hardware delivers and set this to match! -->
-            <format>RGB8</format>
-          </image>
-          <clip>
-            <!-- give the color sensor a maximum range of 50m so that the simulation renders nicely -->
-            <near>0.01</near>
-            <far>50.0</far>
-          </clip>
-        </camera>
-        <plugin name="kinect_controller" filename="libgazebo_ros_openni_kinect.so">
-          <baseline>0.2</baseline>
-          <alwaysOn>true</alwaysOn>
-          <updateRate>0.0</updateRate>
-          <cameraName>kinect</cameraName>
-          <imageTopicName>/color/image_raw</imageTopicName>
-          <cameraInfoTopicName>/color/camera_info</cameraInfoTopicName>
-          <depthImageTopicName>/depth/image_raw</depthImageTopicName>
-          <depthImageInfoTopicName>/depth/camera_info</depthImageInfoTopicName>
-          <pointCloudTopicName>/depth/points</pointCloudTopicName>
-          <frameName>${prefix}_kinect_gazebo_lens</frameName>
-          <!-- the Azure Kinect has an effective depth-sensing range of 0.5m to 5.46m -->
-          <pointCloudCutoff>${min_range}</pointCloudCutoff>
-          <pointCloudCutoffMax>${max_range}</pointCloudCutoffMax>
-          <distortionK1>0.00000001</distortionK1>
-          <distortionK2>0.00000001</distortionK2>
-          <distortionK3>0.00000001</distortionK3>
-          <distortionT1>0.00000001</distortionT1>
-          <distortionT2>0.00000001</distortionT2>
-          <CxPrime>0</CxPrime>
-          <Cx>0</Cx>
-          <Cy>0</Cy>
-          <focalLength>0</focalLength>
-          <hackBaseline>0</hackBaseline>
-        </plugin>
-      </sensor>
-    </gazebo>
+    <xacro:azure_kinect frame="${prefix}_kinect" topic="${topic}"/>
   </xacro:macro>
 </robot>

File: jackal_description/urdf/accessories/intel_realsense.urdf.xacro (robot description, xacro)
@@ -9,6 +9,6 @@
                update_rate:=30
                robot_namespace:=/">
-      <link name="${frame}">
-      </link>
+      <!-- this link is the origin for the camera's data -->
+      <link name="${frame}" />
       <!--
         The gazebo plugin aligns the depth data with the Z axis, with X=left and Y=up
