Commit message: Add support for a secondary 2D laser and a primary 3D laser with env vars

File: jackal_description/urdf/accessories.urdf.xacro (robot description, xacro)
@@ -13,18 +13,65 @@
   <!-- This optional plate mounts both the upgraded GPS and the Velodyne 3D LIDAR. -->
   <xacro:include filename="$(find jackal_description)/urdf/accessories/bridge_plate.urdf.xacro" />
-  <!-- If enabled, generate the LASER payload (by default, a SICK LMS111). -->
+  <xacro:include filename="$(find jackal_description)/urdf/accessories/sick_lms1xx_mount.urdf.xacro" />
+  <xacro:include filename="$(find jackal_description)/urdf/accessories/hokuyo_ust10.urdf.xacro" />
+  <xacro:include filename="$(find velodyne_description)/urdf/VLP-16.urdf.xacro" />
+  <!--
+    Add primary/secondary 2D lidar sensors.  By default these are SICK LMS1xx but can be changed with the
+    JACKAL_LASER_MODEL and JACKAL_LASER2_MODEL environment variables. Valid model designations are:
+    - lms1xx (default) :: SICK LMS1xx
+    - ust10            :: Hokuyo UST10
+  -->
   <xacro:if value="$(optenv JACKAL_LASER 0)">
-    <xacro:if value="$(optenv JACKAL_LASER_HOKUYO 0)">
+    <xacro:property name="lidar_model" value="$(optenv JACKAL_LASER_MODEL lms1xx)" />
+    <xacro:if value="${lidar_model == 'lms1xx'}">
+      <xacro:include filename="$(find jackal_description)/urdf/accessories/sick_lms1xx_mount.urdf.xacro" />
+      <xacro:sick_lms1xx_mount prefix="$(optenv JACKAL_LASER_MOUNT front)"
+           parent_link="$(optenv JACKAL_LASER_MOUNT front)_mount"
+           topic="$(optenv JACKAL_LASER_TOPIC front/scan)">
+           <origin xyz="$(optenv JACKAL_LASER_OFFSET 0 0 0)"
+                   rpy="$(optenv JACKAL_LASER_RPY 0 0 0)" />
+         </xacro:sick_lms1xx_mount>
+    </xacro:if>
+    <xacro:if value="${lidar_model == 'ust10'}">
       <xacro:include filename="$(find jackal_description)/urdf/accessories/hokuyo_ust10.urdf.xacro" />
       <xacro:hokuyo_ust10_mount prefix="$(optenv JACKAL_LASER_MOUNT front)"
-                          parent_link="$(optenv JACKAL_LASER_MOUNT front)_mount"
-                          topic="$(optenv JACKAL_LASER_TOPIC front/scan)" />
+          parent_link="$(optenv JACKAL_LASER_MOUNT front)_mount"
+          topic="$(optenv JACKAL_LASER_TOPIC front/scan)">
+          <origin xyz="$(optenv JACKAL_LASER_OFFSET 0 0 0)"
+                  rpy="$(optenv JACKAL_LASER_RPY 0 0 0)" />
+        </xacro:hokuyo_ust10_mount>
     </xacro:if>
-    <xacro:unless value="$(optenv JACKAL_LASER_HOKUYO 0)">
-      <xacro:include filename="$(find jackal_description)/urdf/accessories/sick_lms1xx_mount.urdf.xacro" />
-      <xacro:sick_lms1xx_mount prefix="$(optenv JACKAL_LASER_MOUNT front)"
-                         parent_link="$(optenv JACKAL_LASER_MOUNT front)_mount"
-                         topic="$(optenv JACKAL_LASER_TOPIC front/scan)"/>
-    </xacro:unless>
+  </xacro:if>
+  <xacro:if value="$(optenv JACKAL_LASER2 0)">
+    <xacro:property name="lidar2_model" value="$(optenv JACKAL_LASER2_MODEL lms1xx)" />
+    <xacro:if value="${lidar2_model == 'lms1xx'}">
+      <xacro:sick_lms1xx_mount prefix="$(optenv JACKAL_LASER2_MOUNT rear)"
+           parent_link="$(optenv JACKAL_LASER2_MOUNT rear)_mount"
+           topic="$(optenv JACKAL_LASER2_TOPIC rear/scan)">
+           <origin xyz="$(optenv JACKAL_LASER2_OFFSET 0 0 0)"
+                   rpy="$(optenv JACKAL_LASER2_RPY 0 0 3.14159)" />
+         </xacro:sick_lms1xx_mount>
+    </xacro:if>
+    <xacro:if value="${lidar2_model == 'ust10'}">
+      <xacro:hokuyo_ust10_mount prefix="$(optenv JACKAL_LASER2_MOUNT rear)"
+          parent_link="$(optenv JACKAL_LASER2_MOUNT rear)_mount"
+          topic="$(optenv JACKAL_LASER2_TOPIC rear/scan)">
+          <origin xyz="$(optenv JACKAL_LASER2_OFFSET 0 0 0)"
+                  rpy="$(optenv JACKAL_LASER2_RPY 0 0 3.14159)" />
+        </xacro:hokuyo_ust10_mount>
+    </xacro:if>
+  </xacro:if>
+  <!--
+    Add a 3D lidar sensor.  By default this is a Velodyne VLP16 but can be changed with the
+    JACKAL_LASER_3D_MODEL environment variable. Valid model designations are:
+    - vlp16 (default)  :: Velodyne VLP16
+  -->
+  <xacro:if value="$(optenv JACKAL_LASER_3D 0)">
+    <xacro:property name="lidar_3d_model" value="$(optenv JACKAL_LASER_3D_MODEL vlp16)" />
+    <xacro:if value="${lidar_3d_model == 'vlp16'}">
+      <xacro:VLP-16 parent="$(optenv JACKAL_LASER_3D_MOUNT front)_mount" topic="$(optenv JACKAL_LASER_3D_TOPIC front/points)">
+        <origin xyz="$(optenv JACKAL_LASER_3D_OFFSET 0 0 0)" rpy="$(optenv JACKAL_LASER_3D_RPY 0 0 0)" />
+      </xacro:VLP-16>
+    </xacro:if>
   </xacro:if>
   <!-- If enabled, generate the upgraded Navsat payload (a Novatel Smart6). -->

Commit message: Rename LASER2 to LASER_SECONDARY

File: jackal_description/urdf/accessories.urdf.xacro (robot description, xacro)
@@ -18,5 +18,5 @@
   <!--
     Add primary/secondary 2D lidar sensors.  By default these are SICK LMS1xx but can be changed with the
-    JACKAL_LASER_MODEL and JACKAL_LASER2_MODEL environment variables. Valid model designations are:
+    JACKAL_LASER_MODEL and JACKAL_LASER_SECONDARY_MODEL environment variables. Valid model designations are:
     - lms1xx (default) :: SICK LMS1xx
     - ust10            :: Hokuyo UST10
@@ -43,20 +43,20 @@
     </xacro:if>
   </xacro:if>
-  <xacro:if value="$(optenv JACKAL_LASER2 0)">
-    <xacro:property name="lidar2_model" value="$(optenv JACKAL_LASER2_MODEL lms1xx)" />
+  <xacro:if value="$(optenv JACKAL_LASER_SECONDARY 0)">
+    <xacro:property name="lidar2_model" value="$(optenv JACKAL_LASER_SECONDARY_MODEL lms1xx)" />
     <xacro:if value="${lidar2_model == 'lms1xx'}">
-      <xacro:sick_lms1xx_mount prefix="$(optenv JACKAL_LASER2_MOUNT rear)"
-           parent_link="$(optenv JACKAL_LASER2_MOUNT rear)_mount"
-           topic="$(optenv JACKAL_LASER2_TOPIC rear/scan)">
-           <origin xyz="$(optenv JACKAL_LASER2_OFFSET 0 0 0)"
-                   rpy="$(optenv JACKAL_LASER2_RPY 0 0 3.14159)" />
+      <xacro:sick_lms1xx_mount prefix="$(optenv JACKAL_LASER_SECONDARY_MOUNT rear)"
+           parent_link="$(optenv JACKAL_LASER_SECONDARY_MOUNT rear)_mount"
+           topic="$(optenv JACKAL_LASER_SECONDARY_TOPIC rear/scan)">
+           <origin xyz="$(optenv JACKAL_LASER_SECONDARY_OFFSET 0 0 0)"
+                   rpy="$(optenv JACKAL_LASER_SECONDARY_RPY 0 0 3.14159)" />
          </xacro:sick_lms1xx_mount>
     </xacro:if>
     <xacro:if value="${lidar2_model == 'ust10'}">
-      <xacro:hokuyo_ust10_mount prefix="$(optenv JACKAL_LASER2_MOUNT rear)"
-          parent_link="$(optenv JACKAL_LASER2_MOUNT rear)_mount"
-          topic="$(optenv JACKAL_LASER2_TOPIC rear/scan)">
-          <origin xyz="$(optenv JACKAL_LASER2_OFFSET 0 0 0)"
-                  rpy="$(optenv JACKAL_LASER2_RPY 0 0 3.14159)" />
+      <xacro:hokuyo_ust10_mount prefix="$(optenv JACKAL_LASER_SECONDARY_MOUNT rear)"
+          parent_link="$(optenv JACKAL_LASER_SECONDARY_MOUNT rear)_mount"
+          topic="$(optenv JACKAL_LASER_SECONDARY_TOPIC rear/scan)">
+          <origin xyz="$(optenv JACKAL_LASER_SECONDARY_OFFSET 0 0 0)"
+                  rpy="$(optenv JACKAL_LASER_SECONDARY_RPY 0 0 3.14159)" />
         </xacro:hokuyo_ust10_mount>
     </xacro:if>

Commit message: Indentation fix

File: jackal_description/urdf/accessories.urdf.xacro (robot description, xacro)
@@ -29,7 +29,7 @@
            parent_link="$(optenv JACKAL_LASER_MOUNT front)_mount"
            topic="$(optenv JACKAL_LASER_TOPIC front/scan)">
-           <origin xyz="$(optenv JACKAL_LASER_OFFSET 0 0 0)"
+        <origin xyz="$(optenv JACKAL_LASER_OFFSET 0 0 0)"
                    rpy="$(optenv JACKAL_LASER_RPY 0 0 0)" />
-         </xacro:sick_lms1xx_mount>
+      </xacro:sick_lms1xx_mount>
     </xacro:if>
     <xacro:if value="${lidar_model == 'ust10'}">
@@ -38,7 +38,7 @@
           parent_link="$(optenv JACKAL_LASER_MOUNT front)_mount"
           topic="$(optenv JACKAL_LASER_TOPIC front/scan)">
-          <origin xyz="$(optenv JACKAL_LASER_OFFSET 0 0 0)"
-                  rpy="$(optenv JACKAL_LASER_RPY 0 0 0)" />
-        </xacro:hokuyo_ust10_mount>
+        <origin xyz="$(optenv JACKAL_LASER_OFFSET 0 0 0)"
+                rpy="$(optenv JACKAL_LASER_RPY 0 0 0)" />
+      </xacro:hokuyo_ust10_mount>
     </xacro:if>
   </xacro:if>
@@ -49,7 +49,7 @@
            parent_link="$(optenv JACKAL_LASER_SECONDARY_MOUNT rear)_mount"
            topic="$(optenv JACKAL_LASER_SECONDARY_TOPIC rear/scan)">
-           <origin xyz="$(optenv JACKAL_LASER_SECONDARY_OFFSET 0 0 0)"
-                   rpy="$(optenv JACKAL_LASER_SECONDARY_RPY 0 0 3.14159)" />
-         </xacro:sick_lms1xx_mount>
+         <origin xyz="$(optenv JACKAL_LASER_SECONDARY_OFFSET 0 0 0)"
+                 rpy="$(optenv JACKAL_LASER_SECONDARY_RPY 0 0 3.14159)" />
+       </xacro:sick_lms1xx_mount>
     </xacro:if>
     <xacro:if value="${lidar2_model == 'ust10'}">
@@ -57,7 +57,7 @@
           parent_link="$(optenv JACKAL_LASER_SECONDARY_MOUNT rear)_mount"
           topic="$(optenv JACKAL_LASER_SECONDARY_TOPIC rear/scan)">
-          <origin xyz="$(optenv JACKAL_LASER_SECONDARY_OFFSET 0 0 0)"
-                  rpy="$(optenv JACKAL_LASER_SECONDARY_RPY 0 0 3.14159)" />
-        </xacro:hokuyo_ust10_mount>
+        <origin xyz="$(optenv JACKAL_LASER_SECONDARY_OFFSET 0 0 0)"
+                rpy="$(optenv JACKAL_LASER_SECONDARY_RPY 0 0 3.14159)" />
+      </xacro:hokuyo_ust10_mount>
     </xacro:if>
   </xacro:if>

Commit message: Add a new envar to specify the navsat model (smart6, smart7) and add the meshes for the smart7

File: jackal_description/urdf/accessories.urdf.xacro (robot description, xacro)
@@ -80,8 +80,15 @@
   <!-- If enabled, generate the upgraded Navsat payload (a Novatel Smart6). -->
   <xacro:if value="$(optenv JACKAL_NAVSAT 0)">
-    <xacro:include filename="$(find jackal_description)/urdf/accessories/novatel_smart6.urdf.xacro" />
+    <xacro:property name="navsat_model" value="$(optenv JACKAL_NAVSAT_MODEL smart6)" />
+    <xacro:if value="${navsat_model == 'smart6'}">
+      <xacro:include filename="$(find jackal_description)/urdf/accessories/novatel_smart6.urdf.xacro" />
+      <xacro:novatel_smart6 prefix="$(optenv JACKAL_NAVSAT_MOUNT rear)"/>
+    </xacro:if>
+    <xacro:if value="${navsat_model == 'smart7'}">
+      <xacro:include filename="$(find jackal_description)/urdf/accessories/novatel_smart7.urdf.xacro" />
+      <xacro:novatel_smart7 prefix="$(optenv JACKAL_NAVSAT_MOUNT rear)"/>
+    </xacro:if>
     <xacro:bridge_plate mount="$(optenv JACKAL_NAVSAT_MOUNT rear)"
                   height="$(optenv JACKAL_NAVSAT_HEIGHT 0.1)" />
-    <xacro:novatel_smart6 prefix="$(optenv JACKAL_NAVSAT_MOUNT rear)"/>
     <joint name="$(optenv JACKAL_NAVSAT_MOUNT rear)_navsat_joint" type="fixed">
       <origin xyz="0 0 0" rpy="0 0 0" />

Commit message: Use the Smart7 by default

File: jackal_description/urdf/accessories.urdf.xacro (robot description, xacro)
@@ -80,5 +80,5 @@
   <!-- If enabled, generate the upgraded Navsat payload (a Novatel Smart6). -->
   <xacro:if value="$(optenv JACKAL_NAVSAT 0)">
-    <xacro:property name="navsat_model" value="$(optenv JACKAL_NAVSAT_MODEL smart6)" />
+    <xacro:property name="navsat_model" value="$(optenv JACKAL_NAVSAT_MODEL smart7)" />
     <xacro:if value="${navsat_model == 'smart6'}">
       <xacro:include filename="$(find jackal_description)/urdf/accessories/novatel_smart6.urdf.xacro" />

Commit message: Revert to the smart6 by default for Melodic

File: jackal_description/urdf/accessories.urdf.xacro (robot description, xacro)
@@ -80,5 +80,5 @@
   <!-- If enabled, generate the upgraded Navsat payload (a Novatel Smart6). -->
   <xacro:if value="$(optenv JACKAL_NAVSAT 0)">
-    <xacro:property name="navsat_model" value="$(optenv JACKAL_NAVSAT_MODEL smart7)" />
+    <xacro:property name="navsat_model" value="$(optenv JACKAL_NAVSAT_MODEL smart6)" />
     <xacro:if value="${navsat_model == 'smart6'}">
       <xacro:include filename="$(find jackal_description)/urdf/accessories/novatel_smart6.urdf.xacro" />

Commit message: Added JACKAL_LASER_3D_TOWER (TRUE/false) environment variable to toggle the Velodyne mounting tower. Added HDL-32E to robot description, set using  JACKAL_LASER_3D_MODEL=hdl32e.

File: jackal_description/urdf/accessories.urdf.xacro (robot description, xacro)
@@ -16,4 +16,5 @@
   <xacro:include filename="$(find jackal_description)/urdf/accessories/hokuyo_ust10.urdf.xacro" />
   <xacro:include filename="$(find jackal_description)/urdf/accessories/vlp16_mount.urdf.xacro" />
+  <xacro:include filename="$(find jackal_description)/urdf/accessories/hdl32_mount.urdf.xacro" />
   <!--
     Add primary/secondary 2D lidar sensors.  By default these are SICK LMS1xx but can be changed with the
@@ -66,4 +67,5 @@
     JACKAL_LASER_3D_MODEL environment variable. Valid model designations are:
     - vlp16 (default)  :: Velodyne VLP16
+    - vlp32e           :: Velodyne HDL-32E
   -->
   <xacro:if value="$(optenv JACKAL_LASER_3D 0)">
@@ -73,7 +75,17 @@
           parent_link="$(optenv JACKAL_LASER_3D_MOUNT mid)_mount"
           prefix="$(optenv JACKAL_LASER_3D_MOUNT mid)"
-          topic="$(optenv JACKAL_LASER_3D_TOPIC mid/points)">
+          topic="$(optenv JACKAL_LASER_3D_TOPIC mid/points)"
+          tower="$(optenv JACKAL_LASER_3D_TOWER True)">
         <origin xyz="$(optenv JACKAL_LASER_3D_OFFSET 0 0 0)" rpy="$(optenv JACKAL_LASER_3D_RPY 0 0 0)" />
       </xacro:vlp16_mount>
+    </xacro:if>
+    <xacro:if value="${lidar_3d_model == 'hdl32e'}">
+      <xacro:hdl32e_mount
+          parent_link="$(optenv JACKAL_LASER_3D_MOUNT mid)_mount"
+          prefix="$(optenv JACKAL_LASER_3D_MOUNT mid)"
+	        topic="$(optenv JACKAL_LASER_3D_TOPIC mid/points)"
+          tower="$(optenv JACKAL_LASER_3D_TOWER 1)">
+	    <origin xyz="$(optenv JACKAL_LASER_3D_OFFSET 0 0 0)" rpy="$(optenv JACKAL_LASER_3D_RPY 0 0 0)" />
+      </xacro:hdl32e_mount>
     </xacro:if>
   </xacro:if>

File: jackal_description/urdf/accessories/vlp16_mount.urdf.xacro (robot description, xacro)
@@ -1,92 +1,99 @@
 <robot xmlns:xacro="http://wiki.ros.org/xacro">
   <xacro:include filename="$(find velodyne_description)/urdf/VLP-16.urdf.xacro" />
-  <xacro:macro name="vlp16_mount" params="prefix parent_link topic height:=0.1 *origin">
-    <link name="${prefix}_vlp16_mount" />
-    <link name="${prefix}_vlp16_plate">
-      <visual>
-        <geometry>
-          <box size="0.1 0.1 0.002" />
-        </geometry>
-        <material name="black" />
-        <origin xyz="0 0 -0.001" rpy="0 0 0" />
-      </visual>
-    </link>
-    <link name="${prefix}_vlp16_leg1">
-      <visual>
-        <geometry>
-          <cylinder length="${height}" radius="0.003" />
-        </geometry>
-        <material name="white">
-          <color rgba="1 1 1 1" />
-        </material>
-        <origin xyz="0 0 ${height/2}" rpy="0 0 0" />
-      </visual>
-    </link>
-    <link name="${prefix}_vlp16_leg2">
-      <visual>
-        <geometry>
-          <cylinder length="${height}" radius="0.003" />
-        </geometry>
-        <material name="white">
-          <color rgba="1 1 1 1" />
-        </material>
-        <origin xyz="0 0 ${height/2}" rpy="0 0 0" />
-      </visual>
-    </link>
-    <link name="${prefix}_vlp16_leg3">
-      <visual>
-        <geometry>
-          <cylinder length="${height}" radius="0.003" />
-        </geometry>
-        <material name="white">
-          <color rgba="1 1 1 1" />
-        </material>
-        <origin xyz="0 0 ${height/2}" rpy="0 0 0" />
-      </visual>
-    </link>
-    <link name="${prefix}_vlp16_leg4">
-      <visual>
-        <geometry>
-          <cylinder length="${height}" radius="0.003" />
-        </geometry>
-        <material name="white">
-          <color rgba="1 1 1 1" />
-        </material>
-        <origin xyz="0 0 ${height/2}" rpy="0 0 0" />
-      </visual>
-    </link>
-    <joint name="${prefix}_vlp16_mount_joint" type="fixed">
-      <parent link="${parent_link}" />
-      <child link="${prefix}_vlp16_mount" />
-      <xacro:insert_block name="origin" />
-    </joint>
-    <joint name="${prefix}_vlp16_leg1_joint" type="fixed">
-      <parent link="${prefix}_mount" />
-      <child link="${prefix}_vlp16_leg1" />
-      <origin xyz="0.05 0.05 0" rpy="0 0 0" />
-    </joint>
-    <joint name="${prefix}_vlp16_leg2_joint" type="fixed">
-      <parent link="${prefix}_mount" />
-      <child link="${prefix}_vlp16_leg2" />
-      <origin xyz="0.05 -0.05 0" rpy="0 0 0" />
-    </joint>
-    <joint name="${prefix}_vlp16_leg3_joint" type="fixed">
-      <parent link="${prefix}_mount" />
-      <child link="${prefix}_vlp16_leg3" />
-      <origin xyz="-0.05 0.05 0" rpy="0 0 0" />
-    </joint>
-    <joint name="${prefix}_vlp16_leg4_joint" type="fixed">
-      <parent link="${prefix}_mount" />
-      <child link="${prefix}_vlp16_leg4" />
-      <origin xyz="-0.05 -0.05 0" rpy="0 0 0" />
-    </joint>
-    <joint name="${prefix}_vlp16_plate_joint" type="fixed">
-      <parent link="${prefix}_vlp16_mount" />
-      <child link="${prefix}_vlp16_plate" />
-      <origin xyz="0 0 ${height}" rpy="0 0 0" />
-    </joint>
-    <xacro:VLP-16 parent="${prefix}_vlp16_plate" topic="${topic}">
-      <origin xyz="0 0 0" rpy="0 0 0" />
-    </xacro:VLP-16>
+  <xacro:macro name="vlp16_mount" params="prefix parent_link topic tower height:=0.1 *origin">
+    <xacro:if value="${tower}">
+      <link name="${prefix}_vlp16_mount" />
+      <link name="${prefix}_vlp16_plate">
+        <visual>
+          <geometry>
+            <box size="0.1 0.1 0.002" />
+          </geometry>
+          <material name="black" />
+          <origin xyz="0 0 -0.001" rpy="0 0 0" />
+        </visual>
+      </link>
+      <link name="${prefix}_vlp16_leg1">
+        <visual>
+          <geometry>
+            <cylinder length="${height}" radius="0.003" />
+          </geometry>
+          <material name="white">
+            <color rgba="1 1 1 1" />
+          </material>
+          <origin xyz="0 0 ${height/2}" rpy="0 0 0" />
+        </visual>
+      </link>
+      <link name="${prefix}_vlp16_leg2">
+        <visual>
+          <geometry>
+            <cylinder length="${height}" radius="0.003" />
+          </geometry>
+          <material name="white">
+            <color rgba="1 1 1 1" />
+          </material>
+          <origin xyz="0 0 ${height/2}" rpy="0 0 0" />
+        </visual>
+      </link>
+      <link name="${prefix}_vlp16_leg3">
+        <visual>
+          <geometry>
+            <cylinder length="${height}" radius="0.003" />
+          </geometry>
+          <material name="white">
+            <color rgba="1 1 1 1" />
+          </material>
+          <origin xyz="0 0 ${height/2}" rpy="0 0 0" />
+        </visual>
+      </link>
+      <link name="${prefix}_vlp16_leg4">
+        <visual>
+          <geometry>
+            <cylinder length="${height}" radius="0.003" />
+          </geometry>
+          <material name="white">
+            <color rgba="1 1 1 1" />
+          </material>
+          <origin xyz="0 0 ${height/2}" rpy="0 0 0" />
+        </visual>
+      </link>
+      <joint name="${prefix}_vlp16_mount_joint" type="fixed">
+        <parent link="${parent_link}" />
+        <child link="${prefix}_vlp16_mount" />
+        <xacro:insert_block name="origin" />
+      </joint>
+      <joint name="${prefix}_vlp16_leg1_joint" type="fixed">
+        <parent link="${prefix}_mount" />
+        <child link="${prefix}_vlp16_leg1" />
+        <origin xyz="0.05 0.05 0" rpy="0 0 0" />
+      </joint>
+      <joint name="${prefix}_vlp16_leg2_joint" type="fixed">
+        <parent link="${prefix}_mount" />
+        <child link="${prefix}_vlp16_leg2" />
+        <origin xyz="0.05 -0.05 0" rpy="0 0 0" />
+      </joint>
+      <joint name="${prefix}_vlp16_leg3_joint" type="fixed">
+        <parent link="${prefix}_mount" />
+        <child link="${prefix}_vlp16_leg3" />
+        <origin xyz="-0.05 0.05 0" rpy="0 0 0" />
+      </joint>
+      <joint name="${prefix}_vlp16_leg4_joint" type="fixed">
+        <parent link="${prefix}_mount" />
+        <child link="${prefix}_vlp16_leg4" />
+        <origin xyz="-0.05 -0.05 0" rpy="0 0 0" />
+      </joint>
+      <joint name="${prefix}_vlp16_plate_joint" type="fixed">
+        <parent link="${prefix}_vlp16_mount" />
+        <child link="${prefix}_vlp16_plate" />
+        <origin xyz="0 0 ${height}" rpy="0 0 0" />
+      </joint>
+      <xacro:VLP-16 parent="${prefix}_vlp16_plate" topic="${topic}">
+        <origin xyz="0 0 0" rpy="0 0 0" />
+      </xacro:VLP-16>
+    </xacro:if>
+    <xacro:unless value="${tower}">
+      <xacro:VLP-16 parent="${parent_link}" topic="${topic}">
+        <xacro:insert_block name="origin" />
+      </xacro:VLP-16>
+    </xacro:unless>
   </xacro:macro>
 </robot>
