Commit message: Removed tab, interim commit

File: jackal_description/urdf/accessories.urdf.xacro (robot description, xacro)
@@ -76,5 +76,5 @@
           prefix="$(optenv JACKAL_LASER_3D_MOUNT mid)"
           topic="$(optenv JACKAL_LASER_3D_TOPIC mid/points)"
-          tower="$(optenv JACKAL_LASER_3D_TOWER True)">
+          tower="$(optenv JACKAL_LASER_3D_TOWER 1)">
         <origin xyz="$(optenv JACKAL_LASER_3D_OFFSET 0 0 0)" rpy="$(optenv JACKAL_LASER_3D_RPY 0 0 0)" />
       </xacro:vlp16_mount>
@@ -84,7 +84,7 @@
           parent_link="$(optenv JACKAL_LASER_3D_MOUNT mid)_mount"
           prefix="$(optenv JACKAL_LASER_3D_MOUNT mid)"
-	        topic="$(optenv JACKAL_LASER_3D_TOPIC mid/points)"
+          topic="$(optenv JACKAL_LASER_3D_TOPIC mid/points)"
           tower="$(optenv JACKAL_LASER_3D_TOWER 1)">
-	    <origin xyz="$(optenv JACKAL_LASER_3D_OFFSET 0 0 0)" rpy="$(optenv JACKAL_LASER_3D_RPY 0 0 0)" />
+        <origin xyz="$(optenv JACKAL_LASER_3D_OFFSET 0 0 0)" rpy="$(optenv JACKAL_LASER_3D_RPY 0 0 0)" />
       </xacro:hdl32e_mount>
     </xacro:if>

File: jackal_description/urdf/accessories/vlp16_mount.urdf.xacro (robot description, xacro)
@@ -2,93 +2,93 @@
   <xacro:include filename="$(find velodyne_description)/urdf/VLP-16.urdf.xacro" />
   <xacro:macro name="vlp16_mount" params="prefix parent_link topic tower height:=0.1 *origin">
-    <xacro:if value="${tower}">
-      <link name="${prefix}_vlp16_mount" />
-      <link name="${prefix}_vlp16_plate">
-        <visual>
-          <geometry>
-            <box size="0.1 0.1 0.002" />
-          </geometry>
-          <material name="black" />
-          <origin xyz="0 0 -0.001" rpy="0 0 0" />
-        </visual>
-      </link>
-      <link name="${prefix}_vlp16_leg1">
-        <visual>
-          <geometry>
-            <cylinder length="${height}" radius="0.003" />
-          </geometry>
-          <material name="white">
-            <color rgba="1 1 1 1" />
-          </material>
-          <origin xyz="0 0 ${height/2}" rpy="0 0 0" />
-        </visual>
-      </link>
-      <link name="${prefix}_vlp16_leg2">
-        <visual>
-          <geometry>
-            <cylinder length="${height}" radius="0.003" />
-          </geometry>
-          <material name="white">
-            <color rgba="1 1 1 1" />
-          </material>
-          <origin xyz="0 0 ${height/2}" rpy="0 0 0" />
-        </visual>
-      </link>
-      <link name="${prefix}_vlp16_leg3">
-        <visual>
-          <geometry>
-            <cylinder length="${height}" radius="0.003" />
-          </geometry>
-          <material name="white">
-            <color rgba="1 1 1 1" />
-          </material>
-          <origin xyz="0 0 ${height/2}" rpy="0 0 0" />
-        </visual>
-      </link>
-      <link name="${prefix}_vlp16_leg4">
-        <visual>
-          <geometry>
-            <cylinder length="${height}" radius="0.003" />
-          </geometry>
-          <material name="white">
-            <color rgba="1 1 1 1" />
-          </material>
-          <origin xyz="0 0 ${height/2}" rpy="0 0 0" />
-        </visual>
-      </link>
-      <joint name="${prefix}_vlp16_mount_joint" type="fixed">
-        <parent link="${parent_link}" />
-        <child link="${prefix}_vlp16_mount" />
-        <xacro:insert_block name="origin" />
-      </joint>
-      <joint name="${prefix}_vlp16_leg1_joint" type="fixed">
-        <parent link="${prefix}_vlp16_mount" />
-        <child link="${prefix}_vlp16_leg1" />
-        <origin xyz="0.05 0.05 0" rpy="0 0 0" />
-      </joint>
-      <joint name="${prefix}_vlp16_leg2_joint" type="fixed">
-        <parent link="${prefix}_vlp16_mount" />
-        <child link="${prefix}_vlp16_leg2" />
-        <origin xyz="0.05 -0.05 0" rpy="0 0 0" />
-      </joint>
-      <joint name="${prefix}_vlp16_leg3_joint" type="fixed">
-        <parent link="${prefix}_vlp16_mount" />
-        <child link="${prefix}_vlp16_leg3" />
-        <origin xyz="-0.05 0.05 0" rpy="0 0 0" />
-      </joint>
-      <joint name="${prefix}_vlp16_leg4_joint" type="fixed">
-        <parent link="${prefix}_vlp16_mount" />
-        <child link="${prefix}_vlp16_leg4" />
-        <origin xyz="-0.05 -0.05 0" rpy="0 0 0" />
-      </joint>
-      <joint name="${prefix}_vlp16_plate_joint" type="fixed">
-        <parent link="${prefix}_vlp16_mount" />
-        <child link="${prefix}_vlp16_plate" />
-        <origin xyz="0 0 ${height}" rpy="0 0 0" />
-      </joint>
-      <xacro:VLP-16 parent="${prefix}_vlp16_plate" topic="${topic}">
-        <origin xyz="0 0 0" rpy="0 0 0" />
-      </xacro:VLP-16>
-    </xacro:if>
+  <xacro:if value="${tower}">
+    <link name="${prefix}_vlp16_mount" />
+    <link name="${prefix}_vlp16_plate">
+      <visual>
+        <geometry>
+          <box size="0.1 0.1 0.002" />
+        </geometry>
+        <material name="black" />
+        <origin xyz="0 0 -0.001" rpy="0 0 0" />
+      </visual>
+    </link>
+    <link name="${prefix}_vlp16_leg1">
+      <visual>
+        <geometry>
+          <cylinder length="${height}" radius="0.003" />
+        </geometry>
+        <material name="white">
+          <color rgba="1 1 1 1" />
+        </material>
+        <origin xyz="0 0 ${height/2}" rpy="0 0 0" />
+      </visual>
+    </link>
+    <link name="${prefix}_vlp16_leg2">
+      <visual>
+        <geometry>
+          <cylinder length="${height}" radius="0.003" />
+        </geometry>
+        <material name="white">
+          <color rgba="1 1 1 1" />
+        </material>
+        <origin xyz="0 0 ${height/2}" rpy="0 0 0" />
+      </visual>
+    </link>
+    <link name="${prefix}_vlp16_leg3">
+      <visual>
+        <geometry>
+          <cylinder length="${height}" radius="0.003" />
+        </geometry>
+        <material name="white">
+          <color rgba="1 1 1 1" />
+        </material>
+        <origin xyz="0 0 ${height/2}" rpy="0 0 0" />
+      </visual>
+    </link>
+    <link name="${prefix}_vlp16_leg4">
+      <visual>
+        <geometry>
+          <cylinder length="${height}" radius="0.003" />
+        </geometry>
+        <material name="white">
+          <color rgba="1 1 1 1" />
+        </material>
+        <origin xyz="0 0 ${height/2}" rpy="0 0 0" />
+      </visual>
+    </link>
+    <joint name="${prefix}_vlp16_mount_joint" type="fixed">
+      <parent link="${parent_link}" />
+      <child link="${prefix}_vlp16_mount" />
+      <xacro:insert_block name="origin" />
+    </joint>
+    <joint name="${prefix}_vlp16_leg1_joint" type="fixed">
+      <parent link="${prefix}_vlp16_mount" />
+      <child link="${prefix}_vlp16_leg1" />
+      <origin xyz="0.05 0.05 0" rpy="0 0 0" />
+    </joint>
+    <joint name="${prefix}_vlp16_leg2_joint" type="fixed">
+      <parent link="${prefix}_vlp16_mount" />
+      <child link="${prefix}_vlp16_leg2" />
+      <origin xyz="0.05 -0.05 0" rpy="0 0 0" />
+    </joint>
+    <joint name="${prefix}_vlp16_leg3_joint" type="fixed">
+      <parent link="${prefix}_vlp16_mount" />
+      <child link="${prefix}_vlp16_leg3" />
+      <origin xyz="-0.05 0.05 0" rpy="0 0 0" />
+    </joint>
+    <joint name="${prefix}_vlp16_leg4_joint" type="fixed">
+      <parent link="${prefix}_vlp16_mount" />
+      <child link="${prefix}_vlp16_leg4" />
+      <origin xyz="-0.05 -0.05 0" rpy="0 0 0" />
+    </joint>
+    <joint name="${prefix}_vlp16_plate_joint" type="fixed">
+      <parent link="${prefix}_vlp16_mount" />
+      <child link="${prefix}_vlp16_plate" />
+      <origin xyz="0 0 ${height}" rpy="0 0 0" />
+    </joint>
+    <xacro:VLP-16 parent="${prefix}_vlp16_plate" topic="${topic}">
+      <origin xyz="0 0 0" rpy="0 0 0" />
+    </xacro:VLP-16>
+  </xacro:if>
     <xacro:unless value="${tower}">
       <xacro:VLP-16 parent="${parent_link}" topic="${topic}">

Commit message: Added velodyne towers and HDL-32E sensor (#88)
* Added JACKAL_LASER_3D_TOWER (TRUE/false) environment variable to toggle the Velodyne mounting tower. Added HDL-32E to robot description, set using  JACKAL_LASER_3D_MODEL=hdl32e.

* Fixed naming errors in HDL-32E urdf

* Fixed issue where setting offset and rpy environment variables wouldn't move the vlp16 tower appropriately

* Removed tab, interim commit

* Added spaces

* Removed tabs

* Added spaces

* Removing tabs...

* Adding spaces...

* Removing tabs...

* Added spaces...

* Removed tabs

* Added 1 space

* Added a tab and space

* Removed tab

* Added tab to vlp16_plate

* Removed tab from vlp16_plate

* Removed indentation

* Restored indentation

* Update vlp16_mount.urdf.xacro

* Update vlp16_mount.urdf.xacro

* Update vlp16_mount.urdf.xacro

* Update vlp16_mount.urdf.xacro

* Update vlp16_mount.urdf.xacro

File: jackal_description/urdf/accessories.urdf.xacro (robot description, xacro)
@@ -16,4 +16,5 @@
   <xacro:include filename="$(find jackal_description)/urdf/accessories/hokuyo_ust10.urdf.xacro" />
   <xacro:include filename="$(find jackal_description)/urdf/accessories/vlp16_mount.urdf.xacro" />
+  <xacro:include filename="$(find jackal_description)/urdf/accessories/hdl32_mount.urdf.xacro" />
   <!--
     Add primary/secondary 2D lidar sensors.  By default these are SICK LMS1xx but can be changed with the
@@ -66,4 +67,5 @@
     JACKAL_LASER_3D_MODEL environment variable. Valid model designations are:
     - vlp16 (default)  :: Velodyne VLP16
+    - vlp32e           :: Velodyne HDL-32E
   -->
   <xacro:if value="$(optenv JACKAL_LASER_3D 0)">
@@ -73,7 +75,17 @@
           parent_link="$(optenv JACKAL_LASER_3D_MOUNT mid)_mount"
           prefix="$(optenv JACKAL_LASER_3D_MOUNT mid)"
-          topic="$(optenv JACKAL_LASER_3D_TOPIC mid/points)">
+          topic="$(optenv JACKAL_LASER_3D_TOPIC mid/points)"
+          tower="$(optenv JACKAL_LASER_3D_TOWER 1)">
         <origin xyz="$(optenv JACKAL_LASER_3D_OFFSET 0 0 0)" rpy="$(optenv JACKAL_LASER_3D_RPY 0 0 0)" />
       </xacro:vlp16_mount>
+    </xacro:if>
+    <xacro:if value="${lidar_3d_model == 'hdl32e'}">
+      <xacro:hdl32e_mount
+          parent_link="$(optenv JACKAL_LASER_3D_MOUNT mid)_mount"
+          prefix="$(optenv JACKAL_LASER_3D_MOUNT mid)"
+          topic="$(optenv JACKAL_LASER_3D_TOPIC mid/points)"
+          tower="$(optenv JACKAL_LASER_3D_TOWER 1)">
+        <origin xyz="$(optenv JACKAL_LASER_3D_OFFSET 0 0 0)" rpy="$(optenv JACKAL_LASER_3D_RPY 0 0 0)" />
+      </xacro:hdl32e_mount>
     </xacro:if>
   </xacro:if>

Commit message: Added BlackflyS to accessories (depends on sensor_mounts and flir_camera_driver)

File: jackal_description/urdf/accessories.urdf.xacro (robot description, xacro)
@@ -112,4 +112,5 @@
   <xacro:include filename="$(find jackal_description)/urdf/accessories/camera_mount.urdf.xacro" />
   <xacro:include filename="$(find pointgrey_camera_description)/urdf/pointgrey_flea3.urdf.xacro" />
+  <xacro:include filename="$(find flir_camera_description)/urdf/flir_blackflys.urdf.xacro" />
   <!-- If enabled, generate the flea3 camera payload with a tilt of 30 degrees. -->
   <xacro:if value="$(optenv JACKAL_FLEA3 0)">
@@ -129,4 +130,19 @@
       <parent link="$(optenv JACKAL_FLEA3_MOUNT front)_camera_beam" />
       <child link="$(optenv JACKAL_FLEA3_MOUNT front)_camera" />
+    </joint>
+  </xacro:if>
+  <xacro:if value="$(optenv JACKAL_BLACKFLYS 0)">
+    <!-- Include Mount (default to lockmount) -->
+    <xacro:include filename="$(find lockmount_description)/urdf/lockmount.urdf.xacro" />
+    <xacro:lockmount prefix="$(optenv JACKAL_BLACKFLYS_PREFIX front)_camera" parent_link="$(optenv JACKAL_BLACKFLYS_PARENT front_mount)" angle="$(optenv JACKAL_BLACKFLYS_TILT 0)">
+      <origin xyz="$(optenv JACKAL_BLACKFLYS_OFFSET)" rpy="$(optenv JACKAL_BLACKFLYS_RPY)" />
+    </xacro:lockmount>
+    <!-- Include Flir BlackflyS -->
+    <xacro:include filename="$(find flir_camera_description)/urdf/flir_blackflys.urdf.xacro" />
+    <xacro:flir_blackflys frame="$(optenv JACKAL_BLACKFLYS_PREFIX front)_camera" />
+    <joint name="$(optenv JACKAL_BLACKFLYS_PREFIX front)_camera_mount_camera_joint" type="fixed">
+      <origin xyz="0 0 0" rpy="0 0 0" />
+      <parent link="$(optenv JACKAL_BLACKFLYS_PREFIX front)_camera_mount_link"/>
+      <child link="$(optenv JACKAL_BLACKFLYS_PREFIX front)_camera"/>
     </joint>
   </xacro:if>
