Commit message: Updated LASER, NAVSAT, and, FLEA3 to enable tower variable

File: jackal_description/urdf/accessories.urdf.xacro (robot description, xacro)
@@ -23,41 +23,43 @@
     - ust10            :: Hokuyo UST10
   -->
+  <!-- Primary 2D Lidar -->
   <xacro:if value="$(optenv JACKAL_LASER 0)">
+    <xacro:property name="mount" value="$(optenv JACKAL_LASER_MOUNT front)" />
+    <xacro:property name="topic" value="$(optenv JACKAL_LASER_TOPIC ${mount}/scan)" />
+    <xacro:property name="tower" value="$(optenv JACKAL_LASER_TOWER 1)" />
+    <xacro:property name="prefix" value="$(optenv JACKAL_LASER_PREFIX ${mount})" />
+    <xacro:property name="parent_link" value="$(optenv JACKAL_LASER_PARENT ${mount}_mount)" />
     <xacro:property name="lidar_model" value="$(optenv JACKAL_LASER_MODEL lms1xx)" />
+    <!-- SICK LMS1xx -->
     <xacro:if value="${lidar_model == 'lms1xx'}">
-      <xacro:include filename="$(find jackal_description)/urdf/accessories/sick_lms1xx_mount.urdf.xacro" />
-      <xacro:sick_lms1xx_mount prefix="$(optenv JACKAL_LASER_MOUNT front)"
-           parent_link="$(optenv JACKAL_LASER_MOUNT front)_mount"
-           topic="$(optenv JACKAL_LASER_TOPIC front/scan)">
-        <origin xyz="$(optenv JACKAL_LASER_OFFSET 0 0 0)"
-                   rpy="$(optenv JACKAL_LASER_RPY 0 0 0)" />
+      <xacro:sick_lms1xx_mount  topic="${topic}" prefix="${prefix}" parent_link="${parent_link}">
+        <origin xyz="$(optenv JACKAL_LASER_OFFSET 0 0 0)" rpy="$(optenv JACKAL_LASER_RPY 0 0 0)" />
       </xacro:sick_lms1xx_mount>
     </xacro:if>
+    <!-- Hokuyo UST10 -->
     <xacro:if value="${lidar_model == 'ust10'}">
-      <xacro:include filename="$(find jackal_description)/urdf/accessories/hokuyo_ust10.urdf.xacro" />
-      <xacro:hokuyo_ust10_mount prefix="$(optenv JACKAL_LASER_MOUNT front)"
-          parent_link="$(optenv JACKAL_LASER_MOUNT front)_mount"
-          topic="$(optenv JACKAL_LASER_TOPIC front/scan)">
-        <origin xyz="$(optenv JACKAL_LASER_OFFSET 0 0 0)"
-                rpy="$(optenv JACKAL_LASER_RPY 0 0 0)" />
-      </xacro:hokuyo_ust10_mount>
-    </xacro:if>
-  </xacro:if>
+      <xacro:hokuyo_ust10_mount topic="${topic}" prefix="${prefix}" parent_link="${parent_link}">
+        <origin xyz="$(optenv JACKAL_LASER_OFFSET 0 0 0)" rpy="$(optenv JACKAL_LASER_RPY 0 0 0)" />
+      </xacro:hokuyo_ust10_mount>
+    </xacro:if>
+  </xacro:if>
+  <!-- Secondary 2D Lidar -->
   <xacro:if value="$(optenv JACKAL_LASER_SECONDARY 0)">
-    <xacro:property name="lidar2_model" value="$(optenv JACKAL_LASER_SECONDARY_MODEL lms1xx)" />
-    <xacro:if value="${lidar2_model == 'lms1xx'}">
-      <xacro:sick_lms1xx_mount prefix="$(optenv JACKAL_LASER_SECONDARY_MOUNT rear)"
-           parent_link="$(optenv JACKAL_LASER_SECONDARY_MOUNT rear)_mount"
-           topic="$(optenv JACKAL_LASER_SECONDARY_TOPIC rear/scan)">
-         <origin xyz="$(optenv JACKAL_LASER_SECONDARY_OFFSET 0 0 0)"
-                 rpy="$(optenv JACKAL_LASER_SECONDARY_RPY 0 0 3.14159)" />
+    <xacro:property name="mount" value="$(optenv JACKAL_LASER_SECONDARY_MOUNT rear)" />
+    <xacro:property name="topic" value="$(optenv JACKAL_LASER_SECONDARY_TOPIC ${mount}/scan)" />
+    <xacro:property name="tower" value="$(optenv JACKAL_LASER_SECONDARY_TOWER 1)" />
+    <xacro:property name="prefix" value="$(optenv JACKAL_LASER_SECONDARY_PREFIX ${mount})" />
+    <xacro:property name="parent_link" value="$(optenv JACKAL_LASER_SECONDARY_PARENT ${mount}_mount)" />
+    <xacro:property name="lidar_model" value="$(optenv JACKAL_LASER_SECONDARY_MODEL lms1xx)" />
+    <!-- SICK LM1xx -->
+    <xacro:if value="${lidar_model == 'lms1xx'}">
+      <xacro:sick_lms1xx_mount  topic="${topic}" prefix="${prefix}" parent_link="${parent_link}">
+         <origin xyz="$(optenv JACKAL_LASER_SECONDARY_OFFSET 0 0 0)" rpy="$(optenv JACKAL_LASER_SECONDARY_RPY 0 0 3.14159)" />
        </xacro:sick_lms1xx_mount>
     </xacro:if>
-    <xacro:if value="${lidar2_model == 'ust10'}">
-      <xacro:hokuyo_ust10_mount prefix="$(optenv JACKAL_LASER_SECONDARY_MOUNT rear)"
-          parent_link="$(optenv JACKAL_LASER_SECONDARY_MOUNT rear)_mount"
-          topic="$(optenv JACKAL_LASER_SECONDARY_TOPIC rear/scan)">
-        <origin xyz="$(optenv JACKAL_LASER_SECONDARY_OFFSET 0 0 0)"
-                rpy="$(optenv JACKAL_LASER_SECONDARY_RPY 0 0 3.14159)" />
+    <!-- Hokuyo UST10 -->
+    <xacro:if value="${lidar_model == 'ust10'}">
+      <xacro:hokuyo_ust10_mount topic="${topic}" prefix="${prefix}" parent_link="${parent_link}">
+        <origin xyz="$(optenv JACKAL_LASER_SECONDARY_OFFSET 0 0 0)" rpy="$(optenv JACKAL_LASER_SECONDARY_RPY 0 0 3.14159)" />
       </xacro:hokuyo_ust10_mount>
     </xacro:if>
@@ -70,42 +72,83 @@
   -->
   <xacro:if value="$(optenv JACKAL_LASER_3D 0)">
+    <xacro:property name="mount" value="$(optenv JACKAL_LASER_3D_MOUNT mid)" />
+    <xacro:property name="topic" value="$(optenv JACKAL_LASER_3D_TOPIC ${mount}/points)" />
+    <xacro:property name="tower" value="$(optenv JACKAL_LASER_3D_TOWER 1)" />
+    <xacro:property name="prefix" value="$(optenv JACKAL_LASER_PREFIX ${mount})" />
+    <xacro:property name="parent_link" value="$(optenv JACKAL_LASER_PARENT ${mount}_mount)" />
     <xacro:property name="lidar_3d_model" value="$(optenv JACKAL_LASER_3D_MODEL vlp16)" />
+    <!-- Velodyne VLP16 -->
     <xacro:if value="${lidar_3d_model == 'vlp16'}">
-      <xacro:vlp16_mount
-          parent_link="$(optenv JACKAL_LASER_3D_MOUNT mid)_mount"
-          prefix="$(optenv JACKAL_LASER_3D_MOUNT mid)"
-          topic="$(optenv JACKAL_LASER_3D_TOPIC mid/points)"
-          tower="$(optenv JACKAL_LASER_3D_TOWER 1)">
+      <xacro:vlp16_mount topic="${topic}" tower="${tower}" prefix="${prefix}" parent_link="${parent_link}" >
         <origin xyz="$(optenv JACKAL_LASER_3D_OFFSET 0 0 0)" rpy="$(optenv JACKAL_LASER_3D_RPY 0 0 0)" />
       </xacro:vlp16_mount>
     </xacro:if>
+    <!-- Velodyne HDL-32E -->
     <xacro:if value="${lidar_3d_model == 'hdl32e'}">
-      <xacro:hdl32e_mount
-          parent_link="$(optenv JACKAL_LASER_3D_MOUNT mid)_mount"
-          prefix="$(optenv JACKAL_LASER_3D_MOUNT mid)"
-          topic="$(optenv JACKAL_LASER_3D_TOPIC mid/points)"
-          tower="$(optenv JACKAL_LASER_3D_TOWER 1)">
+      <xacro:hdl32e_mount topic="${topic}" tower="${tower}" prefix="${prefix}" parent_link="${parent_link}" >
         <origin xyz="$(optenv JACKAL_LASER_3D_OFFSET 0 0 0)" rpy="$(optenv JACKAL_LASER_3D_RPY 0 0 0)" />
       </xacro:hdl32e_mount>
     </xacro:if>
   </xacro:if>
-  <!-- If enabled, generate the upgraded Navsat payload (a Novatel Smart6). -->
+  <!--
+    Add a Nav. Sat. By default this is a Novatel Smart6, but can be changed with the
+    JACKAL_NAVSAT_MODEL environment variable. Valid model designations are:
+    - smart6 (default)    :: Novatel Smart6
+    - smart7              :: Novatel Smart7
+  -->
+  <xacro:include filename="$(find jackal_description)/urdf/accessories/novatel_smart6.urdf.xacro" />
+  <xacro:include filename="$(find jackal_description)/urdf/accessories/novatel_smart7.urdf.xacro" />
   <xacro:if value="$(optenv JACKAL_NAVSAT 0)">
+    <xacro:property name="mount" value="$(optenv JACKAL_NAVSAT_MOUNT rear)" />
+    <xacro:property name="tower" value="$(optenv JACKAL_NAVSAT_TOWER 1)" />
+    <xacro:property name="prefix" value="$(optenv JACKAL_NAVSAT_PREFIX ${mount})" />
+    <xacro:property name="parent" value="$(optenv JACKAL_NAVSAT_PARENT ${mount}_mount)" />
     <xacro:property name="navsat_model" value="$(optenv JACKAL_NAVSAT_MODEL smart6)" />
+    <!--- Novotel Smart6 -->
     <xacro:if value="${navsat_model == 'smart6'}">
-      <xacro:include filename="$(find jackal_description)/urdf/accessories/novatel_smart6.urdf.xacro" />
-      <xacro:novatel_smart6 prefix="$(optenv JACKAL_NAVSAT_MOUNT rear)"/>
-    </xacro:if>
+      <xacro:novatel_smart6 prefix="${prefix}"/>
+      <!-- Tower Enabled -->
+      <xacro:if value="${tower}">
+        <xacro:bridge_plate prefix="${prefix}" parent="${parent}" height="$(optenv JACKAL_NAVSAT_HEIGHT 0.1)">
+          <origin xyz="$(optenv JACKAL_NAVSAT_OFFSET 0 0 0)" rpy="$(optenv JACKAL_NAVSAT_RPY 0 0 0)"/>
+        </xacro:bridge_plate>
+        <joint name="${prefix}_navsat_joint" type="fixed">
+          <origin xyz="0 0 0" rpy="0 0 0" />
+          <parent link="${prefix}_bridge" />
+          <child link="${prefix}_navsat" />
+        </joint>
+      </xacro:if>
+      <!-- Tower Disabled -->
+      <xacro:unless value="${tower}">
+        <joint name="${prefix}_navsat_joint" type="fixed">
+          <origin xyz="$(optenv JACKAL_NAVSAT_OFFSET 0 0 0)" rpy="$(optenv JACKAL_NAVSAT_RPY 0 0 0)" />
+          <parent link="${parent}" />
+          <child link="${prefix}_navsat" />
+        </joint>
+      </xacro:unless>
+    </xacro:if>
+    <!-- Novotel Smart7 -->
     <xacro:if value="${navsat_model == 'smart7'}">
-      <xacro:include filename="$(find jackal_description)/urdf/accessories/novatel_smart7.urdf.xacro" />
-      <xacro:novatel_smart7 prefix="$(optenv JACKAL_NAVSAT_MOUNT rear)"/>
-    </xacro:if>
-    <xacro:bridge_plate mount="$(optenv JACKAL_NAVSAT_MOUNT rear)"
-                  height="$(optenv JACKAL_NAVSAT_HEIGHT 0.1)" />
-    <joint name="$(optenv JACKAL_NAVSAT_MOUNT rear)_navsat_joint" type="fixed">
-      <origin xyz="0 0 0" rpy="0 0 0" />
-      <parent link="$(optenv JACKAL_NAVSAT_MOUNT rear)_bridge" />
-      <child link="$(optenv JACKAL_NAVSAT_MOUNT rear)_navsat" />
-    </joint>
+      <xacro:novatel_smart7 prefix="${prefix}"/>
+      <!-- Tower Enabled -->
+      <xacro:if value="${tower}">
+        <xacro:novatel_smart7_stand prefix="${prefix}" parent="${parent}" height="$(optenv JACKAL_NAVSAT_HEIGHT 0.145)">
+          <origin xyz="$(optenv JACKAL_NAVSAT_OFFSET 0 0 0)" rpy="$(optenv JACKAL_NAVSAT_RPY 0 0 0)" />
+        </xacro:novatel_smart7_stand>
+        <joint name="${prefix}_navsat_joint" type="fixed">
+          <origin xyz="0 0 $(optenv JACKAL_NAVSAT_HEIGHT 0.145)" rpy="0 0 0"/>
+          <parent link="${prefix}_navsat_stand" />
+          <child link="${prefix}_navsat" />
+        </joint>
+      </xacro:if>
+      <!-- Tower Disabled -->
+      <xacro:unless value="${tower}">
+        <joint name="${prefix}_navsat_joint" type="fixed">
+          <origin xyz="$(optenv JACKAL_NAVSAT_OFFSET 0 0 0)" rpy="$(optenv JACKAL_NAVSAT_RPY 0 0 0)" />
+          <parent link="${parent}" />
+          <child link="${prefix}_navsat" />
+        </joint>
+      </xacro:unless>
+    </xacro:if>
   </xacro:if>
   <!-- Common camera mounts and accessory URDFs. -->
@@ -115,34 +158,24 @@
   <!-- If enabled, generate the flea3 camera payload with a tilt of 30 degrees. -->
   <xacro:if value="$(optenv JACKAL_FLEA3 0)">
-    <xacro:camera_mount prefix="$(optenv JACKAL_FLEA3_MOUNT front)"
-                       tilt="$(optenv JACKAL_FLEA3_TILT 0.5236)"/>
-    <joint name="$(optenv JACKAL_FLEA3_MOUNT front)_camera_mount_joint" type="fixed">
+    <xacro:property name="name" value="$(optenv JACKAL_FLEA3_NAME front)" />
+    <xacro:property name="tilt" value="$(optenv JACKAL_FLEA3_TILT 0.5236)" />
+    <xacro:property name="tower" value="$(optenv JACKAL_FLEA3_TOWER 1)" />
+    <xacro:property name="mount" value="$(optenv JACKAL_FLEA3_MOUNT front)" />
+    <xacro:property name="prefix" value="$(optenv JACKAL_FLEA3_PREFIX ${mount})" />
+    <xacro:property name="parent" value="$(optenv JACKAL_FLEA3_PARENT ${mount}_mount)" />
+    <xacro:camera_mount prefix="${prefix}" tilt="${tilt}"/>
+    <joint name="${prefix}_camera_mount_joint" type="fixed">
       <origin xyz="$(optenv JACKAL_FLEA3_OFFSET 0 0 0)"
               rpy="$(optenv JACKAL_FLEA3_RPY 0 0 0)" />
-      <parent link="$(optenv JACKAL_FLEA3_MOUNT front)_mount" />
-      <child link="$(optenv JACKAL_FLEA3_MOUNT front)_camera_mount" />
-    </joint>
-    <xacro:pointgrey_flea3 frame="$(optenv JACKAL_FLEA3_MOUNT front)_camera" name="$(optenv JACKAL_FLEA3_NAME front)"
+      <parent link="${parent}" />
+      <child link="${prefix}_camera_mount" />
+    </joint>
+    <xacro:pointgrey_flea3 frame="${prefix}_camera" name="${name}"
       camera_x="0.0754" camera_y="0.029" camera_z="0.029"
       camera_mass="0.085" hfov="1.0471975512" fps="60" width="640" height="512"/>
-    <joint name="$(optenv JACKAL_FLEA3_MOUNT front)_camera_bracket_joint" type="fixed">
+    <joint name="${prefix}_camera_bracket_joint" type="fixed">
       <origin xyz="0.020 0 0.0245" rpy="0 0 0" />
-      <parent link="$(optenv JACKAL_FLEA3_MOUNT front)_camera_beam" />
-      <child link="$(optenv JACKAL_FLEA3_MOUNT front)_camera" />
-    </joint>
-  </xacro:if>
-  <xacro:if value="$(optenv JACKAL_BLACKFLYS 0)">
-    <!-- Include Mount (default to lockmount) -->
-    <xacro:include filename="$(find lockmount_description)/urdf/lockmount.urdf.xacro" />
-    <xacro:lockmount prefix="$(optenv JACKAL_BLACKFLYS_PREFIX front)_camera" parent_link="$(optenv JACKAL_BLACKFLYS_PARENT front_mount)" angle="$(optenv JACKAL_BLACKFLYS_TILT 0)">
-      <origin xyz="$(optenv JACKAL_BLACKFLYS_OFFSET)" rpy="$(optenv JACKAL_BLACKFLYS_RPY)" />
-    </xacro:lockmount>
-    <!-- Include Flir BlackflyS -->
-    <xacro:include filename="$(find flir_camera_description)/urdf/flir_blackflys.urdf.xacro" />
-    <xacro:flir_blackflys frame="$(optenv JACKAL_BLACKFLYS_PREFIX front)_camera" />
-    <joint name="$(optenv JACKAL_BLACKFLYS_PREFIX front)_camera_mount_camera_joint" type="fixed">
-      <origin xyz="0 0 0" rpy="0 0 0" />
-      <parent link="$(optenv JACKAL_BLACKFLYS_PREFIX front)_camera_mount_link"/>
-      <child link="$(optenv JACKAL_BLACKFLYS_PREFIX front)_camera"/>
+      <parent link="${prefix}_camera_beam" />
+      <child link="${prefix}_camera" />
     </joint>
   </xacro:if>
@@ -196,4 +229,5 @@
     </joint>
   </xacro:if>
+  <!-- Fender Accessories -->
   <xacro:if value="$(optenv JACKAL_FRONT_ACCESSORY_FENDER 0)">
     <xacro:include filename="$(find jackal_description)/urdf/accessories/hokuyo_ust10.urdf.xacro" />

Commit message: Updated BB2 to allow enabling/disabling mount

File: jackal_description/urdf/accessories.urdf.xacro (robot description, xacro)
@@ -152,4 +152,10 @@
     </xacro:if>
   </xacro:if>
+  <!--
+    Add Cameras.
+    - JACKAL_FLEA3
+    - JACKAL_STEREO_FLEA3
+    - JACKAL_BB2
+  -->
   <!-- Common camera mounts and accessory URDFs. -->
   <xacro:include filename="$(find jackal_description)/urdf/accessories/camera_mount.urdf.xacro" />
@@ -164,19 +170,31 @@
     <xacro:property name="prefix" value="$(optenv JACKAL_FLEA3_PREFIX ${mount})" />
     <xacro:property name="parent" value="$(optenv JACKAL_FLEA3_PARENT ${mount}_mount)" />
-    <xacro:camera_mount prefix="${prefix}" tilt="${tilt}"/>
-    <joint name="${prefix}_camera_mount_joint" type="fixed">
-      <origin xyz="$(optenv JACKAL_FLEA3_OFFSET 0 0 0)"
-              rpy="$(optenv JACKAL_FLEA3_RPY 0 0 0)" />
-      <parent link="${parent}" />
-      <child link="${prefix}_camera_mount" />
-    </joint>
     <xacro:pointgrey_flea3 frame="${prefix}_camera" name="${name}"
       camera_x="0.0754" camera_y="0.029" camera_z="0.029"
       camera_mass="0.085" hfov="1.0471975512" fps="60" width="640" height="512"/>
-    <joint name="${prefix}_camera_bracket_joint" type="fixed">
-      <origin xyz="0.020 0 0.0245" rpy="0 0 0" />
-      <parent link="${prefix}_camera_beam" />
-      <child link="${prefix}_camera" />
-    </joint>
+    <!-- Mount Enabled -->
+    <xacro:if value="${tower}">
+      <xacro:camera_mount prefix="${prefix}" tilt="${tilt}"/>
+      <joint name="${prefix}_camera_mount_joint" type="fixed">
+        <origin xyz="$(optenv JACKAL_FLEA3_OFFSET 0 0 0)"
+                rpy="$(optenv JACKAL_FLEA3_RPY 0 0 0)" />
+        <parent link="${parent}" />
+        <child link="${prefix}_camera_mount" />
+      </joint>
+      <joint name="${prefix}_camera_bracket_joint" type="fixed">
+        <origin xyz="0.020 0 0.0245" rpy="0 0 0" />
+        <parent link="${prefix}_camera_beam" />
+        <child link="${prefix}_camera" />
+      </joint>
+    </xacro:if>
+    <!-- Mount Disabled -->
+    <xacro:unless value="${tower}">
+      <joint name="${prefix}_camera_bracket_joint" type="fixed">
+        <origin xyz="$(optenv JACKAL_FLEA3_OFFSET 0 0 0.0145)"
+                rpy="$(optenv JACKAL_FLEA3_RPY 0 0 0)" />
+        <parent link="${parent}" />
+        <child link="${prefix}_camera" />
+      </joint>
+    </xacro:unless>
   </xacro:if>
   <xacro:include filename="$(find jackal_description)/urdf/accessories/stereo_camera_mount.urdf.xacro" />
@@ -184,27 +202,33 @@
   <!-- Disabled temporarily due to metapackage issue. -->
   <xacro:if value="$(optenv JACKAL_STEREO_FLEA3 0)">
-    <xacro:stereo_camera_mount prefix="$(optenv JACKAL_FLEA3_MOUNT front)"
-                       tilt="$(optenv JACKAL_FLEA3_TILT 0.5236)"/>
-    <joint name="$(optenv JACKAL_FLEA3_MOUNT front)_stereo_camera_mount_joint" type="fixed">
+    <xacro:property name="tilt" value="$(optenv JACKAL_FLEA3_TILT 0.5236)"/>
+    <xacro:property name="mount" value="$(optenv JACKAL_FLEA3_MOUNT front)"/>
+    <xacro:property name="prefix" value="$(optenv JACKAL_FLEA3_PREFIX ${mount})"/>
+    <xacro:property name="parent" value="$(optenv JACKAL_FLEA3_PARENT ${mount}_mount)"/>
+    <xacro:property name="left_name" value="$(optenv JACKAL_FLEA3_LEFT_NAME front/left)"/>
+    <xacro:property name="right_name" value="$(optenv JACKAL_FLEA3_RIGHT_NAME front/right)"/>
+    <xacro:property name="separation" value="$(optenv JACKAL_STEREO_SEPERATION 0.16)"/>
+    <xacro:stereo_camera_mount prefix="${prefix}" tilt="${tilt}"/>
+    <joint name="${prefix}_stereo_camera_mount_joint" type="fixed">
       <origin xyz="$(optenv JACKAL_FLEA3_OFFSET 0 0 0)"
               rpy="$(optenv JACKAL_FLEA3_RPY 0 0 0)" />
-      <parent link="$(optenv JACKAL_FLEA3_MOUNT front)_mount" />
-      <child link="$(optenv JACKAL_FLEA3_MOUNT front)_stereo_camera_mount" />
+      <parent link="${parent}" />
+      <child link="${prefix}_stereo_camera_mount" />
     </joint>
-    <xacro:pointgrey_flea3 frame="$(optenv JACKAL_FLEA3_MOUNT front)_left_camera" name="$(optenv JACKAL_FLEA3_LEFT_NAME front/left)"
+    <xacro:pointgrey_flea3 frame="${prefix}_left_camera" name="${left_name}"
       camera_x="0.0754" camera_y="0.029" camera_z="0.029"
       camera_mass="0.085" hfov="1.0471975512" fps="60" width="640" height="512"/>
-    <joint name="$(optenv JACKAL_FLEA3_MOUNT front)_left_stereo_camera_bracket_joint" type="fixed">
-      <origin xyz="0.015 $(optenv JACKAL_STEREO_SEPERATION 0.16) 0.0599" rpy="0 0 0" />
-      <parent link="$(optenv JACKAL_FLEA3_MOUNT front)_stereo_camera_beam" />
-      <child link="$(optenv JACKAL_FLEA3_MOUNT front)_left_camera" />
+    <joint name="${prefix}_left_stereo_camera_bracket_joint" type="fixed">
+      <origin xyz="0.015 ${separation} 0.0599" rpy="0 0 0" />
+      <parent link="${prefix}_stereo_camera_beam" />
+      <child link="${prefix}_left_camera" />
     </joint>
-    <xacro:pointgrey_flea3 frame="$(optenv JACKAL_FLEA3_MOUNT front)_right_camera" name="$(optenv JACKAL_FLEA3_RIGHT_NAME front/right)"
+    <xacro:pointgrey_flea3 frame="${prefix}_right_camera" name="${right_name}"
       camera_x="0.0754" camera_y="0.029" camera_z="0.029"
       camera_mass="0.085" hfov="1.0471975512" fps="60" width="640" height="512"/>
-    <joint name="$(optenv JACKAL_FLEA3_MOUNT front)_right_stereo_camera_bracket_joint" type="fixed">
-      <origin xyz="0.015 -$(optenv JACKAL_STEREO_SEPERATION 0.16) 0.0599" rpy="0 0 0" />
-      <parent link="$(optenv JACKAL_FLEA3_MOUNT front)_stereo_camera_beam" />
-      <child link="$(optenv JACKAL_FLEA3_MOUNT front)_right_camera" />
+    <joint name="${prefix}_right_stereo_camera_bracket_joint" type="fixed">
+      <origin xyz="0.015 -${separation} 0.0599" rpy="0 0 0" />
+      <parent link="${prefix}_stereo_camera_beam" />
+      <child link="${prefix}_right_camera" />
     </joint>
   </xacro:if>
@@ -214,18 +238,34 @@
   <!-- Disabled temporarily due to metapackage issue. -->
   <xacro:if value="$(optenv JACKAL_BB2 0)">
-    <xacro:camera_mount prefix="$(optenv JACKAL_BB2_MOUNT front)"
-                        tilt="$(optenv JACKAL_BB2_TILT 0)"/>
-    <joint name="$(optenv JACKAL_BB2_MOUNT front)_camera_mount_joint" type="fixed">
-      <origin xyz="$(optenv JACKAL_BB2_OFFSET 0 0 0)"
-              rpy="$(optenv JACKAL_BB2_RPY 0 0 0)" />
-      <parent link="$(optenv JACKAL_BB2_MOUNT front)_mount" />
-      <child link="$(optenv JACKAL_BB2_MOUNT front)_camera_mount" />
-    </joint>
-    <xacro:BB2-08S2C-38 frame="$(optenv JACKAL_BB2_MOUNT front)_camera" name="$(optenv JACKAL_BB2_NAME front)" />
-    <joint name="$(optenv JACKAL_BB2_MOUNT front)_camera_bracket_joint" type="fixed">
-      <origin xyz="0.007 0 0.02450" rpy="0 0 0" />
-      <parent link="$(optenv JACKAL_BB2_MOUNT front)_camera_beam" />
-      <child link="$(optenv JACKAL_BB2_MOUNT front)_camera" />
-    </joint>
+    <xacro:property name="tilt" value="$(optenv JACKAL_BB2_TILT 0)" />
+    <xacro:property name="name" value="$(optenv JACKAL_BB2_NAME front)" />
+    <xacro:property name="tower" value="$(optenv JACKAL_BB2_TOWER 1)"/>
+    <xacro:property name="mount" value="$(optenv JACKAL_BB2_MOUNT front)" />
+    <xacro:property name="prefix" value="$(optenv JACKAL_BB2_PREFIX ${mount})"/>
+    <xacro:property name="parent" value="$(optenv JACKAL_BB2_PARENT ${mount}_mount)"/>
+    <xacro:BB2-08S2C-38 frame="${prefix}_camera" name="${name}" />
+    <!-- Mount Enabled -->
+    <xacro:if value="${tower}">
+      <xacro:camera_mount prefix="${prefix}" tilt="${tilt}"/>
+      <joint name="${prefix}_camera_mount_joint" type="fixed">
+        <origin xyz="$(optenv JACKAL_BB2_OFFSET 0 0 0)"
+                rpy="$(optenv JACKAL_BB2_RPY 0 0 0)" />
+        <parent link="${parent}" />
+        <child link="${prefix}_camera_mount" />
+      </joint>
+      <joint name="${prefix}_camera_bracket_joint" type="fixed">
+        <origin xyz="0.007 0 0.02450" rpy="0 0 0" />
+        <parent link="${prefix}_camera_beam" />
+        <child link="${prefix}_camera" />
+      </joint>
+    </xacro:if>
+    <xacro:unless value="${tower}">
+      <joint name="${prefix}_camera_joint" type="fixed">
+        <origin xyz="$(optenv JACKAL_BB2_OFFSET 0 0 0.018)"
+                rpy="$(optenv JACKAL_BB2_RPY 0 0 0)" />
+        <parent link="${parent}" />
+        <child link="${prefix}_camera" />
+      </joint>
+    </xacro:unless>
   </xacro:if>
   <!-- Fender Accessories -->
