Commit message: Added LMS1xx disable mount and fixed typos

File: jackal_description/urdf/accessories.urdf.xacro (robot description, xacro)
@@ -13,4 +13,6 @@
   <!-- This optional plate mounts both the upgraded GPS and the Velodyne 3D LIDAR. -->
   <xacro:include filename="$(find jackal_description)/urdf/accessories/bridge_plate.urdf.xacro" />
+  <!-- 2D Lidars -->
+  <xacro:include filename="$(find lms1xx)/urdf/sick_lms1xx.urdf.xacro" />
   <xacro:include filename="$(find jackal_description)/urdf/accessories/sick_lms1xx_mount.urdf.xacro" />
   <xacro:include filename="$(find jackal_description)/urdf/accessories/hokuyo_ust10.urdf.xacro" />
@@ -29,15 +31,27 @@
     <xacro:property name="tower" value="$(optenv JACKAL_LASER_TOWER 1)" />
     <xacro:property name="prefix" value="$(optenv JACKAL_LASER_PREFIX ${mount})" />
-    <xacro:property name="parent_link" value="$(optenv JACKAL_LASER_PARENT ${mount}_mount)" />
+    <xacro:property name="parent" value="$(optenv JACKAL_LASER_PARENT ${mount}_mount)" />
     <xacro:property name="lidar_model" value="$(optenv JACKAL_LASER_MODEL lms1xx)" />
     <!-- SICK LMS1xx -->
     <xacro:if value="${lidar_model == 'lms1xx'}">
-      <xacro:sick_lms1xx_mount  topic="${topic}" prefix="${prefix}" parent_link="${parent_link}">
-        <origin xyz="$(optenv JACKAL_LASER_OFFSET 0 0 0)" rpy="$(optenv JACKAL_LASER_RPY 0 0 0)" />
-      </xacro:sick_lms1xx_mount>
+      <!-- Mount Enabled -->
+      <xacro:if value="${tower}">
+        <xacro:sick_lms1xx_mount topic="${topic}" prefix="${prefix}" parent_link="${parent}">
+          <origin xyz="$(optenv JACKAL_LASER_OFFSET 0 0 0)" rpy="$(optenv JACKAL_LASER_RPY 0 0 0)" />
+        </xacro:sick_lms1xx_mount>
+      </xacro:if>
+      <!-- Mount Disabled -->
+      <xacro:unless value="${tower}">
+        <xacro:sick_lms1xx frame="${prefix}_laser" topic="${topic}" />
+        <joint name="${prefix}_laser_joint" type="fixed">
+          <origin xyz="$(optenv JACKAL_LASER_OFFSET 0 0 0.116)" rpy="$(optenv JACKAL_LASER_RPY 0 0 0)"/>
+          <parent link="${parent}"/>
+          <child link="${prefix}_laser"/>
+        </joint>
+      </xacro:unless>
     </xacro:if>
     <!-- Hokuyo UST10 -->
     <xacro:if value="${lidar_model == 'ust10'}">
-      <xacro:hokuyo_ust10_mount topic="${topic}" prefix="${prefix}" parent_link="${parent_link}">
+      <xacro:hokuyo_ust10_mount topic="${topic}" prefix="${prefix}" parent_link="${parent}">
         <origin xyz="$(optenv JACKAL_LASER_OFFSET 0 0 0)" rpy="$(optenv JACKAL_LASER_RPY 0 0 0)" />
       </xacro:hokuyo_ust10_mount>
@@ -50,15 +64,27 @@
     <xacro:property name="tower" value="$(optenv JACKAL_LASER_SECONDARY_TOWER 1)" />
     <xacro:property name="prefix" value="$(optenv JACKAL_LASER_SECONDARY_PREFIX ${mount})" />
-    <xacro:property name="parent_link" value="$(optenv JACKAL_LASER_SECONDARY_PARENT ${mount}_mount)" />
+    <xacro:property name="parent" value="$(optenv JACKAL_LASER_SECONDARY_PARENT ${mount}_mount)" />
     <xacro:property name="lidar_model" value="$(optenv JACKAL_LASER_SECONDARY_MODEL lms1xx)" />
-    <!-- SICK LM1xx -->
+    <!-- SICK LMS1xx -->
     <xacro:if value="${lidar_model == 'lms1xx'}">
-      <xacro:sick_lms1xx_mount  topic="${topic}" prefix="${prefix}" parent_link="${parent_link}">
-         <origin xyz="$(optenv JACKAL_LASER_SECONDARY_OFFSET 0 0 0)" rpy="$(optenv JACKAL_LASER_SECONDARY_RPY 0 0 3.14159)" />
-       </xacro:sick_lms1xx_mount>
+      <!-- Mount Enabled -->
+      <xacro:if value="${tower}">
+        <xacro:sick_lms1xx_mount topic="${topic}" prefix="${prefix}" parent_link="${parent}">
+          <origin xyz="$(optenv JACKAL_LASER_SECONDARY_OFFSET 0 0 0)" rpy="$(optenv JACKAL_LASER_SECONDARY_RPY 0 0 3.14159)" />
+        </xacro:sick_lms1xx_mount>
+      </xacro:if>
+      <!-- Mount Disabled -->
+      <xacro:unless value="${tower}">
+        <xacro:sick_lms1xx frame="${prefix}_laser" topic="${topic}" />
+        <joint name="${prefix}_laser_joint" type="fixed">
+          <origin xyz="$(optenv JACKAL_LASER_SECONDARY_OFFSET 0 0 0.116)" rpy="$(optenv JACKAL_LASER_SECONDARY_RPY 0 0 3.14159)"/>
+          <parent link="${parent}"/>
+          <child link="${prefix}_laser"/>
+        </joint>
+      </xacro:unless>
     </xacro:if>
     <!-- Hokuyo UST10 -->
     <xacro:if value="${lidar_model == 'ust10'}">
-      <xacro:hokuyo_ust10_mount topic="${topic}" prefix="${prefix}" parent_link="${parent_link}">
+      <xacro:hokuyo_ust10_mount topic="${topic}" prefix="${prefix}" parent_link="${parent}">
         <origin xyz="$(optenv JACKAL_LASER_SECONDARY_OFFSET 0 0 0)" rpy="$(optenv JACKAL_LASER_SECONDARY_RPY 0 0 3.14159)" />
       </xacro:hokuyo_ust10_mount>
@@ -76,9 +102,9 @@
     <xacro:property name="tower" value="$(optenv JACKAL_LASER_3D_TOWER 1)" />
     <xacro:property name="prefix" value="$(optenv JACKAL_LASER_PREFIX ${mount})" />
-    <xacro:property name="parent_link" value="$(optenv JACKAL_LASER_PARENT ${mount}_mount)" />
+    <xacro:property name="parent" value="$(optenv JACKAL_LASER_PARENT ${mount}_mount)" />
     <xacro:property name="lidar_3d_model" value="$(optenv JACKAL_LASER_3D_MODEL vlp16)" />
     <!-- Velodyne VLP16 -->
     <xacro:if value="${lidar_3d_model == 'vlp16'}">
-      <xacro:vlp16_mount topic="${topic}" tower="${tower}" prefix="${prefix}" parent_link="${parent_link}" >
+      <xacro:vlp16_mount topic="${topic}" tower="${tower}" prefix="${prefix}" parent_link="${parent}" >
         <origin xyz="$(optenv JACKAL_LASER_3D_OFFSET 0 0 0)" rpy="$(optenv JACKAL_LASER_3D_RPY 0 0 0)" />
       </xacro:vlp16_mount>
@@ -86,5 +112,5 @@
     <!-- Velodyne HDL-32E -->
     <xacro:if value="${lidar_3d_model == 'hdl32e'}">
-      <xacro:hdl32e_mount topic="${topic}" tower="${tower}" prefix="${prefix}" parent_link="${parent_link}" >
+      <xacro:hdl32e_mount topic="${topic}" tower="${tower}" prefix="${prefix}" parent_link="${parent}" >
         <origin xyz="$(optenv JACKAL_LASER_3D_OFFSET 0 0 0)" rpy="$(optenv JACKAL_LASER_3D_RPY 0 0 0)" />
       </xacro:hdl32e_mount>
@@ -260,4 +286,5 @@
       </joint>
     </xacro:if>
+    <!-- Mount Disabled -->
     <xacro:unless value="${tower}">
       <joint name="${prefix}_camera_joint" type="fixed">

Commit message: Fixed typo LASER->LASER_3D

File: jackal_description/urdf/accessories.urdf.xacro (robot description, xacro)
@@ -28,5 +28,5 @@
   <xacro:if value="$(optenv JACKAL_LASER 0)">
     <xacro:property name="mount" value="$(optenv JACKAL_LASER_MOUNT front)" />
-    <xacro:property name="topic" value="$(optenv JACKAL_LASER_TOPIC ${mount}/scan)" />
+    <xacro:property name="topic" value="$(optenv JACKAL_LASER_TOPIC front/scan)" />
     <xacro:property name="tower" value="$(optenv JACKAL_LASER_TOWER 1)" />
     <xacro:property name="prefix" value="$(optenv JACKAL_LASER_PREFIX ${mount})" />
@@ -61,5 +61,5 @@
   <xacro:if value="$(optenv JACKAL_LASER_SECONDARY 0)">
     <xacro:property name="mount" value="$(optenv JACKAL_LASER_SECONDARY_MOUNT rear)" />
-    <xacro:property name="topic" value="$(optenv JACKAL_LASER_SECONDARY_TOPIC ${mount}/scan)" />
+    <xacro:property name="topic" value="$(optenv JACKAL_LASER_SECONDARY_TOPIC rear/scan)" />
     <xacro:property name="tower" value="$(optenv JACKAL_LASER_SECONDARY_TOWER 1)" />
     <xacro:property name="prefix" value="$(optenv JACKAL_LASER_SECONDARY_PREFIX ${mount})" />
@@ -99,8 +99,8 @@
   <xacro:if value="$(optenv JACKAL_LASER_3D 0)">
     <xacro:property name="mount" value="$(optenv JACKAL_LASER_3D_MOUNT mid)" />
-    <xacro:property name="topic" value="$(optenv JACKAL_LASER_3D_TOPIC ${mount}/points)" />
+    <xacro:property name="topic" value="$(optenv JACKAL_LASER_3D_TOPIC mid/points)" />
     <xacro:property name="tower" value="$(optenv JACKAL_LASER_3D_TOWER 1)" />
-    <xacro:property name="prefix" value="$(optenv JACKAL_LASER_PREFIX ${mount})" />
-    <xacro:property name="parent" value="$(optenv JACKAL_LASER_PARENT ${mount}_mount)" />
+    <xacro:property name="prefix" value="$(optenv JACKAL_LASER_3D_PREFIX ${mount})" />
+    <xacro:property name="parent" value="$(optenv JACKAL_LASER_3D_PARENT ${mount}_mount)" />
     <xacro:property name="lidar_3d_model" value="$(optenv JACKAL_LASER_3D_MODEL vlp16)" />
     <!-- Velodyne VLP16 -->

Commit message: Added base_links s.t. all XYZ/RPY defaults are all zero

File: jackal_description/urdf/accessories.urdf.xacro (robot description, xacro)
@@ -44,7 +44,13 @@
       <xacro:unless value="${tower}">
         <xacro:sick_lms1xx frame="${prefix}_laser" topic="${topic}" />
+        <link name="${prefix}_laser_base"/>
+        <joint name="${prefix}_laser_base_joint" type="fixed">
+          <origin xyz="$(optenv JACKAL_LASER_OFFSET 0 0 0)" rpy="$(optenv JACKAL_LASER_RPY 0 0 0)"/>
+          <parent link="${parent}"/>
+          <child link="${prefix}_laser_base"/>
+        </joint>
         <joint name="${prefix}_laser_joint" type="fixed">
-          <origin xyz="$(optenv JACKAL_LASER_OFFSET 0 0 0.116)" rpy="$(optenv JACKAL_LASER_RPY 0 0 0)"/>
-          <parent link="${parent}"/>
+          <origin xyz="0 0 0.116" rpy="0 0 0"/>
+          <parent link="${prefix}_laser_base"/>
           <child link="${prefix}_laser"/>
         </joint>
@@ -77,7 +83,13 @@
       <xacro:unless value="${tower}">
         <xacro:sick_lms1xx frame="${prefix}_laser" topic="${topic}" />
+        <link name="${prefix}_laser_base"/>
+        <joint name="${prefix}_laser_base_joint" type="fixed">
+          <origin xyz="$(optenv JACKAL_LASER_SECONDARY_OFFSET 0 0 0)" rpy="$(optenv JACKAL_LASER_SECONDARY_RPY 0 0 3.14159)"/>
+          <parent link="${parent}"/>
+          <child link="${prefix}_laser_base"/>
+        </joint>
         <joint name="${prefix}_laser_joint" type="fixed">
-          <origin xyz="$(optenv JACKAL_LASER_SECONDARY_OFFSET 0 0 0.116)" rpy="$(optenv JACKAL_LASER_SECONDARY_RPY 0 0 3.14159)"/>
-          <parent link="${parent}"/>
+          <origin xyz="0 0 0.116" rpy="0 0 0"/>
+          <parent link="${prefix}_laser_base"/>
           <child link="${prefix}_laser"/>
         </joint>
@@ -215,8 +227,15 @@
     <!-- Mount Disabled -->
     <xacro:unless value="${tower}">
-      <joint name="${prefix}_camera_bracket_joint" type="fixed">
-        <origin xyz="$(optenv JACKAL_FLEA3_OFFSET 0 0 0.0145)"
+      <link name="${prefix}_camera_base"/>
+      <joint name="${prefix}_camera_base_joint" type="fixed">
+        <origin xyz="$(optenv JACKAL_FLEA3_OFFSET 0 0 0)"
                 rpy="$(optenv JACKAL_FLEA3_RPY 0 0 0)" />
         <parent link="${parent}" />
+        <child link="${prefix}_camera_base" />
+      </joint>
+      <joint name="${prefix}_camera_joint" type="fixed">
+        <origin xyz="0 0 0.0145"
+                rpy="0 0 0" />
+        <parent link="${prefix}_camera_base" />
         <child link="${prefix}_camera" />
       </joint>
@@ -287,8 +306,14 @@
     <!-- Mount Disabled -->
     <xacro:unless value="${tower}">
-      <joint name="${prefix}_camera_joint" type="fixed">
-        <origin xyz="$(optenv JACKAL_BB2_OFFSET 0 0 0.018)"
+      <link name="${prefix}_camera_base" type="fixed"/>
+      <joint name="${prefix}_camera_base_joint" type="fixed">
+        <origin xyz="$(optenv JACKAL_BB2_OFFSET 0 0 0)"
                 rpy="$(optenv JACKAL_BB2_RPY 0 0 0)" />
         <parent link="${parent}" />
+        <child link="${prefix}_camera_base" />
+      </joint>
+      <joint name="${prefix}_camera_joint" type="fixed">
+        <origin xyz="0 0 0.018" rpy="0 0 0" />
+        <parent link="${prefix}_camera_base" />
         <child link="${prefix}_camera" />
       </joint>

Commit message: Added Wibotic mesh and STL

File: jackal_description/urdf/accessories.urdf.xacro (robot description, xacro)
@@ -205,4 +205,26 @@
     </xacro:if>
   </xacro:if>
+  <!-- Bumper Accessories -->
+  <xacro:if value="$(optenv JACKAL_WIBOTIC_BUMPER 0)">
+    <link name="wibotic_bumper">
+      <visual>
+        <geometry>
+          <mesh filename="package://jackal_description/meshes/wibotic_bumper.stl" />
+        </geometry>
+        <material name="dark_grey" />
+      </visual>
+      <collision>
+        <geometry>
+          <box size="0.115 0.25 0.145"/>
+        </geometry>
+        <origin xyz="-0.017575 0 0.0575" rpy="0 0 0"/>
+      </collision>
+    </link>
+    <joint name="wibotic_bumper_joint" type="fixed">
+      <origin xyz="0.285 0 0.07455" rpy="0 0 0"/>
+      <parent link="base_link"/>
+      <child link="wibotic_bumper"/>
+    </joint>
+  </xacro:if>
   <xacro:if value="$(optenv JACKAL_ARK_ENCLOSURE 0)">
     <link name="ark_enclosure_link">

Commit message: Updated SICK LMS1XX mount and NAVSAT mount

File: jackal_description/urdf/accessories.urdf.xacro (robot description, xacro)
@@ -188,10 +188,10 @@
       <!-- Tower Enabled -->
       <xacro:if value="${tower}">
-        <xacro:novatel_smart7_stand prefix="${prefix}" parent="${parent}" height="$(optenv JACKAL_NAVSAT_HEIGHT 0.145)">
-          <origin xyz="$(optenv JACKAL_NAVSAT_OFFSET 0 0 0)" rpy="$(optenv JACKAL_NAVSAT_RPY 0 0 0)" />
-        </xacro:novatel_smart7_stand>
+        <xacro:bridge_plate prefix="${prefix}" parent="${parent}" height="$(optenv JACKAL_NAVSAT_HEIGHT 0.1)">
+          <origin xyz="$(optenv JACKAL_NAVSAT_OFFSET 0 0 0)" rpy="$(optenv JACKAL_NAVSAT_RPY 0 0 0)"/>
+        </xacro:bridge_plate>
         <joint name="${prefix}_navsat_joint" type="fixed">
-          <origin xyz="0 0 $(optenv JACKAL_NAVSAT_HEIGHT 0.145)" rpy="0 0 0"/>
-          <parent link="${prefix}_navsat_stand" />
+          <origin xyz="0 0 0" rpy="0 0 0" />
+          <parent link="${prefix}_bridge" />
           <child link="${prefix}_navsat" />
         </joint>

File: jackal_description/urdf/accessories/sick_lms1xx_mount.urdf.xacro (robot description, xacro)
@@ -46,5 +46,5 @@
     <joint name="${prefix}_laser_joint" type="fixed">
       <!-- This offset is from the base of the bracket to the LIDAR's focal point. -->
-      <origin xyz="0 0 0.149" rpy="0 0 0" />
+      <origin xyz="0.04 0 0.066" rpy="3.141592 0 0" />
       <parent link="${prefix}_laser_mount" />
       <child link="${prefix}_laser" />

Commit message: Maintained backward compatibility with LMS1xx standard upright poisition by adding mount types

File: jackal_description/urdf/accessories.urdf.xacro (robot description, xacro)
@@ -15,5 +15,6 @@
   <!-- 2D Lidars -->
   <xacro:include filename="$(find lms1xx)/urdf/sick_lms1xx.urdf.xacro" />
-  <xacro:include filename="$(find jackal_description)/urdf/accessories/sick_lms1xx_mount.urdf.xacro" />
+  <xacro:include filename="$(find jackal_description)/urdf/accessories/sick_lms1xx_inverted_mount.urdf.xacro" />
+  <xacro:include filename="$(find jackal_description)/urdf/accessories/sick_lms1xx_upright_mount.urdf.xacro" />
   <xacro:include filename="$(find jackal_description)/urdf/accessories/hokuyo_ust10.urdf.xacro" />
   <xacro:include filename="$(find jackal_description)/urdf/accessories/vlp16_mount.urdf.xacro" />
@@ -50,11 +51,19 @@
     <xacro:property name="parent" value="$(optenv JACKAL_LASER_PARENT ${mount}_mount)" />
     <xacro:property name="lidar_model" value="$(optenv JACKAL_LASER_MODEL lms1xx)" />
+    <xacro:property name="mount_type" value="$(optenv JACKAL_LASER_MOUNT_TYPE upright)" />
     <!-- SICK LMS1xx -->
     <xacro:if value="${lidar_model == 'lms1xx'}">
       <!-- Mount Enabled -->
       <xacro:if value="${tower}">
-        <xacro:sick_lms1xx_mount topic="${topic}" prefix="${prefix}" parent_link="${parent}">
-          <origin xyz="$(optenv JACKAL_LASER_OFFSET 0 0 0)" rpy="$(optenv JACKAL_LASER_RPY 0 0 0)" />
-        </xacro:sick_lms1xx_mount>
+        <xacro:if value="${mount_type == 'upright'}">
+          <xacro:sick_lms1xx_upright_mount topic="${topic}" prefix="${prefix}" parent_link="${parent}">
+            <origin xyz="$(optenv JACKAL_LASER_OFFSET 0 0 0)" rpy="$(optenv JACKAL_LASER_RPY 0 0 0)" />
+          </xacro:sick_lms1xx_upright_mount>
+        </xacro:if>
+        <xacro:if value="${mount_type == 'inverted'}">
+          <xacro:sick_lms1xx_inverted_mount topic="${topic}" prefix="${prefix}" parent_link="${parent}">
+            <origin xyz="$(optenv JACKAL_LASER_OFFSET 0 0 0)" rpy="$(optenv JACKAL_LASER_RPY 0 0 0)" />
+          </xacro:sick_lms1xx_inverted_mount>
+        </xacro:if>
       </xacro:if>
       <!-- Mount Disabled -->

File: jackal_description/urdf/accessories/sick_lms1xx_inverted_mount.urdf.xacro (robot description, xacro)
@@ -27,5 +27,5 @@
 <robot xmlns:xacro="http://www.ros.org/wiki/xacro">
   <xacro:include filename="$(find lms1xx)/urdf/sick_lms1xx.urdf.xacro" />
-  <xacro:macro name="sick_lms1xx_mount" params="prefix topic parent_link *origin">
+  <xacro:macro name="sick_lms1xx_inverted_mount" params="prefix topic parent_link *origin">
     <xacro:sick_lms1xx frame="${prefix}_laser" topic="${topic}" />
     <joint name="${prefix}_laser_mount_joint" type="fixed">
@@ -39,5 +39,5 @@
         <geometry>
           <!-- Origin of this mesh is the base of the bracket. -->
-          <mesh filename="package://jackal_description/meshes/sick-lms1xx-bracket.stl" />
+          <mesh filename="package://jackal_description/meshes/sick-lms1xx-inverted-bracket.stl" />
         </geometry>
         <material name="dark_grey" />

Commit message: Maintained backward compatibility with LMS1xx standard upright poisition by adding mount types

File: jackal_description/urdf/accessories.urdf.xacro (robot description, xacro)
@@ -15,5 +15,6 @@
   <!-- 2D Lidars -->
   <xacro:include filename="$(find lms1xx)/urdf/sick_lms1xx.urdf.xacro" />
-  <xacro:include filename="$(find jackal_description)/urdf/accessories/sick_lms1xx_mount.urdf.xacro" />
+  <xacro:include filename="$(find jackal_description)/urdf/accessories/sick_lms1xx_inverted_mount.urdf.xacro" />
+  <xacro:include filename="$(find jackal_description)/urdf/accessories/sick_lms1xx_upright_mount.urdf.xacro" />
   <xacro:include filename="$(find jackal_description)/urdf/accessories/hokuyo_ust10.urdf.xacro" />
   <xacro:include filename="$(find jackal_description)/urdf/accessories/vlp16_mount.urdf.xacro" />
@@ -33,11 +34,19 @@
     <xacro:property name="parent" value="$(optenv JACKAL_LASER_PARENT ${mount}_mount)" />
     <xacro:property name="lidar_model" value="$(optenv JACKAL_LASER_MODEL lms1xx)" />
+    <xacro:property name="mount_type" value="$(optenv JACKAL_LASER_MOUNT_TYPE upright)" />
     <!-- SICK LMS1xx -->
     <xacro:if value="${lidar_model == 'lms1xx'}">
       <!-- Mount Enabled -->
       <xacro:if value="${tower}">
-        <xacro:sick_lms1xx_mount topic="${topic}" prefix="${prefix}" parent_link="${parent}">
-          <origin xyz="$(optenv JACKAL_LASER_OFFSET 0 0 0)" rpy="$(optenv JACKAL_LASER_RPY 0 0 0)" />
-        </xacro:sick_lms1xx_mount>
+        <xacro:if value="${mount_type == 'upright'}">
+          <xacro:sick_lms1xx_upright_mount topic="${topic}" prefix="${prefix}" parent_link="${parent}">
+            <origin xyz="$(optenv JACKAL_LASER_OFFSET 0 0 0)" rpy="$(optenv JACKAL_LASER_RPY 0 0 0)" />
+          </xacro:sick_lms1xx_upright_mount>
+        </xacro:if>
+        <xacro:if value="${mount_type == 'inverted'}">
+          <xacro:sick_lms1xx_inverted_mount topic="${topic}" prefix="${prefix}" parent_link="${parent}">
+            <origin xyz="$(optenv JACKAL_LASER_OFFSET 0 0 0)" rpy="$(optenv JACKAL_LASER_RPY 0 0 0)" />
+          </xacro:sick_lms1xx_inverted_mount>
+        </xacro:if>
       </xacro:if>
       <!-- Mount Disabled -->

File: jackal_description/urdf/accessories/sick_lms1xx_inverted_mount.urdf.xacro (robot description, xacro)
@@ -27,5 +27,5 @@
 <robot xmlns:xacro="http://www.ros.org/wiki/xacro">
   <xacro:include filename="$(find lms1xx)/urdf/sick_lms1xx.urdf.xacro" />
-  <xacro:macro name="sick_lms1xx_mount" params="prefix topic parent_link *origin">
+  <xacro:macro name="sick_lms1xx_inverted_mount" params="prefix topic parent_link *origin">
     <xacro:sick_lms1xx frame="${prefix}_laser" topic="${topic}" />
     <joint name="${prefix}_laser_mount_joint" type="fixed">
@@ -39,5 +39,5 @@
         <geometry>
           <!-- Origin of this mesh is the base of the bracket. -->
-          <mesh filename="package://jackal_description/meshes/sick-lms1xx-bracket.stl" />
+          <mesh filename="package://jackal_description/meshes/sick-lms1xx-inverted-bracket.stl" />
         </geometry>
         <material name="dark_grey" />

Commit message: Updated Novatel Smart7 Mount

File: jackal_description/urdf/accessories.urdf.xacro (robot description, xacro)
@@ -180,10 +180,10 @@
       <!-- Tower Enabled -->
       <xacro:if value="${tower}">
-        <xacro:novatel_smart7_stand prefix="${prefix}" parent="${parent}" height="$(optenv JACKAL_NAVSAT_HEIGHT 0.145)">
-          <origin xyz="$(optenv JACKAL_NAVSAT_OFFSET 0 0 0)" rpy="$(optenv JACKAL_NAVSAT_RPY 0 0 0)" />
-        </xacro:novatel_smart7_stand>
+        <xacro:bridge_plate prefix="${prefix}" parent="${parent}" height="$(optenv JACKAL_NAVSAT_HEIGHT 0.1)">
+          <origin xyz="$(optenv JACKAL_NAVSAT_OFFSET 0 0 0)" rpy="$(optenv JACKAL_NAVSAT_RPY 0 0 0)"/>
+        </xacro:bridge_plate>
         <joint name="${prefix}_navsat_joint" type="fixed">
-          <origin xyz="0 0 $(optenv JACKAL_NAVSAT_HEIGHT 0.145)" rpy="0 0 0"/>
-          <parent link="${prefix}_navsat_stand" />
+          <origin xyz="0 0 0" rpy="0 0 0" />
+          <parent link="${prefix}_bridge" />
           <child link="${prefix}_navsat" />
         </joint>

Commit message: Updated inverted position

File: jackal_description/urdf/accessories.urdf.xacro (robot description, xacro)
@@ -14,5 +14,4 @@
   <xacro:include filename="$(find jackal_description)/urdf/accessories/bridge_plate.urdf.xacro" />
   <!-- 2D Lidars -->
-  <xacro:include filename="$(find lms1xx)/urdf/sick_lms1xx.urdf.xacro" />
   <xacro:include filename="$(find jackal_description)/urdf/accessories/sick_lms1xx_inverted_mount.urdf.xacro" />
   <xacro:include filename="$(find jackal_description)/urdf/accessories/sick_lms1xx_upright_mount.urdf.xacro" />

File: jackal_description/urdf/accessories/sick_lms1xx_inverted_mount.urdf.xacro (robot description, xacro)
@@ -46,5 +46,5 @@
     <joint name="${prefix}_laser_joint" type="fixed">
       <!-- This offset is from the base of the bracket to the LIDAR's focal point. -->
-      <origin xyz="0 0 0.149" rpy="0 0 0" />
+      <origin xyz="0.04 0 0.066" rpy="3.141592 0 0" />
       <parent link="${prefix}_laser_mount" />
       <child link="${prefix}_laser" />
