Commit message: Updated Mounts (#104)
* Maintained backward compatibility with LMS1xx standard upright poisition by adding mount types

* Updated Novatel Smart7 Mount

* Updated inverted position

File: jackal_description/urdf/accessories.urdf.xacro (robot description, xacro)
@@ -14,6 +14,6 @@
   <xacro:include filename="$(find jackal_description)/urdf/accessories/bridge_plate.urdf.xacro" />
   <!-- 2D Lidars -->
-  <xacro:include filename="$(find lms1xx)/urdf/sick_lms1xx.urdf.xacro" />
-  <xacro:include filename="$(find jackal_description)/urdf/accessories/sick_lms1xx_mount.urdf.xacro" />
+  <xacro:include filename="$(find jackal_description)/urdf/accessories/sick_lms1xx_inverted_mount.urdf.xacro" />
+  <xacro:include filename="$(find jackal_description)/urdf/accessories/sick_lms1xx_upright_mount.urdf.xacro" />
   <xacro:include filename="$(find jackal_description)/urdf/accessories/hokuyo_ust10.urdf.xacro" />
   <xacro:include filename="$(find jackal_description)/urdf/accessories/vlp16_mount.urdf.xacro" />
@@ -33,11 +33,19 @@
     <xacro:property name="parent" value="$(optenv JACKAL_LASER_PARENT ${mount}_mount)" />
     <xacro:property name="lidar_model" value="$(optenv JACKAL_LASER_MODEL lms1xx)" />
+    <xacro:property name="mount_type" value="$(optenv JACKAL_LASER_MOUNT_TYPE upright)" />
     <!-- SICK LMS1xx -->
     <xacro:if value="${lidar_model == 'lms1xx'}">
       <!-- Mount Enabled -->
       <xacro:if value="${tower}">
-        <xacro:sick_lms1xx_mount topic="${topic}" prefix="${prefix}" parent_link="${parent}">
-          <origin xyz="$(optenv JACKAL_LASER_OFFSET 0 0 0)" rpy="$(optenv JACKAL_LASER_RPY 0 0 0)" />
-        </xacro:sick_lms1xx_mount>
+        <xacro:if value="${mount_type == 'upright'}">
+          <xacro:sick_lms1xx_upright_mount topic="${topic}" prefix="${prefix}" parent_link="${parent}">
+            <origin xyz="$(optenv JACKAL_LASER_OFFSET 0 0 0)" rpy="$(optenv JACKAL_LASER_RPY 0 0 0)" />
+          </xacro:sick_lms1xx_upright_mount>
+        </xacro:if>
+        <xacro:if value="${mount_type == 'inverted'}">
+          <xacro:sick_lms1xx_inverted_mount topic="${topic}" prefix="${prefix}" parent_link="${parent}">
+            <origin xyz="$(optenv JACKAL_LASER_OFFSET 0 0 0)" rpy="$(optenv JACKAL_LASER_RPY 0 0 0)" />
+          </xacro:sick_lms1xx_inverted_mount>
+        </xacro:if>
       </xacro:if>
       <!-- Mount Disabled -->
@@ -171,10 +179,10 @@
       <!-- Tower Enabled -->
       <xacro:if value="${tower}">
-        <xacro:novatel_smart7_stand prefix="${prefix}" parent="${parent}" height="$(optenv JACKAL_NAVSAT_HEIGHT 0.145)">
-          <origin xyz="$(optenv JACKAL_NAVSAT_OFFSET 0 0 0)" rpy="$(optenv JACKAL_NAVSAT_RPY 0 0 0)" />
-        </xacro:novatel_smart7_stand>
+        <xacro:bridge_plate prefix="${prefix}" parent="${parent}" height="$(optenv JACKAL_NAVSAT_HEIGHT 0.1)">
+          <origin xyz="$(optenv JACKAL_NAVSAT_OFFSET 0 0 0)" rpy="$(optenv JACKAL_NAVSAT_RPY 0 0 0)"/>
+        </xacro:bridge_plate>
         <joint name="${prefix}_navsat_joint" type="fixed">
-          <origin xyz="0 0 $(optenv JACKAL_NAVSAT_HEIGHT 0.145)" rpy="0 0 0"/>
-          <parent link="${prefix}_navsat_stand" />
+          <origin xyz="0 0 0" rpy="0 0 0" />
+          <parent link="${prefix}_bridge" />
           <child link="${prefix}_navsat" />
         </joint>

Commit message: Added JACKAL_IMU_MICROSTRAIN environment variable to accessories

File: jackal_description/urdf/accessories.urdf.xacro (robot description, xacro)
@@ -19,4 +19,25 @@
   <xacro:include filename="$(find jackal_description)/urdf/accessories/vlp16_mount.urdf.xacro" />
   <xacro:include filename="$(find jackal_description)/urdf/accessories/hdl32_mount.urdf.xacro" />
+  <!--
+    Add Microstrain IMU. By default the Jackal comes equipped with an IMU linked to "imu_link". These extra
+    optional microstrain IMU's will be added to another frame, by default, "microstrain_link".
+  -->
+  <xacro:property name="microstrain_enable" value="$(optenv JACKAL_GX5_IMU 0)"/>
+  <xacro:property name="microstrain_enable" value="$(optenv JACKAL_IMU_MICROSTRAIN ${microstrain_enable})" lazy_eval="false"/>
+  <xacro:if value="${microstrain_enable}">
+    <xacro:property name="frame"  value="$(optenv JACKAL_IMU_MICROSTRAIN_LINK microstrain_link)"/>
+    <xacro:property name="parent" value="$(optenv JACKAL_GX5_IMU_PARENT base_link)"/>
+    <xacro:property name="parent" value="$(optenv JACKAL_IMU_MICROSTRAIN_PARENT ${parent})" lazy_eval="false"/>
+    <xacro:property name="xyz"    value="$(optenv JACKAL_GX5_IMU_OFFSET -0.139 0.096 0.100)"/>
+    <xacro:property name="xyz"    value="$(optenv JACKAL_IMU_MICROSTRAIN_OFFSET ${xyz})" lazy_eval="false"/>
+    <xacro:property name="rpy"    value="$(optenv JACKAL_GX5_IMU_RPY ${PI} 0 -${PI/2})"/>
+    <xacro:property name="rpy"    value="$(optenv JACKAL_IMU_MICROSTRAIN_RPY ${rpy})" lazy_eval="false"/>
+    <link name="${frame}" />
+    <joint name="${frame}_joint" type="fixed">
+      <parent link="${parent}" />
+      <child link="${frame}" />
+      <origin xyz="${xyz}" rpy="${rpy}" />
+    </joint>
+  </xacro:if>
   <!--
     Add primary/secondary 2D lidar sensors.  By default these are SICK LMS1xx but can be changed with the

File: jackal_description/urdf/jackal.urdf.xacro (robot description, xacro)
@@ -203,16 +203,4 @@
     <origin xyz="-0.180 0.126 0.1815" />
   </joint>
-  <!--
-    Optionally add a GX5 IMU
-  -->
-  <xacro:if value="$(optenv JACKAL_GX5_IMU 0)">
-    <link name="gx5_link" />
-    <joint name="gx5_joint" type="fixed">
-      <parent link="$(optenv JACKAL_GX5_IMU_PARENT base_link)" />
-      <child link="gx5_link" />
-      <!-- TODO This offset & rotation may not be final, but it's good enough for now.  May update, pending RSCI-10 -->
-      <origin xyz="$(optenv JACKAL_GX5_IMU_OFFSET -0.139 0.096 0.100)" rpy="$(optenv JACKAL_GX5_IMU_RPY ${PI} 0 -${PI/2})" />
-    </joint>
-  </xacro:if>
   <link name="mid_mount"></link>
   <joint name="mid_mount_joint" type="fixed">

Commit message: Updated Microstrain Environment Variables (#105)
* Added JACKAL_IMU_MICROSTRAIN environment variable to accessories

* Updated variables in control.launch

File: jackal_description/urdf/accessories.urdf.xacro (robot description, xacro)
@@ -19,4 +19,25 @@
   <xacro:include filename="$(find jackal_description)/urdf/accessories/vlp16_mount.urdf.xacro" />
   <xacro:include filename="$(find jackal_description)/urdf/accessories/hdl32_mount.urdf.xacro" />
+  <!--
+    Add Microstrain IMU. By default the Jackal comes equipped with an IMU linked to "imu_link". These extra
+    optional microstrain IMU's will be added to another frame, by default, "microstrain_link".
+  -->
+  <xacro:property name="microstrain_enable" value="$(optenv JACKAL_GX5_IMU 0)"/>
+  <xacro:property name="microstrain_enable" value="$(optenv JACKAL_IMU_MICROSTRAIN ${microstrain_enable})" lazy_eval="false"/>
+  <xacro:if value="${microstrain_enable}">
+    <xacro:property name="frame"  value="$(optenv JACKAL_IMU_MICROSTRAIN_LINK microstrain_link)"/>
+    <xacro:property name="parent" value="$(optenv JACKAL_GX5_IMU_PARENT base_link)"/>
+    <xacro:property name="parent" value="$(optenv JACKAL_IMU_MICROSTRAIN_PARENT ${parent})" lazy_eval="false"/>
+    <xacro:property name="xyz"    value="$(optenv JACKAL_GX5_IMU_OFFSET -0.139 0.096 0.100)"/>
+    <xacro:property name="xyz"    value="$(optenv JACKAL_IMU_MICROSTRAIN_OFFSET ${xyz})" lazy_eval="false"/>
+    <xacro:property name="rpy"    value="$(optenv JACKAL_GX5_IMU_RPY ${PI} 0 -${PI/2})"/>
+    <xacro:property name="rpy"    value="$(optenv JACKAL_IMU_MICROSTRAIN_RPY ${rpy})" lazy_eval="false"/>
+    <link name="${frame}" />
+    <joint name="${frame}_joint" type="fixed">
+      <parent link="${parent}" />
+      <child link="${frame}" />
+      <origin xyz="${xyz}" rpy="${rpy}" />
+    </joint>
+  </xacro:if>
   <!--
     Add primary/secondary 2D lidar sensors.  By default these are SICK LMS1xx but can be changed with the

Commit message: Added UTM30

File: jackal_description/urdf/accessories.urdf.xacro (robot description, xacro)
@@ -15,5 +15,11 @@
   <!-- 2D Lidars -->
   <xacro:include filename="$(find lms1xx)/urdf/sick_lms1xx.urdf.xacro" />
+<<<<<<< Updated upstream
   <xacro:include filename="$(find jackal_description)/urdf/accessories/sick_lms1xx_mount.urdf.xacro" />
+=======
+  <xacro:include filename="$(find jackal_description)/urdf/accessories/sick_lms1xx_inverted_mount.urdf.xacro" />
+  <xacro:include filename="$(find jackal_description)/urdf/accessories/sick_lms1xx_upright_mount.urdf.xacro" />
+  <xacro:include filename="$(find jackal_description)/urdf/accessories/hokuyo_utm30.urdf.xacro" />
+>>>>>>> Stashed changes
   <xacro:include filename="$(find jackal_description)/urdf/accessories/hokuyo_ust10.urdf.xacro" />
   <xacro:include filename="$(find jackal_description)/urdf/accessories/vlp16_mount.urdf.xacro" />
@@ -41,4 +47,5 @@
     - lms1xx (default) :: SICK LMS1xx
     - ust10            :: Hokuyo UST10
+    - utm30            :: Hokuyo UTM30
   -->
   <!-- Primary 2D Lidar -->
@@ -80,4 +87,10 @@
       </xacro:hokuyo_ust10_mount>
     </xacro:if>
+    <!-- Hokuyo UTM30 -->
+    <xacro:if value="${lidar_model == 'utm30'}">
+      <xacro:hokuyo_utm30_mount topic="${topic}" prefix="${prefix}" parent_link="${parent}">
+        <origin xyz="$(optenv JACKAL_LASER_OFFSET 0 0 0)" rpy="$(optenv JACKAL_LASER_RPY 0 0 0)" />
+      </xacro:hokuyo_utm30_mount>
+    </xacro:if>
   </xacro:if>
   <!-- Secondary 2D Lidar -->
@@ -119,4 +132,10 @@
       </xacro:hokuyo_ust10_mount>
     </xacro:if>
+    <!-- Hokuyo UTM30 -->
+    <xacro:if value="${lidar_model == 'utm30'}">
+      <xacro:hokuyo_utm30_mount topic="${topic}" prefix="${prefix}" parent_link="${parent}">
+        <origin xyz="$(optenv JACKAL_LASER_SECONDARY_OFFSET 0 0 0)" rpy="$(optenv JACKAL_LASER_SECONDARY_RPY 0 0 3.14159)" />
+      </xacro:hokuyo_utm30_mount>
+    </xacro:if>
   </xacro:if>
   <!--

Commit message: Merge from luis-camero/noetic-tim
Added SICK TIM551 to URDF and package.xml

File: jackal_description/urdf/accessories.urdf.xacro (robot description, xacro)
@@ -14,4 +14,6 @@
   <xacro:include filename="$(find jackal_description)/urdf/accessories/bridge_plate.urdf.xacro" />
   <!-- 2D Lidars -->
+  <xacro:include filename="$(find sick_tim)/urdf/sick_tim.urdf.xacro" />
+  <xacro:include filename="$(find lms1xx)/urdf/sick_lms1xx.urdf.xacro" />
   <xacro:include filename="$(find jackal_description)/urdf/accessories/sick_lms1xx_inverted_mount.urdf.xacro" />
   <xacro:include filename="$(find jackal_description)/urdf/accessories/sick_lms1xx_upright_mount.urdf.xacro" />
@@ -86,4 +88,14 @@
       </xacro:unless>
     </xacro:if>
+    <!-- SICK Tim -->
+    <xacro:if value="${lidar_model == 'tim551'}">
+      <xacro:property name="prefix" value="$(optenv JACKAL_LASER_PREFIX tim551)" />
+      <xacro:sick_tim551 name="${prefix}" ros_topic="${topic}"/>
+      <joint name="${prefix}_mount_link_joint" type="fixed">
+        <origin xyz="$(optenv JACKAL_LASER_OFFSET 0 0 0)" rpy="$(optenv JACKAL_LASER_RPY 0 0 0)"/>
+        <parent link="${parent}"/>
+        <child link="${prefix}_mount_link"/>
+      </joint>
+    </xacro:if>
     <!-- Hokuyo UST10 -->
     <xacro:if value="${lidar_model == 'ust10'}">
@@ -125,4 +137,14 @@
       </xacro:unless>
     </xacro:if>
+    <!-- SICK Tim -->
+    <xacro:if value="${lidar_model == 'tim551'}">
+      <xacro:property name="prefix" value="$(optenv JACKAL_LASER_SECONDARY_PREFIX tim551_2)" />
+      <xacro:sick_tim551 name="${prefix}" ros_topic="${topic}"/>
+      <joint name="${prefix}_mount_link_joint" type="fixed">
+        <origin xyz="$(optenv JACKAL_LASER_SECONDARY_OFFSET 0 0 0)" rpy="$(optenv JACKAL_LASER_SECONDARY_RPY 0 0 3.14159)"/>
+        <parent link="${parent}"/>
+        <child link="${prefix}_mount_link"/>
+      </joint>
+    </xacro:if>
     <!-- Hokuyo UST10 -->
     <xacro:if value="${lidar_model == 'ust10'}">

Commit message: Added ros2_control to description

File: jackal_description/urdf/accessories.urdf.xacro (robot description, xacro)
@@ -16,7 +16,7 @@
   <!--xacro:include filename="$(find lms1xx)/urdf/sick_lms1xx.urdf.xacro" />
   <xacro:include filename="$(find jackal_description)/urdf/accessories/sick_lms1xx_mount.urdf.xacro" /-->
-  <xacro:include filename="$(find jackal_description)/urdf/accessories/hokuyo_ust10.urdf.xacro" />
+  <!-- <xacro:include filename="$(find jackal_description)/urdf/accessories/hokuyo_ust10.urdf.xacro" />
   <xacro:include filename="$(find jackal_description)/urdf/accessories/vlp16_mount.urdf.xacro" />
-  <xacro:include filename="$(find jackal_description)/urdf/accessories/hdl32_mount.urdf.xacro" />
+  <xacro:include filename="$(find jackal_description)/urdf/accessories/hdl32_mount.urdf.xacro" /> -->
   <!--
     Add primary/secondary 2D lidar sensors.  By default these are SICK LMS1xx but can be changed with the

File: jackal_description/urdf/jackal.urdf.xacro (robot description, xacro)
@@ -1,4 +1,5 @@
 <?xml version="1.0"?>
 <robot name="jackal" xmlns:xacro="http://www.ros.org/wiki/xacro">
+  <xacro:arg name="is_sim" default="false" />
   <xacro:property name="PI" value="3.1415926535897931" />
   <xacro:property name="wheelbase" value="0.262" />
@@ -50,5 +51,5 @@
       <fdir1 value="1 0 0"/>
     </gazebo>
-    <joint name="${prefix}_wheel" type="continuous">
+    <joint name="${prefix}_wheel_joint" type="continuous">
       <parent link="chassis_link"/>
       <child link="${prefix}_wheel_link" />
@@ -221,4 +222,53 @@
     <origin xyz="${mount_spacing} 0 0" />
   </joint>
+  <ros2_control name="jackal_hardware" type="system">
+    <hardware>
+      <xacro:if value="$(arg is_sim)">
+        <plugin>gazebo_ros2_control/GazeboSystem</plugin>
+      </xacro:if>
+      <xacro:unless value="$(arg is_sim)">
+        <plugin>jackal_base/JackalHardware</plugin>
+        <plugin>fake_components/GenericSystem</plugin>
+        <param name="hw_start_duration_sec">2.0</param>
+        <param name="hw_stop_duration_sec">3.0</param>
+        <param name="wheel_diameter">0.196</param>
+        <param name="max_accel">5.0</param>
+        <param name="max_speed">1.0</param>
+        <param name="polling_timeout">10.0</param>
+      </xacro:unless>
+    </hardware>
+    <joint name="front_left_wheel_joint">
+      <command_interface name="velocity">
+        <param name="min">-1</param>
+        <param name="max">1</param>
+      </command_interface>
+      <state_interface name="position"/>
+      <state_interface name="velocity"/>
+    </joint>
+    <joint name="rear_left_wheel_joint">
+      <command_interface name="velocity">
+        <param name="min">-1</param>
+        <param name="max">1</param>
+      </command_interface>
+      <state_interface name="position"/>
+      <state_interface name="velocity"/>
+    </joint>
+    <joint name="front_right_wheel_joint">
+      <command_interface name="velocity">
+        <param name="min">-1</param>
+        <param name="max">1</param>
+      </command_interface>
+      <state_interface name="position"/>
+      <state_interface name="velocity"/>
+    </joint>
+    <joint name="rear_right_wheel_joint">
+      <command_interface name="velocity">
+        <param name="min">-1</param>
+        <param name="max">1</param>
+      </command_interface>
+      <state_interface name="position"/>
+      <state_interface name="velocity"/>
+    </joint>
+  </ros2_control>
   <!-- Bring in simulation data for Gazebo. -->
   <xacro:include filename="$(find jackal_description)/urdf/jackal.gazebo" />

Commit message: Added Nav2 and slam_toolbox to jackal_navigation

File: jackal_description/urdf/accessories.urdf.xacro (robot description, xacro)
@@ -14,9 +14,9 @@
   <xacro:include filename="$(find jackal_description)/urdf/accessories/bridge_plate.urdf.xacro" />
   <!-- 2D Lidars -->
-  <!--xacro:include filename="$(find lms1xx)/urdf/sick_lms1xx.urdf.xacro" />
-  <xacro:include filename="$(find jackal_description)/urdf/accessories/sick_lms1xx_mount.urdf.xacro" /-->
-  <!-- <xacro:include filename="$(find jackal_description)/urdf/accessories/hokuyo_ust10.urdf.xacro" />
+  <!-- <xacro:include filename="$(find lms1xx)/urdf/sick_lms1xx.urdf.xacro" />
+  <xacro:include filename="$(find jackal_description)/urdf/accessories/sick_lms1xx_mount.urdf.xacro" />-->
+  <xacro:include filename="$(find jackal_description)/urdf/accessories/hokuyo_ust10.urdf.xacro" />
   <xacro:include filename="$(find jackal_description)/urdf/accessories/vlp16_mount.urdf.xacro" />
-  <xacro:include filename="$(find jackal_description)/urdf/accessories/hdl32_mount.urdf.xacro" /> -->
+  <xacro:include filename="$(find jackal_description)/urdf/accessories/hdl32_mount.urdf.xacro" />
   <!--
     Add primary/secondary 2D lidar sensors.  By default these are SICK LMS1xx but can be changed with the
@@ -32,5 +32,5 @@
     <xacro:property name="prefix" value="$(optenv JACKAL_LASER_PREFIX ${mount})" />
     <xacro:property name="parent" value="$(optenv JACKAL_LASER_PARENT ${mount}_mount)" />
-    <xacro:property name="lidar_model" value="$(optenv JACKAL_LASER_MODEL lms1xx)" />
+    <xacro:property name="lidar_model" value="$(optenv JACKAL_LASER_MODEL ust10)" />
     <!-- SICK LMS1xx -->
     <xacro:if value="${lidar_model == 'lms1xx'}">
@@ -71,5 +71,5 @@
     <xacro:property name="prefix" value="$(optenv JACKAL_LASER_SECONDARY_PREFIX ${mount})" />
     <xacro:property name="parent" value="$(optenv JACKAL_LASER_SECONDARY_PARENT ${mount}_mount)" />
-    <xacro:property name="lidar_model" value="$(optenv JACKAL_LASER_SECONDARY_MODEL lms1xx)" />
+    <xacro:property name="lidar_model" value="$(optenv JACKAL_LASER_SECONDARY_MODEL ust10)" />
     <!-- SICK LMS1xx -->
     <xacro:if value="${lidar_model == 'lms1xx'}">

Commit message: Remove recursive variable definition of microstrain_enable

File: jackal_description/urdf/accessories.urdf.xacro (robot description, xacro)
@@ -26,5 +26,5 @@
   -->
   <xacro:property name="microstrain_enable" value="$(optenv JACKAL_GX5_IMU 0)"/>
-  <xacro:property name="microstrain_enable" value="$(optenv JACKAL_IMU_MICROSTRAIN ${microstrain_enable})" lazy_eval="false"/>
+  <xacro:property name="microstrain_enable" value="$(optenv JACKAL_IMU_MICROSTRAIN 0)" lazy_eval="false"/>
   <xacro:if value="${microstrain_enable}">
     <xacro:property name="frame"  value="$(optenv JACKAL_IMU_MICROSTRAIN_LINK microstrain_link)"/>

Commit message: Integrated sick-lms1xx lidar

File: jackal_description/urdf/accessories.urdf.xacro (robot description, xacro)
@@ -14,6 +14,6 @@
   <xacro:include filename="$(find jackal_description)/urdf/accessories/bridge_plate.urdf.xacro" />
   <!-- 2D Lidars -->
-  <!-- <xacro:include filename="$(find lms1xx)/urdf/sick_lms1xx.urdf.xacro" />
-  <xacro:include filename="$(find jackal_description)/urdf/accessories/sick_lms1xx_mount.urdf.xacro" />-->
+  <xacro:include filename="$(find jackal_description)/urdf/accessories/sick_lms1xx.urdf.xacro" />
+  <xacro:include filename="$(find jackal_description)/urdf/accessories/sick_lms1xx_mount.urdf.xacro" />
   <xacro:include filename="$(find jackal_description)/urdf/accessories/hokuyo_ust10.urdf.xacro" />
   <xacro:include filename="$(find jackal_description)/urdf/accessories/vlp16_mount.urdf.xacro" />
@@ -26,11 +26,11 @@
   -->
   <!-- Primary 2D Lidar -->
-  <xacro:if value="$(optenv JACKAL_LASER 0)">
+  <xacro:if value="$(optenv JACKAL_LASER 1)">
     <xacro:property name="mount" value="$(optenv JACKAL_LASER_MOUNT front)" />
-    <xacro:property name="topic" value="$(optenv JACKAL_LASER_TOPIC front/scan)" />
+    <xacro:property name="topic" value="$(optenv JACKAL_LASER_TOPIC /scan)" />
     <xacro:property name="tower" value="$(optenv JACKAL_LASER_TOWER 1)" />
     <xacro:property name="prefix" value="$(optenv JACKAL_LASER_PREFIX ${mount})" />
     <xacro:property name="parent" value="$(optenv JACKAL_LASER_PARENT ${mount}_mount)" />
-    <xacro:property name="lidar_model" value="$(optenv JACKAL_LASER_MODEL ust10)" />
+    <xacro:property name="lidar_model" value="$(optenv JACKAL_LASER_MODEL lms1xx)" />
     <!-- SICK LMS1xx -->
     <xacro:if value="${lidar_model == 'lms1xx'}">
@@ -107,10 +107,10 @@
     JACKAL_LASER_3D_MODEL environment variable. Valid model designations are:
     - vlp16 (default)  :: Velodyne VLP16
-    - vlp32e           :: Velodyne HDL-32E
+    - hdl32e           :: Velodyne HDL-32E
   -->
   <xacro:if value="$(optenv JACKAL_LASER_3D 0)">
     <xacro:property name="mount" value="$(optenv JACKAL_LASER_3D_MOUNT mid)" />
-    <xacro:property name="topic" value="$(optenv JACKAL_LASER_3D_TOPIC mid/points)" />
-    <xacro:property name="tower" value="$(optenv JACKAL_LASER_3D_TOWER 1)" />
+    <xacro:property name="topic" value="$(optenv JACKAL_LASER_3D_TOPIC points)" />
+    <xacro:property name="tower" value="$(optenv JACKAL_LASER_3D_TOWER 0)" />
     <xacro:property name="prefix" value="$(optenv JACKAL_LASER_3D_PREFIX ${mount})" />
     <xacro:property name="parent" value="$(optenv JACKAL_LASER_3D_PARENT ${mount}_mount)" />

File: jackal_description/urdf/accessories/sick_lms1xx_mount.urdf.xacro (robot description, xacro)
@@ -26,5 +26,5 @@
 -->
 <robot xmlns:xacro="http://www.ros.org/wiki/xacro">
-  <xacro:include filename="$(find lms1xx)/urdf/sick_lms1xx.urdf.xacro" />
+  <xacro:include filename="$(find jackal_description)/urdf/accessories/sick_lms1xx.urdf.xacro" />
   <xacro:macro name="sick_lms1xx_mount" params="prefix topic parent_link *origin">
     <xacro:sick_lms1xx frame="${prefix}_laser" topic="${topic}" />

Commit message: 

File: jackal_description/urdf/accessories.urdf.xacro (robot description, xacro)
@@ -109,8 +109,8 @@
     - hdl32e           :: Velodyne HDL-32E
   -->
-  <xacro:if value="$(optenv JACKAL_LASER_3D 0)">
+  <xacro:if value="$(optenv JACKAL_LASER_3D 1)">
     <xacro:property name="mount" value="$(optenv JACKAL_LASER_3D_MOUNT mid)" />
     <xacro:property name="topic" value="$(optenv JACKAL_LASER_3D_TOPIC points)" />
-    <xacro:property name="tower" value="$(optenv JACKAL_LASER_3D_TOWER 0)" />
+    <xacro:property name="tower" value="$(optenv JACKAL_LASER_3D_TOWER 1)" />
     <xacro:property name="prefix" value="$(optenv JACKAL_LASER_3D_PREFIX ${mount})" />
     <xacro:property name="parent" value="$(optenv JACKAL_LASER_3D_PARENT ${mount}_mount)" />
